File: Hardware/PCB/3340vco/3340vco.kicad_pcb (KiCad board)
At the start: 2 copper layers, 105 parts, among them J1 Conn_01x10, J10 AudioJack2, J11 AudioJack2, J12 AudioJack2, J13 AudioJack2, J14 AudioJack2, J2 4 pin Molex connector, J3 Conn_01x10, J4 Synth_power_2x5, J5 AudioJack2, J6 AudioJack2, J7 AudioJack2, J8 AudioJack2, J9 AudioJack2, Q1 MMBFJ201, Q2 J201, SW1 SW_Rotary12, SW2 SW_SPDT, U1 TL072, U2 CEM3340, U3 TL074, U4 LM4040AIZ-8.2, U5 L79L05_TO92

Commit message: Preliminary board division and layout
Parts:
- removed the C11 at (88.6, 247.1)
- removed the C12 at (385.1, 108.2)
- removed the C13 at (385.1, 111.3)
- removed the C8 at (399.3, 48.1)
- removed the D1 at (462.8, 80.0)
- removed the D2 at (437.7, 87.3)
- removed the J2 at (398.0, 85.5)
- removed the R1 at (396.3, 94.3)
- removed the R2 at (439.2, 51.1)
- removed the R21 at (424.4, 81.7)
- removed the R22 at (437.7, 67.3)
- removed the R24 at (422.9, 93.9)
- removed the R26 at (437.7, 71.4)
- removed the RV8 at (155.0, 90.0)
- removed the RV9 at (224.0, 71.0)
- added C10: 100nF, ao_tht:C_Disc_D3.0mm_W1.6mm_P2.50mm, B.Cu at (193.0, 96.5)
- added C15: 100nF, ao_tht:C_Disc_D3.0mm_W1.6mm_P2.50mm, F.Cu at (411.0, 63.7)
- added C16: 180pF, ao_tht:C_Disc_D3.0mm_W1.6mm_P2.50mm, F.Cu at (411.0, 60.6)
- added C17: 180pF, ao_tht:C_Disc_D3.0mm_W1.6mm_P2.50mm, F.Cu at (413.2, 57.4)
- added C2: 10nF, ao_tht:C_Rect_L7.2mm_W2.5mm_P5.00mm_FKS2_FKP2_MKS2_MKP2, B.Cu at (168.9, 125.7)
- added C9: 100nF, ao_tht:C_Disc_D3.0mm_W1.6mm_P2.50mm, B.Cu at (174.0, 88.9)
- added D4: 1N4148, Diode_THT:D_DO-35_SOD27_P7.62mm_Horizontal, F.Cu at (399.9, 72.3)
- added D5: 1N4148, Diode_THT:D_DO-35_SOD27_P7.62mm_Horizontal, F.Cu at (386.6, 75.7)
- added D6: 1N4732A, Diode_THT:D_DO-41_SOD81_P10.16mm_Horizontal, B.Cu at (197.0, 71.0)
- added GRAF2: Holes, 3340vco:3340vco_panel_holes, F.Cu at (300.0, 115.0)
- added H1: MountingHole, ao_tht:MountingHole_3.2mm_M3, F.Cu at (172.5, 31.5)
- added H2: MountingHole, ao_tht:MountingHole_3.2mm_M3, F.Cu at (136.0, 112.0)
- added H3: MountingHole, ao_tht:MountingHole_3.2mm_M3, F.Cu at (224.0, 151.0)
- added H4: MountingHole, ao_tht:MountingHole_3.2mm_M3, F.Cu at (292.5, 31.5)
- added H5: MountingHole, ao_tht:MountingHole_3.2mm_M3, F.Cu at (256.0, 112.0)
- added H6: MountingHole, ao_tht:MountingHole_3.2mm_M3, F.Cu at (344.0, 151.0)
- added J1: Conn_02x04_Odd_Even, Connector_IDC:IDC-Header_2x04_P2.54mm_Vertical, F.Cu at (261.6, 38.1)
- added J16: 3_pin_Molex_connector, ao_tht:Molex_KK-254_AE-6410-03A_1x03_P2.54mm_Vertical, F.Cu at (-91.4, 12.7)
- added J17: Conn_01x03, Connector_PinHeader_2.54mm:PinHeader_1x03_P2.54mm_Vertical, B.Cu at (168.9, 83.8)
- added J18: Conn_01x03, Connector_PinSocket_2.54mm:PinSocket_1x03_P2.54mm_Vertical, F.Cu at (288.9, 83.8)
- added J19: Conn_01x03, Connector_PinHeader_2.54mm:PinHeader_1x03_P2.54mm_Vertical, B.Cu at (168.9, 101.6)
- added J20: Conn_01x03, Connector_PinSocket_2.54mm:PinSocket_1x03_P2.54mm_Vertical, F.Cu at (288.9, 101.6)
- added J3: 3_pin_Molex_header, ao_tht:Molex_KK-254_AE-6410-03A_1x03_P2.54mm_Vertical, B.Cu at (158.8, 68.6)
- added R11: 10k, ao_tht:R_Axial_DIN0207_L6.3mm_D2.5mm_P10.16mm_Horizontal, B.Cu at (198.0, 119.0)
- added R17: 100k, ao_tht:R_Axial_DIN0207_L6.3mm_D2.5mm_P10.16mm_Horizontal, B.Cu at (207.2, 101.0)
- added R18: 10k, ao_tht:R_Axial_DIN0207_L6.3mm_D2.5mm_P10.16mm_Horizontal, B.Cu at (174.0, 92.7)
- added R19: 47k, ao_tht:R_Axial_DIN0207_L6.3mm_D2.5mm_P10.16mm_Horizontal, B.Cu at (185.4, 53.3)
- added R49: 16k, ao_tht:R_Axial_DIN0207_L6.3mm_D2.5mm_P10.16mm_Horizontal, F.Cu at (373.2, 71.8)
- added R50: 18k, ao_tht:R_Axial_DIN0207_L6.3mm_D2.5mm_P10.16mm_Horizontal, F.Cu at (385.0, 59.7)
- added R51: 18k, ao_tht:R_Axial_DIN0207_L6.3mm_D2.5mm_P10.16mm_Horizontal, F.Cu at (386.6, 63.8)
- added R52: 18k, ao_tht:R_Axial_DIN0207_L6.3mm_D2.5mm_P10.16mm_Horizontal, F.Cu at (373.2, 75.9)
- added R53: 1k, ao_tht:R_Axial_DIN0207_L6.3mm_D2.5mm_P10.16mm_Horizontal, F.Cu at (398.3, 51.6)
- added R54: 1k, ao_tht:R_Axial_DIN0207_L6.3mm_D2.5mm_P10.16mm_Horizontal, F.Cu at (399.9, 55.6)
- added R55: 1k, ao_tht:R_Axial_DIN0207_L6.3mm_D2.5mm_P10.16mm_Horizontal, F.Cu at (386.6, 67.8)
- added R56: 300k, ao_tht:R_Axial_DIN0207_L6.3mm_D2.5mm_P10.16mm_Horizontal, B.Cu at (148.6, 71.1)
- added R57: 8.2k, ao_tht:R_Axial_DIN0207_L6.3mm_D2.5mm_P10.16mm_Horizontal, B.Cu at (207.2, 36.0)
- added R58: 1k, ao_tht:R_Axial_DIN0207_L6.3mm_D2.5mm_P10.16mm_Horizontal, B.Cu at (225.2, 35.0)
- added R9: 10k, ao_tht:R_Axial_DIN0207_L6.3mm_D2.5mm_P10.16mm_Horizontal, B.Cu at (208.2, 123.0)
- added RV12: 10k, ao_tht:Potentiometer_Bourns_3296W_Vertical_screw_centered, F.Cu at (224.0, 91.0)
- added RV13: 50k, ao_tht:Potentiometer_Bourns_3296W_Vertical_screw_centered, F.Cu at (224.0, 51.0)
- added RV2: 100k, ao_tht:Potentiometer_Alpha_RD901F-40-00D_Single_Vertical_CircularHoles_centered, F.Cu at (155.0, 90.0)
- added U6: TL074, ao_tht:DIP-14_W7.62mm_Socket_LongPads, F.Cu at (360.4, 47.6)
- C1: footprint ao_tht:C_Disc_D3.0mm_W1.6mm_P2.50mm -> ao_tht:C_Rect_L7.2mm_W2.5mm_P5.00mm_FKS2_FKP2_MKS2_MKP2; moved to B.Cu
- C13: renamed from C15; moved to B.Cu
- C14: value 0.1uF -> 100nF
- C3: value 100n -> 100nF; moved to B.Cu
- C4: value 1n -> 1nF; footprint ao_tht:C_Disc_D3.0mm_W1.6mm_P2.50mm -> ao_tht:C_Rect_L7.2mm_W2.5mm_P5.00mm_FKS2_FKP2_MKS2_MKP2; moved to B.Cu
- C5: value 10n -> 10nF; footprint ao_tht:C_Disc_D3.0mm_W1.6mm_P2.50mm -> ao_tht:C_Rect_L7.2mm_W2.5mm_P5.00mm_FKS2_FKP2_MKS2_MKP2; moved to B.Cu
- C6, C7: value 10pF -> 100nF; moved to B.Cu
- C8: renamed from C2; footprint ao_tht:C_Disc_D3.0mm_W1.6mm_P2.50mm -> ao_tht:C_Rect_L7.2mm_W2.5mm_P5.00mm_FKS2_FKP2_MKS2_MKP2; moved to B.Cu
- D3: renamed from D5; moved to B.Cu
- J2: renamed from J1; value Conn_01x10 -> Conn_01x11; footprint ao_tht:PinSocket_1x10_P2.54mm_Vertical -> Connector_PinHeader_2.54mm:PinHeader_1x11_P2.54mm_Vertical; moved to B.Cu
- J4: renamed from J3; value Conn_01x10 -> Conn_01x11; footprint ao_tht:PinHeader_1x10_P2.54mm_Vertical -> Connector_PinSocket_2.54mm:PinSocket_1x11_P2.54mm_Vertical
- R1: renamed from R3; value 10M -> 3M; moved to B.Cu
- R10: value 4.7k -> 100k; moved to B.Cu
- R12: renamed from R17; moved to B.Cu
- R13: renamed from R18; moved to B.Cu
- R14: renamed from R19; moved to B.Cu
- R15: renamed from R11; moved to B.Cu
- R16: renamed from R12; moved to B.Cu
- R2: renamed from R4; moved to B.Cu
- R20: value 1M -> 20k; moved to B.Cu
- R21: renamed from R6; value 470k -> 240k; moved to B.Cu
- R22: renamed from R7; value 470k -> 100k; moved to B.Cu
- R23: value 180k -> 1M; moved to B.Cu
- R24: renamed from R9; moved to B.Cu
- R25: value 100k -> 10k; moved to B.Cu
- R26: renamed from R49; value 4.7k -> 1k; footprint ao_tht:R_Axial_DIN0207_L6.3mm_D2.5mm_P7.62mm_Horizontal -> ao_tht:R_Axial_DIN0207_L6.3mm_D2.5mm_P10.16mm_Horizontal; moved to B.Cu
- R27, R28: value 240k -> 10k
- R29, R30: value 1k -> 10k
- R3: renamed from R5; moved to B.Cu
- R31, R32, R33: value 91k -> 10k
- R34: value 100k -> 10k
- R35, R36: value 100k -> 1M
- R4: renamed from R13; moved to B.Cu
- R40: value 1k -> 18k
- R41: value 100k -> 33k; footprint ao_tht:R_Axial_DIN0207_L6.3mm_D2.5mm_P7.62mm_Horizontal -> ao_tht:R_Axial_DIN0207_L6.3mm_D2.5mm_P10.16mm_Horizontal
- R42, R43: value 100k -> 18k; footprint ao_tht:R_Axial_DIN0207_L6.3mm_D2.5mm_P7.62mm_Horizontal -> ao_tht:R_Axial_DIN0207_L6.3mm_D2.5mm_P10.16mm_Horizontal
- R44, R45, R46: value 100k -> 43k; footprint ao_tht:R_Axial_DIN0207_L6.3mm_D2.5mm_P7.62mm_Horizontal -> ao_tht:R_Axial_DIN0207_L6.3mm_D2.5mm_P10.16mm_Horizontal
- R47, R48: value 100k -> 16k; footprint ao_tht:R_Axial_DIN0207_L6.3mm_D2.5mm_P7.62mm_Horizontal -> ao_tht:R_Axial_DIN0207_L6.3mm_D2.5mm_P10.16mm_Horizontal
- R5: renamed from R14; moved to B.Cu
- R6: renamed from R16; moved to B.Cu
- R7: renamed from R15; moved to B.Cu
- R8: value 1.5M -> 100k; moved to B.Cu
- SW1: value SW_Rotary12 -> SW_SPDT_MSM; footprint ao_tht:Rotary_Switch -> ao_tht:SPDT-toggle-switch-1M-series
- SW2: value SW_SPDT -> SW_Rotary12; footprint ao_tht:SPDT-toggle-switch-1M-series -> ao_tht:Rotary_Switch
- TP1: footprint MountingHole:MountingHole_2.2mm_M2_Pad -> TestPoint:TestPoint_Pad_2.5x2.5mm; moved to B.Cu
- U1: value TL072 -> TL074; footprint ao_tht:DIP-8_W7.62mm_Socket_LongPads -> ao_tht:DIP-14_W7.62mm_Socket_LongPads; moved to B.Cu
- U2: value CEM3340 -> AS3340A; moved to B.Cu
- U3: value TL074 -> TL072; footprint ao_tht:DIP-14_W7.62mm_Socket_LongPads -> ao_tht:DIP-8_W7.62mm_Socket_LongPads; moved to B.Cu
- U4: value LM4040AIZ-8.2 -> TL431LP; footprint Package_TO_SOT_THT:TO-92_Inline -> ao_tht:TO-92_Inline_Wide; moved to B.Cu
- U5: footprint Package_TO_SOT_THT:TO-92_Inline -> ao_tht:TO-92_Inline_Wide; moved to B.Cu
- moved R34 539.5 mm to (-67.7, -25.2)
- moved R28 537.3 mm to (-67.7, -13.0)
- moved R33 526.2 mm to (-67.7, -21.1)
- moved R31 523.2 mm to (-67.7, -4.92)
- moved R30 513.8 mm to (-67.7, -17.1)
- moved R32 503.1 mm to (-54.4, -25.2)
- moved R29 501.9 mm to (-67.7, -8.97)
- moved R27 490.6 mm to (-54.4, -21.1)
- moved C5 331.5 mm to (148.6, 78.7), turned to 180 degrees
- moved C6 311.7 mm to (174.0, 114.3), turned to 180 degrees
- moved R25 291.1 mm to (163.8, 96.5)
- moved C4 286.5 mm to (148.6, 74.9), turned to 180 degrees
- moved U1 276.4 mm to (179.1, 121.9)
- moved R5 271.7 mm to (174.0, 118.1), turned to 180 degrees
- moved R14 264.0 mm to (174.0, 74.9), turned to 180 degrees
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- renumbered C9 to C11, C10 to C12, D3 to D1, D4 to D2, J9 to J10, J10 to J11, J11 to J12, J12 to J13, J13 to J14, J14 to J15, J4 to J5, J5 to J6, J6 to J7, J7 to J8, J8 to J9, RV4 to RV1, RV7 to RV3, RV1 to RV7, RV2 to RV8, RV3 to RV9
Connections:
- C11 pad 2: GND -> GND1
- C12 pad 1: GND -> GND1
- C14 pad 1: GND -> +12V
- C14 pad 2: -12V -> GND1
- C3 pad 1: +12V -> +12V_P
- C6 pad 1: Net-(C6-Pad1) -> +12V_P
- C6 pad 2: Net-(C6-Pad2) -> GND
- C7 pad 1: Net-(C7-Pad1) -> GND
- C7 pad 2: Net-(C7-Pad2) -> -12V_P
- C8 pad 1: Net-(C2-Pad1) -> Net-(C8-Pad1)
- C8 pad 2: Net-(C2-Pad2) -> LINK_OUT_FM
- D3 pad 2: -12V -> -12V_P
- J15 pad T: CV_IN2_J -> V_OCT2_J
- J2 pad 10: SIN -> SIN_A_W
- J2 pad 3: CV_IN -> V_OCT2
- J2 pad 4: SYNC -> CV_IN
- J2 pad 5: LIN_FM_IN -> SYNC
- J2 pad 6: PWMIN -> LIN_FM_IN
- J2 pad 7: SAW -> PWMIN
- J2 pad 8: PULSE -> SIN_S_W
- J2 pad 9: TRI -> SIN_S_CCW
- J4 pad 10: SIN_J -> SIN_A_W_S
- J4 pad 3: CV_IN_J -> V_OCT2_J
- J4 pad 4: SYNC_J -> CV_IN_J
- J4 pad 5: LIN_FM_IN_J -> SYNC_J
- J4 pad 6: PWMIN_J -> LIN_FM_IN_J
- J4 pad 7: SAW_J -> PWMIN_J
- J4 pad 8: PULSE_J -> SIN_S_W_S
- J4 pad 9: TRI_J -> SIN_S_CCW_S
- J5 pad 3: GND -> GND1
- J5 pad 4: GND -> GND1
- J5 pad 5: GND -> GND1
- J5 pad 6: GND -> GND1
- J5 pad 7: GND -> GND1
- J5 pad 8: GND -> GND1
- Q1 pad 3: Net-(D1-Pad2) (its old number) -> Net-(D4-Pad2)
- Q2 pad 3: Net-(D1-Pad2) (its old number) -> Net-(D4-Pad2)
- R10 pad 1: GND -> Net-(R10-Pad1)
- R10 pad 2: PWM_IN -> Net-(R10-Pad2)
- R13 pad 1: +12V -> +12V_P
- R13 pad 2: Net-(R18-Pad2) -> LIN_FM
- R14 pad 1: Net-(R18-Pad2) -> LIN_FM
- R20 pad 1: /SIN_SHAPE -> Net-(R19-Pad1)
- R20 pad 2: Net-(D1-Pad2) (its old number) -> Net-(R18-Pad2)
- R21 pad 1: Net-(R6-Pad1) -> Net-(R21-Pad1)
- R22 pad 1: Net-(R6-Pad1) -> Net-(R21-Pad1)
- R23 pad 1: Net-(R23-Pad1) -> LIN_FM
- R23 pad 2: PULSE_OUT -> Net-(C8-Pad1)
- R24 pad 1: PWM_IN -> Net-(R18-Pad2)
- R24 pad 2: Net-(R9-Pad2) -> Net-(R21-Pad1)
- R25 pad 1: Net-(R23-Pad1) -> LINK_OUT_PW
- R25 pad 2: GND -> Net-(R18-Pad1)
- R26 pad 1: Net-(R49-Pad1) -> +8V_REF
- R26 pad 2: +12V -> +12V_P
- R27 pad 1: Net-(C6-Pad2) -> Net-(R27-Pad1)
- R27 pad 2: +12V -> /Panel components and power/+8V_REF_P
- R28 pad 1: Net-(C7-Pad2) -> Net-(R28-Pad1)
- R28 pad 2: +12V -> Net-(R27-Pad1)
- R29 pad 1: /SIN_SHAPE -> Net-(R29-Pad1)
- R29 pad 2: Net-(Q1-Pad1) -> Net-(R28-Pad1)
- R30 pad 1: Net-(Q1-Pad2) -> Net-(R30-Pad1)
- R30 pad 2: GND -> Net-(R29-Pad1)
- R31 pad 1: Net-(R26-Pad1) -> Net-(R31-Pad1)
- R31 pad 2: GND -> Net-(R30-Pad1)
- R32 pad 1: Net-(C6-Pad2) -> Net-(R32-Pad1)
- R32 pad 2: GND -> Net-(R31-Pad1)
- R33 pad 1: Net-(C7-Pad2) -> Net-(R33-Pad1)
- R33 pad 2: GND -> Net-(R32-Pad1)
- R34 pad 1: TRI_RAW -> /Panel components and power/0V
- R34 pad 2: Net-(R26-Pad1) -> Net-(R33-Pad1)
- R35 pad 1: Net-(C6-Pad1) -> SIN_S_W_S
- R35 pad 2: Net-(C6-Pad2) -> Net-(D4-Pad2)
- R36 pad 1: Net-(C7-Pad1) -> Net-(D4-Pad2)
- R36 pad 2: Net-(C7-Pad2) -> GND1
- R37 pad 1: SIN -> SIN_S_W_S
- R37 pad 2: Net-(R37-Pad2) -> Net-(Q1-Pad1)
- R38 pad 1: TRI -> Net-(Q1-Pad2)
- R38 pad 2: TRI_RAW -> GND1
- R39 pad 1: SAW -> SIN
- R39 pad 2: Net-(C6-Pad1) -> SIN_A_CCW_S
- R4 pad 1: CV_NODE -> Net-(R10-Pad2)
- R40 pad 1: PULSE -> Net-(R40-Pad1)
- R40 pad 2: Net-(C7-Pad1) -> SAW_OUT_S
- R41 pad 2: Net-(J2-Pad3) -> PULSE_OUT_S
- R42 pad 1: Net-(R42-Pad1) -> Net-(R40-Pad1)
- R42 pad 2: Net-(R41-Pad1) -> GND1
- R43 pad 1: Net-(R43-Pad1) -> Net-(R41-Pad1)
- R43 pad 2: Net-(R42-Pad1) -> GND1
- R44 pad 2: Net-(R43-Pad1) -> +12V
- R45 pad 1: Net-(R45-Pad1) -> Net-(C16-Pad2)
- R45 pad 2: Net-(R44-Pad1) -> +12V
- R46 pad 1: Net-(J2-Pad2) -> Net-(C17-Pad2)
- R46 pad 2: Net-(R45-Pad1) -> +12V
- R47 pad 1: Net-(R47-Pad1) -> Net-(R44-Pad1)
- R47 pad 2: Net-(J2-Pad2) -> GND1
- R48 pad 1: Net-(J2-Pad1) -> Net-(C16-Pad2)
- R48 pad 2: Net-(R47-Pad1) -> GND1
- R5 pad 1: CV_NODE -> Net-(R10-Pad2)
- R6 pad 1: CV_NODE -> Net-(R10-Pad2)
- R7 pad 1: CV_NODE -> Net-(R10-Pad2)
- R8 pad 1: LIN_FM -> Net-(R8-Pad1)
- R8 pad 2: Net-(C2-Pad1) -> V_OCT2
- RV10 pad 1: GND -> Net-(R58-Pad2)
- RV10 pad 2: /SIN_AMP -> /Panel components and power/VREF
- RV10 pad 3: Net-(R37-Pad2) -> Net-(R57-Pad1)
- RV11 pad 2: +8V_REF -> SIN_S_W
- RV11 pad 3: Net-(R49-Pad1) -> SIN_S_CCW
- RV6 pad 3: +12V -> +8V_REF
- RV7 pad 2: Net-(C2-Pad2) -> /LIN_FM_CV
- RV8 pad 1: Net-(R2-Pad1) (its old number) -> -12V_P
- RV8 pad 3: Net-(R1-Pad2) -> +12V_P
- SW1 pad 1: Net-(J2-Pad1) -> HARD_SYNC
- SW1 pad 2: Net-(R47-Pad1) -> Net-(C2-Pad1)
- SW1 pad 3: Net-(J2-Pad2) -> SOFT_SYNC
- SW2 pad 1: SOFT_SYNC -> /Panel components and power/0V
- SW2 pad 2: Net-(C8-Pad1) -> Net-(R33-Pad1)
- SW2 pad 3: HARD_SYNC -> Net-(R32-Pad1)
- U1 pad 4: -12V -> +12V_P
- U1 pad 5: Net-(R6-Pad1) -> GND
- U1 pad 6: Net-(R9-Pad2) -> Net-(R10-Pad2)
- U1 pad 7: PWM_IN -> Net-(R10-Pad1)
- U1 pad 8: +12V -> LINK_OUT_CV
- U2 pad 16: +12V -> +12V_P
- U3 pad 1: Net-(C6-Pad1) -> Net-(R18-Pad2)
- U3 pad 2: Net-(C6-Pad2) -> Net-(R21-Pad1)
- U3 pad 3: Net-(R22-Pad1) -> GND
- U3 pad 4: +12V -> -12V_P
- U3 pad 5: Net-(R23-Pad1) -> GND
- U3 pad 6: Net-(C7-Pad2) -> Net-(R18-Pad1)
- U3 pad 7: Net-(C7-Pad1) -> LINK_OUT_PW
- U3 pad 8: TRI_RAW -> +12V_P
- U4 pad 1: (no net) -> /Panel components and power/VREF
- U4 pad 2: Net-(R49-Pad1) -> GND
- U4 pad 3: GND -> +8V_REF
- U5 pad 2: -12V -> -12V_P
Routing:
- net -12V_P: track 0.00 -> 82.0 mm
- net +12V_P: track 0.00 -> 72.8 mm
- net -5V: track 0.00 -> 37.0 mm
- added copper zone on B.Cu, net GND
- added copper zone on F.Cu, net GND
- added copper zone on B.Cu, net GND1
- added copper zone on F.Cu, net GND1
Other:
- board outline added: 214 x 172 mm
- net class Power added: clearance 0.2, trace_width 0.75, via_dia 0.8, via_drill 0.4

Commit message: More layout work
Parts:
- added J21: Conn_01x03, Connector_PinHeader_2.54mm:PinHeader_1x03_P2.54mm_Vertical, B.Cu at (172.7, 38.1)
- added J22: Conn_01x03, Connector_PinSocket_2.54mm:PinSocket_1x03_P2.54mm_Vertical, F.Cu at (292.7, 38.1)
- C11, C12, C14, C15, C16, C17, D1, D2, D4, D5, J1, J5, Q1, Q2, R35, R36, R37, R38, R39, R40, R41, R42, R43, R44, R45, R46, R47, R48, R49, R50, R51, R52, R53, R54, R55, U6: moved to B.Cu
- J10, J11, J12, J13, J14, J15, J6, J7, J8, J9: footprint ao_tht:Jack_6.35mm_PJ_629HAN -> ao_tht:Jack_6.35mm_PJ_629HAN_slots
- RV2, RV3, RV7, RV8, RV9: footprint ao_tht:Potentiometer_Alpha_RD901F-40-00D_Single_Vertical_CircularHoles_centered -> ao_tht:Potentiometer_Alpha_RD901F-40-00D_Single_Vertical_centered
- TP1: moved to F.Cu
- moved J16 328.9 mm to (166.6, 216.7)
- moved R27 328.9 mm to (203.6, 182.9)
- moved R28 328.9 mm to (190.3, 191.0)
- moved R29 328.9 mm to (190.3, 195.0)
- moved R30 328.9 mm to (190.3, 186.9)
- moved R31 328.9 mm to (190.3, 199.1)
- moved R32 328.9 mm to (203.6, 178.8)
- moved R33 328.9 mm to (190.3, 182.9)
- moved R34 328.9 mm to (190.3, 178.8)
- moved SW2 328.9 mm to (174.8, 190.8)
- moved C12 151.4 mm to (310.4, 48.3)
- moved C11 150.2 mm to (312.4, 38.1), turned to 180 degrees
- moved R54 117.4 mm to (304.8, 124.5)
- moved C16 115.5 mm to (312.4, 120.7)
- moved C17 102.3 mm to (312.4, 74.9)
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Connections:
- net Net-(D1-Pad2) renamed /Panel components and power/+12V_IN
- net Net-(D2-Pad1) renamed /Panel components and power/-12V_IN
- J1 pad 4: LINK_OUT_FM_L -> LINK_OUT_CV_L
- J1 pad 8: LINK_OUT_CV_L -> LINK_OUT_FM_L
- J11 pad T: SIN_J -> SIN
- J12 pad T: TRI_J -> TRI
- J13 pad T: PULSE_J -> PULSE
- J14 pad T: SAW_J -> SAW
Routing:
- net +12V: track 0.00 -> 101.2 mm
- net -12V: track 0.00 -> 84.2 mm
- net -12V_P: track 82.0 -> 103.9 mm
- net +12V_P: track 72.8 -> 94.4 mm
- net /Panel components and power/-12V_IN: track 0.00 -> 10.2 mm
- net /Panel components and power/+12V_IN: track 0.00 -> 10.2 mm
- net -5V: track 37.0 -> 40.0 mm
Other:
- outline, holes or cut-outs redrawn

Commit message: Replace tri to sine, more layout
Parts:
- removed D4, D5: 1N4148, Diode_THT:D_DO-35_SOD27_P7.62mm_Horizontal
- added J23: Conn_01x07, Connector_PinHeader_2.54mm:PinHeader_1x07_P2.54mm_Vertical, B.Cu at (217.2, 143.5)
- added J24: Conn_01x07, Connector_PinSocket_2.54mm:PinSocket_1x07_P2.54mm_Vertical, F.Cu at (337.2, 143.5)
- added R59: 10k, ao_tht:R_Axial_DIN0207_L6.3mm_D2.5mm_P10.16mm_Horizontal, B.Cu at (326.4, 61.0)
- added R60: 18k, ao_tht:R_Axial_DIN0207_L6.3mm_D2.5mm_P10.16mm_Horizontal, B.Cu at (326.4, 73.7)
- added R61: 2.2k, ao_tht:R_Axial_DIN0207_L6.3mm_D2.5mm_P10.16mm_Horizontal, B.Cu at (336.6, 57.1)
- added R62: 20k, ao_tht:R_Axial_DIN0207_L6.3mm_D2.5mm_P10.16mm_Horizontal, B.Cu at (326.4, 90.2)
- added R63: 20k, ao_tht:R_Axial_DIN0207_L6.3mm_D2.5mm_P10.16mm_Horizontal, B.Cu at (336.6, 94.0)
- added RV4: 50k, ao_tht:Potentiometer_Bourns_3296W_Vertical_screw_centered, F.Cu at (224.0, 115.0)
- J2: value Conn_01x11 -> Conn_01x06; footprint Connector_PinHeader_2.54mm:PinHeader_1x11_P2.54mm_Vertical -> Connector_PinHeader_2.54mm:PinHeader_1x06_P2.54mm_Vertical
- J4: value Conn_01x11 -> Conn_01x06; footprint Connector_PinSocket_2.54mm:PinSocket_1x11_P2.54mm_Vertical -> Connector_PinSocket_2.54mm:PinSocket_1x06_P2.54mm_Vertical
- Q1: value MMBFJ201 -> 2N3904; footprint ao_tht:SOT-23_Handsoldering -> ao_tht:TO-92_Inline_Wide
- Q2: value J201 -> 2N3904
- R27, R28, R29, R30, R31, R32, R33, R34: value 10k -> 10k 1/8W
- R35: value 1M -> 30k
- R36: value 1M -> 2.2k
- R37: value 1k -> 10k
- R38: value 1k -> 390R
- R39: value 1k -> 2k
- RV11: value 10k -> 50k
- RV12: value 10k -> 5k
- moved J21 98.5 mm to (184.2, 135.9), turned to 0 degrees
- moved J22 98.4 mm to (303.5, 135.9), turned to 180 degrees
- moved R9 60.2 mm to (148.6, 114.3), turned to 0 degrees
- moved R47 57.2 mm to (298.4, 55.9)
- moved R44 57.2 mm to (298.4, 59.7)
- moved R20 49.1 mm to (176.5, 55.9), turned to 0 degrees
- moved R53 44.7 mm to (298.4, 63.5), turned to 0 degrees
- moved R11 40.2 mm to (158.8, 110.5), turned to 180 degrees
- moved R50 34.7 mm to (298.4, 67.3)
- moved J4 30.3 mm to (311.8, 143.5)
- moved J2 30.3 mm to (191.8, 143.5)
- moved R38 23.3 mm to (326.4, 69.8), turned to 0 degrees
- moved RV13 20.0 mm to (224.0, 75.0)
- moved R35 17.7 mm to (336.6, 53.3)
- moved C12 13.1 mm to (320.0, 39.4)
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Connections:
- J2 pad 1: GND -> V_OCT
- J2 pad 2: V_OCT -> V_OCT2
- J2 pad 3: V_OCT2 -> LIN_FM_IN
- J2 pad 4: CV_IN -> SYNC
- J2 pad 5: SYNC -> CV_IN
- J2 pad 6: LIN_FM_IN -> PWMIN
- J4 pad 1: GND1 -> V_OCT_J
- J4 pad 2: V_OCT_J -> V_OCT2_J
- J4 pad 3: V_OCT2_J -> LIN_FM_IN_J
- J4 pad 4: CV_IN_J -> SYNC_J
- J4 pad 5: SYNC_J -> CV_IN_J
- J4 pad 6: LIN_FM_IN_J -> PWMIN_J
- Q1 pad 1: Net-(Q1-Pad1) -> SIN_S_CCW_S
- Q1 pad 2: Net-(Q1-Pad2) -> SIN_R_CCW_S
- Q1 pad 3: Net-(D4-Pad2) -> Net-(Q1-Pad3)
- Q2 pad 1: Net-(Q1-Pad1) -> SIN_S_CW_S
- Q2 pad 2: Net-(Q1-Pad2) -> Net-(Q2-Pad2)
- Q2 pad 3: Net-(D4-Pad2) -> Net-(Q2-Pad3)
- R35 pad 1: SIN_S_W_S -> SIN_R_W_S
- R35 pad 2: Net-(D4-Pad2) -> TRI_RAW
- R36 pad 1: Net-(D4-Pad2) -> SIN_R_CCW_S
- R37 pad 1: SIN_S_W_S -> +12V
- R37 pad 2: Net-(Q1-Pad1) -> Net-(Q1-Pad3)
- R38 pad 1: Net-(Q1-Pad2) -> SIN_S_CW_S
- R38 pad 2: GND1 -> SIN_S_CCW_S
- R39 pad 2: SIN_A_CCW_S -> Net-(R39-Pad2)
- R50 pad 1: SIN_S_CCW_S -> TRI_RAW
- R53 pad 2: SIN_S_CCW_S -> TRI_RAW
- RV11 pad 1: GND -> SIN_R_CCW
- RV11 pad 2: SIN_S_W -> SIN_R_W
- RV11 pad 3: SIN_S_CCW -> SIN_R_W
- RV12 pad 3: SIN_A_CCW -> SIN_A_W
- U6 pad 12: Net-(Q1-Pad2) -> Net-(Q2-Pad3)
- U6 pad 13: SIN_A_W_S -> Net-(Q1-Pad3)
- U6 pad 14: SIN_A_CCW_S -> Net-(R39-Pad2)
- U6 pad 8: SIN_S_CCW_S -> TRI_RAW
Routing:
- net -12V: track 84.2 -> 112.9 mm
- net +12V: track 101.2 -> 116.8 mm
- net +12V_P: track 94.4 -> 102.6 mm
- net -12V_P: track 103.9 -> 99.7 mm
- net -5V: track 40.0 -> 38.7 mm

Commit message: More layout work
Parts:
- moved R27 166.4 mm to (140.6, 28.9)
- moved R28 166.4 mm to (127.3, 37.0)
- moved R29 166.4 mm to (127.3, 41.0)
- moved R30 166.4 mm to (127.3, 32.9)
- moved R31 166.4 mm to (127.3, 45.1)
- moved R32 166.4 mm to (140.6, 24.8)
- moved R33 166.4 mm to (127.3, 28.9)
- moved R34 166.4 mm to (127.3, 24.8)
- moved J16 164.5 mm to (131.5, 56.0)
- moved SW2 142.1 mm to (155.0, 50.0)
- moved J5 96.9 mm to (327.7, 141.0)
- moved D2 86.7 mm to (321.3, 130.8), turned to 90 degrees
- moved D1 86.4 mm to (316.2, 120.7), turned to 270 degrees
- moved C12 74.9 mm to (319.3, 114.3)
- moved C11 74.9 mm to (315.0, 114.3)
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Routing:
- net +12V: track 116.8 -> 51.8 mm
- net -12V: track 112.9 -> 51.9 mm
- net /Panel components and power/+12V_IN: track 10.2 -> 15.4 mm
- net /Panel components and power/-12V_IN: track 10.2 -> 15.3 mm
- net -5V: track 38.7 -> 35.8 mm
- net -12V_P: track 99.7 -> 98.9 mm
Other:
- outline, holes or cut-outs redrawn

Commit message: Fix label
Parts:
- moved R47 30.5 mm to (327.7, 68.6)
- moved R44 30.5 mm to (327.7, 64.8)
- moved R38 19.1 mm to (327.7, 88.9)
- moved Q1 19.1 mm to (337.8, 97.8)
- moved R39 19.1 mm to (337.8, 120.7)
- moved R35 19.1 mm to (337.8, 80.0)
- moved R61 19.1 mm to (337.8, 76.2)
- moved R37 19.1 mm to (327.7, 105.4)
- moved R59 19.1 mm to (327.7, 72.4)
- moved R60 19.1 mm to (327.7, 92.7)
- moved R63 19.1 mm to (327.7, 113.0)
- moved Q2 19.1 mm to (337.8, 85.1)
- moved R36 19.1 mm to (337.8, 101.6)
- moved R62 19.1 mm to (337.8, 109.2)
Connections:
- RV4 pad 3: SIN_S_CCW -> SIN_S_CW
Routing:
- net -12V_P: track 98.9 -> 99.7 mm

Commit message: Revise power ports
Connections:
- C10 pad 2: -12V_P -> -12V
- C11 pad 1: +12V -> +12V_1
- C12 pad 2: -12V -> -12V_1
- C14 pad 1: +12V -> +12V_1
- C15 pad 2: -12V -> -12V_1
- C3 pad 1: +12V_P -> +12V
- C6 pad 1: +12V_P -> +12V
- C7 pad 2: -12V_P -> -12V
- C9 pad 1: +12V_P -> +12V
- D1 pad 1: +12V -> +12V_1
- D2 pad 2: -12V -> -12V_1
- D3 pad 2: -12V_P -> -12V
- J21 pad 2: +12V_P -> +12V
- J21 pad 3: -12V_P -> -12V
- J22 pad 2: +12V -> +12V_1
- J22 pad 3: -12V -> -12V_1
- R13 pad 1: +12V_P -> +12V
- R19 pad 2: +12V_P -> +12V
- R26 pad 2: +12V_P -> +12V
- R37 pad 1: +12V -> +12V_1
- R44 pad 2: +12V -> +12V_1
- R45 pad 2: +12V -> +12V_1
- R46 pad 2: +12V -> +12V_1
- R59 pad 1: +12V -> +12V_1
- R60 pad 1: -12V -> -12V_1
- R8 pad 1: Net-(R8-Pad1) -> Net-(R10-Pad2)
- RV8 pad 1: -12V_P -> -12V
- RV8 pad 3: +12V_P -> +12V
- U1 pad 11: -12V_P -> -12V
- U1 pad 4: +12V_P -> +12V
- U2 pad 16: +12V_P -> +12V
- U3 pad 4: -12V_P -> -12V
- U3 pad 8: +12V_P -> +12V
- U5 pad 2: -12V_P -> -12V
- U6 pad 11: -12V -> -12V_1
- U6 pad 4: +12V -> +12V_1
Routing:
- net +12V_P: track 102.6 -> 0.00 mm
- net -12V_P: track 99.7 -> 0.00 mm
- net -12V_1: track 0.00 -> 51.9 mm
- net +12V_1: track 0.00 -> 51.8 mm
- net +12V: track 51.8 -> 102.6 mm
- net -12V: track 51.9 -> 99.7 mm
