File: Hardware/PCB_back/herovco_back/herovco_back.kicad_pcb (KiCad board)
At the start: 2 copper layers, 94 x 156 mm, 55 parts, among them J201 Conn_01x06, J202 Conn_01x09, J203 Conn_01x07, J204 Conn_02x04_Odd_Even, J205 AudioJack2, J206 AudioJack2, J207 AudioJack2, J208 AudioJack2, J209 AudioJack2, J210 Synth_power_2x5, J211 AudioJack2, J212 AudioJack2, J213 AudioJack2, J214 AudioJack2, J215 AudioJack2, Q201 2N3904, Q202 2N3904, U201 TL074

Commit message: First routing
Parts:
- added GRAF201: Holes, herovco_panel:3340vco_panel_holes, F.Cu at (254.0, 24.2)
- added GRAF202: AO logo, ao_tht:analogoutput, B.Cu at (162.0, 51.0)
- added GRAF203: CC0 logo, ao_tht:CC0_logo, B.Cu at (157.0, 34.0)
- C203, C204: value 180pF -> 330pF
- R215, R216, R217: value 43k -> 24k
- R218, R219, R220: value 16k -> 9.1k
- R221, R222, R223: value 18k -> 10k
- moved J202 20.6 mm to (156.8, 108.3)
- moved J203 20.6 mm to (182.2, 108.3)
- moved C204 20.6 mm to (148.5, 54.9)
- moved R201 20.6 mm to (182.8, 60.0)
- moved R226 20.6 mm to (151.1, 51.1)
- moved C201 20.6 mm to (151.1, 77.8)
- moved C202 20.6 mm to (173.9, 77.8)
- moved C203 20.6 mm to (148.5, 100.7)
- moved C205 20.6 mm to (160.0, 94.3)
- moved C206 20.6 mm to (164.3, 94.3)
- moved D201 20.6 mm to (161.2, 100.7)
- moved D202 20.6 mm to (166.3, 110.8)
- moved H201 20.6 mm to (138.0, 28.0)
- moved H202 20.6 mm to (101.0, 92.0)
- moved H203 20.6 mm to (189.0, 131.0)
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Connections:
- J201 pad 2: SAW_OUT_S -> PULSE_OUT_S
- J201 pad 3: PULSE_OUT_S -> SAW_OUT_S
Routing:
- net TRI: track 0.00 -> 134.4 mm
- net PULSE: track 0.00 -> 131.8 mm
- net +12V_1: track 49.7 -> 152.8 mm
- net SIN: track 0.00 -> 102.5 mm
- net SIN_S_CW_S: track 0.00 -> 70.9 mm
- net Net-(R215-Pad1): track 0.00 -> 67.7 mm
- net SIN_R_W_S: track 0.00 -> 66.6 mm
- net SAW: track 0.00 -> 65.8 mm
- net V_OCT_J: track 0.00 -> 55.2 mm
- net SYNC_J: track 0.00 -> 52.8 mm
- net Net-(Q202-Pad3): track 0.00 -> 52.7 mm
- net TRI_RAW: track 0.00 -> 52.1 mm
- net SIN_S_CCW_S: track 0.00 -> 49.9 mm
- net SIN_S_W_S: track 0.00 -> 48.0 mm
- net TRIANGLE_OUT_S: track 0.00 -> 47.2 mm
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Other:
- board text added: "Rich Holmes CC0 1.0 Nov 2021 https://github.com/holmesrichards/hero"
- board text removed: "Rich Holmes CC0 1.0 ??/202? https://github.com/holmesrichards/hero"

Commit message: PCB labels
Parts:
- moved C201 2.54 mm to (153.6, 77.8)
Routing:
- net Net-(R215-Pad1): track 67.7 -> 64.1 mm
- net +12V_1: track 152.8 -> 154.6 mm
Other:
- board text added: "FM CV"
- board text added: "PW CV"
- board text added: "Pitch CV"
- board text added: "RED STRIPE"
- board text added: "Saw"
