File: Hardware/PCB_front/herovco_front/herovco_front.kicad_pcb (KiCad board)
At the start: 2 copper layers, 94 x 125 mm, 80 parts, among them J101 3_pin_Molex_header, J102 Conn_01x06, J103 Conn_01x09, J104 Conn_01x07, J105 3_pin_Molex_connector, SW101 SW_SPDT_MSM, SW102 SW_Rotary12, U101 TL074, U102 AS3340A, U103 TL072, U104 TL431LP, U105 L79L05_TO92

Commit message: Change regulator output cap and rearrange
Parts:
- C101: footprint ao_tht:C_Rect_L7.2mm_W2.5mm_P5.00mm_FKS2_FKP2_MKS2_MKP2 -> ao_tht:C_Disc_D3.0mm_W1.6mm_P2.50mm
- C111: value 1uF -> 10nF; footprint ao_tht:CP_Radial_D5.0mm_P2.00mm -> ao_tht:C_Disc_D3.0mm_W1.6mm_P2.50mm; moved to B.Cu
- D101, U105: moved to B.Cu
- moved U105 11.7 mm to (179.1, 43.2), turned to 0 degrees
- moved R120 10.2 mm to (197.0, 36.0), turned to 0 degrees
- moved R121 10.2 mm to (214.0, 39.0), turned to 0 degrees
- moved R122 10.2 mm to (197.0, 40.0), turned to 0 degrees
- moved D101 7.62 mm to (186.7, 48.3), turned to 180 degrees
- moved C111 2.82 mm to (181.7, 39.4)
Connections:
- R120 pad 1: Net-(R120-Pad1) -> +8V_REF
- R120 pad 2: +8V_REF -> Net-(R120-Pad2)
- R121 pad 1: GND -> Net-(R121-Pad1)
- R121 pad 2: Net-(R121-Pad2) -> GND
- R122 pad 1: +8V_REF -> +12V
- R122 pad 2: +12V -> +8V_REF
- RV107 pad 1: Net-(R121-Pad2) -> Net-(R121-Pad1)
- RV107 pad 3: Net-(R120-Pad1) -> Net-(R120-Pad2)
Routing:
- net -5V: track 35.8 -> 28.1 mm
- net -12V: track 102.9 -> 105.2 mm

Commit message: First routing
Parts:
- moved R104 10.2 mm to (207.2, 59.0), turned to 180 degrees
- moved C101 10.0 mm to (197.0, 63.0), turned to 0 degrees
- moved R108 7.62 mm to (158.8, 114.3)
- moved R110 3.81 mm to (148.6, 110.5)
- moved R112 3.81 mm to (158.8, 106.7)
Connections:
- J102 pad 2: SAW_OUT -> PULSE_OUT
- J102 pad 3: PULSE_OUT -> SAW_OUT
Routing:
- net +8V_REF: track 0.00 -> 158.9 mm
- net HARD_SYNC: track 0.00 -> 122.8 mm
- net CV_NODE: track 0.00 -> 86.9 mm
- net Net-(R125-Pad2): track 0.00 -> 69.1 mm
- net SOFT_SYNC: track 0.00 -> 61.9 mm
- net Net-(R105-Pad1): track 0.00 -> 61.4 mm
- net PULSE_OUT: track 0.00 -> 60.6 mm
- net LINK_OUT_FM: track 0.00 -> 59.0 mm, vias 0 -> 1
- net Net-(R127-Pad1): track 0.00 -> 57.7 mm, vias 0 -> 1
- net PWMIN: track 0.00 -> 55.8 mm
- net +12V: track 106.7 -> 157.8 mm
- net SIN_R_W: track 0.00 -> 50.2 mm
- net OCTAVE: track 0.00 -> 49.5 mm, vias 0 -> 1
- net /PULSE_WIDTH: track 0.00 -> 47.9 mm
- net Net-(R110-Pad1): track 0.00 -> 46.0 mm
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
Commit message: Panel in KiCad
Parts:
- GRAF101: footprint herovco_panel:3340vco_panel_holes -> herovco_panel:herovco_panel_holes

Commit message: PCB labels
Parts:
- D102: footprint Diode_THT:D_DO-41_SOD81_P10.16mm_Horizontal -> ao_tht:D_DO-41_SOD81_P10.16mm_Horizontal
- moved C101 6.02 mm to (191.0, 63.0)
Routing:
- net -5V: track 68.4 -> 72.1 mm
