File: Hardware/PCB/herovco/herovco.kicad_pcb (KiCad board)
At the start: 2 copper layers, 219 x 172 mm, 140 parts, among them J1 Conn_01x09, J10 AudioJack2, J11 AudioJack2, J12 AudioJack2, J13 AudioJack2, J14 AudioJack2, J15 Synth_power_2x5, J16 AudioJack2, J17 AudioJack2, J18 AudioJack2, J19 AudioJack2, J2 Conn_01x07, J20 AudioJack2, J3 Conn_01x06, J4 3_pin_Molex_header, J5 Conn_01x09, J6 Conn_01x07, J7 Conn_01x06, J8 3_pin_Molex_connector, J9 Conn_02x04_Odd_Even, Q1 2N3904, Q2 2N3904, SW1 SW_Rotary12, SW2 SW_SPDT_MSM, U1 TL074, U2 AS3340A, U3 TL072, U4 TL431LP, U5 L79L05_TO92, U6 TL074

Commit message: Test points
Parts:
- added TP2: +12V, ao_tht:TestPoint_THTPad_D1.5mm_Drill0.7mm, F.Cu at (224.8, 138.4)
- added TP3: -12V, ao_tht:TestPoint_THTPad_D1.5mm_Drill0.7mm, F.Cu at (224.8, 142.2)
- added TP4: GND, ao_tht:TestPoint_THTPad_1.5x1.5mm_Drill0.7mm, F.Cu at (224.8, 134.6)
- added TP5: +12V, ao_tht:TestPoint_THTPad_D1.5mm_Drill0.7mm, F.Cu at (349.8, 132.1)
- added TP6: -12V, ao_tht:TestPoint_THTPad_D1.5mm_Drill0.7mm, F.Cu at (349.8, 135.9)
- added TP7: GND, ao_tht:TestPoint_THTPad_1.5x1.5mm_Drill0.7mm, F.Cu at (349.8, 128.3)
- moved C11 26.4 mm to (181.7, 39.4), turned to 0 degrees
Routing:
- net +12V: track 157.8 -> 208.4 mm
- net -12V: track 126.4 -> 172.2 mm
- net +12V_1: track 154.6 -> 184.5 mm
- net -12V_1: track 49.6 -> 79.4 mm
- net PULSE: track 131.8 -> 134.2 mm, vias 0 -> 1
- net /Front PCB/LIN_FM_CV: track 27.6 -> 28.9 mm
- net /Front PCB/V_OCT2: track 41.5 -> 42.5 mm
- net /Front PCB/V_OCT: track 42.1 -> 43.1 mm
- net /Outputs and sin/SIN_S_CW_S: track 70.9 -> 70.3 mm

Commit message: Version 6 (PCB)
Other:
- net class Default removed
- net class Power removed

Commit message: Pre-breadboard updates
Parts:
- C16, C17: footprint ao_tht:CP_Radial_D5.0mm_P2.00mm -> ao_tht:CP_Radial_D6.3mm_P2.50mm
- C2, C6, C7, C8: footprint ao_tht:C_Rect_L7.2mm_W2.5mm_P5.00mm_FKS2_FKP2_MKS2_MKP2 -> ao_tht:C_Disc_D3.0mm_W1.6mm_P2.50mm
- D2: footprint ao_tht:D_DO-41_SOD81_P10.16mm_Horizontal -> Diode_THT:D_DO-41_SOD81_P10.16mm_Horizontal
- U4, U5: footprint ao_tht:TO-92_Inline_Wide -> Package_TO_SOT_THT:TO-92_Inline
Connections:
- net /Front PCB/LINK_OUT_CV renamed /Front PCB/CV_SUM
- SW1 pad 10: Net-(SW1-Pad10) -> unconnected-(SW1-Pad10)
- SW1 pad 11: Net-(SW1-Pad11) -> unconnected-(SW1-Pad11)
- SW1 pad 12: Net-(SW1-Pad12) -> unconnected-(SW1-Pad12)
Routing:
- net /Front PCB/V_OCT2: track 42.5 -> 45.0 mm
- net /Front PCB/SYNC: track 24.5 -> 27.0 mm
- net -5V: track 72.1 -> 74.2 mm
- net /Front PCB/+8V_REF: track 158.9 -> 156.9 mm
- net -12V: track 172.2 -> 170.2 mm
- net /Front PCB/PULSE_OUT: track 60.6 -> 62.1 mm
- net /Front PCB/TRIANGLE_OUT: track 41.8 -> 43.3 mm
- net /Front PCB/SAW_OUT: track 40.7 -> 42.1 mm
- net /Front PCB/LINK_OUT_FM: track 59.0 -> 60.1 mm
- net /Front PCB/V_OCT: track 43.1 -> 43.7 mm

Commit message: rm Zener, change adj ref to fixed and modify octave switch and fine tune accordingly
Parts:
- added C18: 10nF, ao_tht:C_Disc_D3.0mm_W1.6mm_P2.50mm, B.Cu at (193.5, 59.2)
- added R64: 470R, ao_tht:R_Axial_DIN0207_L6.3mm_D2.5mm_P10.16mm_Horizontal, B.Cu at (207.2, 59.0)
- D3, D4: footprint Diode_THT:D_DO-41_SOD81_P10.16mm_Horizontal -> ao_tht:D_DO-41_SOD81_P10.16mm_Horizontal
- J10, J11, J12, J13, J14, J16, J17, J18, J19, J20: footprint ao_tht:Jack_6.35mm_PJ_629HAN_slots -> ao_tht:Jack_6.35mm_PJ_629HAN
- R9: value 3M -> 10M
- moved TP5 11.4 mm to (350.4, 120.7)
- moved R12 3.97 mm to (207.2, 63.0)
- moved TP6 0.65 mm to (350.4, 135.9)
- moved TP7 0.65 mm to (350.4, 128.3)
- turned J8 to 0 degrees
Connections:
- C6 pad 1: Net-(C6-Pad1) -> GND
- C6 pad 2: GND -> Net-(U2-Pad11)
- J4 pad 1: /Front PCB/OCTAVE -> GND
- J4 pad 2: /Front PCB/+8V_REF -> /Front PCB/OCTAVE
- J4 pad 3: GND -> /Front PCB/+8V_REF
- J8 pad 1: /Octave switch/OCTAVE_P -> /Octave switch/0V
- J8 pad 2: /Octave switch/+8V_REF_P -> /Octave switch/OCTAVE_P
- J8 pad 3: /Octave switch/0V -> /Octave switch/+8V_REF_P
- U2 pad 11: Net-(C6-Pad1) -> Net-(U2-Pad11)
Routing:
- net Net-(U2-Pad11): track 0.00 -> 34.0 mm
- net Net-(C6-Pad1): track 31.5 -> 0.00 mm
- net +12V_1: track 184.5 -> 177.1 mm
- net -5V: track 74.2 -> 67.8 mm
- net /Octave switch/+8V_REF_P: track 25.4 -> 20.8 mm
- net Net-(C18-Pad1): track 0.00 -> 3.54 mm
- net /Jacks, power, etc/V_OCT_J: track 55.2 -> 57.9 mm
- net /Octave switch/OCTAVE_P: track 17.5 -> 20.0 mm
- net /Front PCB/OCTAVE: track 49.3 -> 51.8 mm
- net /Front PCB/+8V_REF: track 156.9 -> 154.3 mm
- net /Octave switch/0V: track 25.3 -> 23.2 mm
- net /Jacks, power, etc/SIN: track 102.5 -> 103.8 mm
- net Net-(R12-Pad1): track 21.8 -> 21.1 mm
- net -12V_1: track 79.4 -> 80.0 mm

Commit message: rm Zener, change adj ref to fixed, cont'd
Parts:
- removed D2: 1N4732A, Diode_THT:D_DO-41_SOD81_P10.16mm_Horizontal
- removed RV7: 10k, ao_tht:Potentiometer_Bourns_3296W_Vertical_screw_centered
- removed TP1: TestPoint, TestPoint:TestPoint_Pad_2.5x2.5mm
- R10: value 300k -> 200k
- R28: value 8.2k -> 10k 1/8W; moved to F.Cu
- R29: value 1k -> 10k 1/8W; moved to F.Cu
- RV1: value 100k -> 50k
- U4: value TL431LP -> LM4040LP-10; footprint Package_TO_SOT_THT:TO-92_Inline -> ao_tht:TO-92_Inline_Wide
- moved R29 96.8 mm to (119.9, 61.7), turned to -90 degrees
- moved R28 89.4 mm to (113.5, 68.1), turned to 180 degrees
- moved J8 19.1 mm to (97.0, 74.5)
- moved R8 0.58 mm to (96.5, 68.1)
Connections:
- J4 pad 3: /Front PCB/+8V_REF -> /Front PCB/+10V_REF
- J8 pad 3: /Octave switch/+8V_REF_P -> /Octave switch/+10V_REF_P
- R1 pad 2: /Octave switch/+8V_REF_P -> Net-(R1-Pad2)
- R10 pad 1: /Front PCB/+8V_REF -> /Front PCB/+10V_REF
- R28 pad 1: /Front PCB/+8V_REF -> Net-(SW1-Pad10)
- R28 pad 2: Net-(R28-Pad2) -> /Octave switch/+10V_REF_P
- R29 pad 1: Net-(R29-Pad1) -> Net-(R1-Pad2)
- R29 pad 2: GND -> Net-(SW1-Pad10)
- R30 pad 2: /Front PCB/+8V_REF -> /Front PCB/+10V_REF
- RV6 pad 3: /Front PCB/+8V_REF -> /Front PCB/+10V_REF
- SW1 pad 10: unconnected-(SW1-Pad10) -> Net-(SW1-Pad10)
- SW1 pad 11: unconnected-(SW1-Pad11) -> /Octave switch/+10V_REF_P
- SW1 pad 9: /Octave switch/+8V_REF_P -> Net-(R1-Pad2)
- U4 pad 1: /Front PCB/VREF -> (no net)
- U4 pad 2: GND -> /Front PCB/+10V_REF
- U4 pad 3: /Front PCB/+8V_REF -> GND
Routing:
- net /Front PCB/+8V_REF: track 154.3 -> 0.00 mm
- net /Front PCB/+10V_REF: track 0.00 -> 133.7 mm
- net /Front PCB/VREF: track 32.2 -> 0.00 mm
- net Net-(SW1-Pad10): track 0.00 -> 23.8 mm
- net /Octave switch/+10V_REF_P: track 0.00 -> 20.8 mm
- net /Octave switch/+8V_REF_P: track 20.8 -> 0.00 mm
- net Net-(R1-Pad2): track 0.00 -> 17.8 mm
- net Net-(R28-Pad2): track 14.1 -> 0.00 mm
- net Net-(R29-Pad1): track 11.0 -> 0.00 mm
- net /Octave switch/0V: track 23.2 -> 16.1 mm
- net /Octave switch/OCTAVE_P: track 20.0 -> 24.1 mm
- net Net-(R7-Pad1): track 15.4 -> 16.4 mm
