File: Hardware/PCB/herovco/herovco.kicad_pcb (KiCad board)
At the start: 2 copper layers, 219 x 172 mm, 145 parts, among them J1 Conn_01x09, J10 AudioJack2, J11 AudioJack2, J12 AudioJack2, J13 AudioJack2, J14 AudioJack2, J15 Synth_power_2x5, J16 AudioJack2, J17 AudioJack2, J18 AudioJack2, J19 AudioJack2, J2 Conn_01x07, J20 AudioJack2, J3 Conn_01x06, J4 3_pin_Molex_header, J5 Conn_01x09, J6 Conn_01x07, J7 Conn_01x06, J8 3_pin_Molex_connector, J9 Conn_02x04_Odd_Even, Q1 2N3904, Q2 2N3904, SW1 SW_Rotary12, SW2 SW_SPDT_MSM, U1 TL074, U2 AS3340A, U3 TL072, U4 LM4040LP-10, U5 L79L05_TO92, U6 TL074

Commit message: Panel updates; reannotate; correct PCB errors
Parts:
- moved R35 6.95 mm to (84.3, 41.4)
- moved R36 6.92 mm to (84.3, 55.4)
- moved R37 6.89 mm to (84.3, 69.3)
- moved R38 3.06 mm to (99.6, 68.1)
- moved J8 2.54 mm to (99.6, 74.5)
- moved R30 2.54 mm to (119.9, 59.2)
- moved R31 1.78 mm to (119.9, 45.2)
- moved SW2 1.35 mm to (102.1, 50.3)
- moved R29 1.27 mm to (114.8, 68.1)
- moved R32 1.26 mm to (119.9, 31.2)
- moved R34 1.10 mm to (89.4, 32.5)
- renumbered C9 to C10, C10 to C11, C11 to C12, C16 to C13, C17 to C14, C12 to C15, C13 to C16, C14 to C17, C15 to C18, C18 to C4, C4 to C5, C5 to C6, C6 to C7, C7 to C8, C8 to C9, D3 to D2, D4 to D3, R9 to R1, R18 to R10, R19 to R11, R64 to R12, R20 to R13, R21 to R14, R22 to R15, R23 to R16, R24 to R17, R25 to R18, R26 to R19, R10 to R2, R27 to R20, R30 to R21, R31 to R22, R32 to R23, R33 to R24, R34 to R25, R35 to R26, R36 to R27, R37 to R28, R28 to R29, R11 to R3, R29 to R30, R1 to R31, R2 to R32, R3 to R33, R4 to R34, R5 to R35, R6 to R36, R7 to R37, R8 to R38, R38 to R39, R12 to R4, R39 to R40, R40 to R41, R41 to R42, R42 to R43, R43 to R44, R44 to R45, R45 to R46, R46 to R47, R47 to R48, R48 to R49, R13 to R5, R49 to R50, R50 to R51, R51 to R52, R52 to R53, R53 to R54, R54 to R55, R55 to R56, R56 to R57, R57 to R58, R58 to R59, R14 to R6, R59 to R60, R60 to R61, R61 to R62, R62 to R63, R63 to R64, R15 to R7, R16 to R8, R17 to R9, RV9 to RV10, RV12 to RV11, RV13 to RV12, RV10 to RV7, RV11 to RV8, RV8 to RV9, SW2 to SW1, SW1 to SW2, TP2 to TP1, TP3 to TP2, TP4 to TP3, TP5 to TP4, TP6 to TP5, TP7 to TP6
Routing:
- net Net-(R30-Pad1): track 17.8 -> 14.7 mm
- net Net-(R34-Pad1): track 20.2 -> 17.6 mm
- net Net-(R29-Pad1): track 23.8 -> 21.3 mm
- net /Octave switch/0V: track 16.1 -> 13.6 mm
- net /Octave switch/+10V_REF_P: track 20.8 -> 18.5 mm
- net Net-(R36-Pad1): track 9.47 -> 11.8 mm
- net Net-(R35-Pad1): track 13.8 -> 11.8 mm
- net Net-(R33-Pad1): track 10.2 -> 12.2 mm
- net Net-(R32-Pad1): track 16.6 -> 18.4 mm
- net /Octave switch/OCTAVE_P: track 24.1 -> 22.6 mm
- net Net-(R37-Pad1): track 16.4 -> 17.5 mm
- net /Outputs and sin/SIN_S_CW_S: track 70.3 -> 70.9 mm

Commit message: Big panel and PCB revisions
Parts:
- removed the J7 at (283.8, 101.6)
- removed the SW1 at (142.5, 122.0)
- added C12: 100nF, ao_tht:C_Rect_L7.2mm_W2.5mm_P5.00mm_FKS2_FKP2_MKS2_MKP2, B.Cu at (144.8, 80.0)
- added D1: 1N4148, ao_tht:D_DO-35_SOD27_P7.62mm_Horizontal, B.Cu at (141.0, 72.4)
- added J10: Conn_01x03, Connector_PinSocket_2.54mm:PinSocket_1x03_P2.54mm_Vertical, F.Cu at (291.4, 95.2)
- added J12: 4_pin_Molex_connector, Connector_Molex:Molex_KK-254_AE-6410-04A_1x04_P2.54mm_Vertical, F.Cu at (99.1, 91.5)
- added J4: Conn_01x03, Connector_PinHeader_2.54mm:PinHeader_1x03_P2.54mm_Vertical, B.Cu at (166.4, 95.2)
- added J6: 4_pin_Molex_header, Connector_Molex:Molex_KK-254_AE-6410-04A_1x04_P2.54mm_Vertical, B.Cu at (137.2, 95.2)
- added J9: Conn_01x03, Connector_PinSocket_2.54mm:PinSocket_1x03_P2.54mm_Vertical, F.Cu at (319.3, 67.3)
- added R17: 5.6k, ao_tht:R_Axial_DIN0207_L6.3mm_D2.5mm_P10.16mm_Horizontal, B.Cu at (148.6, 68.6)
- added R18: 47k, ao_tht:R_Axial_DIN0207_L6.3mm_D2.5mm_P10.16mm_Horizontal, B.Cu at (176.5, 76.2)
- added R23: 10k, ao_tht:R_Axial_DIN0207_L6.3mm_D2.5mm_P10.16mm_Horizontal, B.Cu at (138.4, 76.2)
- added SW2: SW_DP3T, ao_tht:Heatsink_17x17mm_A-5093, F.Cu at (326.7, -31.3)
- C10: renamed from C8; footprint ao_tht:C_Disc_D3.0mm_W1.6mm_P2.50mm -> ao_tht:C_Rect_L7.2mm_W2.5mm_P5.00mm_FKS2_FKP2_MKS2_MKP2
- C11: renamed from C9; footprint ao_tht:C_Disc_D3.0mm_W1.6mm_P2.50mm -> ao_tht:C_Rect_L7.2mm_W2.5mm_P5.00mm_FKS2_FKP2_MKS2_MKP2
- C13: renamed from C12; footprint ao_tht:C_Disc_D3.0mm_W1.6mm_P2.50mm -> ao_tht:C_Rect_L7.2mm_W2.5mm_P5.00mm_FKS2_FKP2_MKS2_MKP2
- C7: renamed from C2; value 10nF -> 100nF; footprint ao_tht:C_Disc_D3.0mm_W1.6mm_P2.50mm -> ao_tht:C_Rect_L7.2mm_W2.5mm_P5.00mm_FKS2_FKP2_MKS2_MKP2
- C8: renamed from C4; footprint ao_tht:C_Disc_D3.0mm_W1.6mm_P2.50mm -> ao_tht:C_Rect_L7.2mm_W2.5mm_P5.00mm_FKS2_FKP2_MKS2_MKP2
- C9: renamed from C7; footprint ao_tht:C_Disc_D3.0mm_W1.6mm_P2.50mm -> Capacitor_THT:C_Rect_L7.2mm_W4.5mm_P5.00mm_FKS2_FKP2_MKS2_MKP2
- GRAF1: footprint herovco_panel:herovco_panel_holes -> herovco:herovco_panel_behind
- J3: value Conn_01x06 -> Conn_01x03; footprint Connector_PinHeader_2.54mm:PinHeader_1x06_P2.54mm_Vertical -> Connector_PinHeader_2.54mm:PinHeader_1x03_P2.54mm_Vertical
- R1: value 10M -> 1M
- moved R2 90.4 mm to (224.8, 44.5), turned to 180 degrees
- moved R10 60.3 mm to (208.3, 101.6), turned to 180 degrees
- moved C7 51.1 mm to (139.7, 83.8)
- moved R30 49.9 mm to (224.8, 68.6), turned to 180 degrees
- moved J3 49.4 mm to (194.3, 67.3), turned to 180 degrees
- moved R13 40.4 mm to (198.1, 97.8), turned to 0 degrees
- moved R25 34.6 mm to (198.1, 58.4)
- moved R27 34.4 mm to (208.3, 90.2)
- moved R31 34.4 mm to (198.1, 94.0)
- moved R62 32.2 mm to (342.9, 72.4)
- moved R65 32.2 mm to (332.7, 68.6)
- moved R12 30.8 mm to (176.5, 62.2)
- moved R22 30.6 mm to (176.5, 100.3)
- moved R29 26.4 mm to (208.3, 67.3)
- moved R26 25.9 mm to (198.1, 71.1)
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- renumbered C13 to C14, C14 to C15, C15 to C16, C16 to C17, C17 to C18, C18 to C19, C5 to C2, C6 to C3, C10 to C4, C11 to C5, C3 to C6, D1 to D2, D2 to D3, D3 to D4, J8 to J11, J9 to J13, J10 to J14, J11 to J15, J12 to J16, J13 to J17, J14 to J18, J15 to J19, J16 to J20, J17 to J21, J18 to J22, J19 to J23, J20 to J24, J4 to J5, J5 to J7, J6 to J8, R17 to R19, R18 to R20, R19 to R21, R20 to R22, R21 to R24, R22 to R25, R23 to R26, R24 to R27, R25 to R28, R26 to R29, R27 to R30, R28 to R31, R29 to R32, R30 to R33, R31 to R34, R32 to R35, R33 to R36, R34 to R37, R35 to R38, R36 to R39, R37 to R40, R38 to R41, R39 to R42, R40 to R43, R41 to R44, R42 to R45, R43 to R46, R44 to R47, R45 to R48, R46 to R49, R47 to R50, R48 to R51, R49 to R52, R50 to R53, R51 to R54, R52 to R55, R53 to R56, R54 to R57, R55 to R58, R56 to R59, R57 to R60, R58 to R61, R59 to R62, R60 to R63, R61 to R64, R62 to R65, R63 to R66, R64 to R67, SW2 to SW1, U3 to U2, U2 to U3
Connections:
- net /Octave switch/+10V_REF_P renamed /Octave and sync switches/+10V_REF_P
- net /Octave switch/0V renamed /Octave and sync switches/0V
- net /Octave switch/OCTAVE_P renamed /Octave and sync switches/OCTAVE_P
- C7 pad 1: Net-(C2-Pad1) -> /Front PCB/SYNCA
Routing:
- net Net-(R2-Pad2): track 22.8 -> 110.7 mm
- net HARD_SYNC: track 122.8 -> 43.3 mm
- net /Front PCB/SYNC: track 27.0 -> 87.9 mm
- net SOFT_SYNC: track 61.5 -> 7.17 mm
- net Net-(R56-Pad1): track 64.1 -> 24.2 mm
- net /Front PCB/SOFT_SYNCA: track 0.00 -> 36.7 mm
- net TRI: track 134.1 -> 170.7 mm
- net /Front PCB/SAW_OUT: track 42.1 -> 5.62 mm
- net /Front PCB/PULSE_OUT: track 62.1 -> 27.4 mm
- net /Front PCB/PULSE_WIDTH: track 47.9 -> 14.3 mm
- net /Outputs and sin/SAW_OUT_S: track 13.1 -> 44.8 mm
- net CV_NODE: track 86.9 -> 118.7 mm
- net Net-(R29-Pad1): track 57.7 -> 27.0 mm, vias 1 -> 0
- net /Front PCB/TRIANGLE_OUT: track 43.3 -> 13.1 mm
- net /Front PCB/V_OCT: track 43.7 -> 72.7 mm
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Other:
- outline, holes or cut-outs redrawn
- board text removed: "LINK HEADER If you are having trouble connecting a power cable here, that's because this is not a power header. HINT: Count the pins! Power header's over there."

Commit message: Sch cleanup, switch footprint
Parts:
- SW2: footprint ao_tht:Heatsink_17x17mm_A-5093 -> herovco:G-1128S_DP3T
- moved SW2 234.9 mm to (143.2, 115.4)
- moved J12 41.1 mm to (124.3, 123.8), turned to 90 degrees
- moved J13 6.35 mm to (292.0, 113.0)
Routing:
- net /Octave and sync switches/SOFT_SYNCA_P: track 0.00 -> 60.6 mm
- net /Octave and sync switches/SYNCA_P: track 0.00 -> 51.2 mm
- net /Octave and sync switches/SOFT_SYNC_OFF_P: track 0.00 -> 29.2 mm
- net /Octave and sync switches/HARD_SYNCA_P: track 0.00 -> 19.2 mm
- net LINK_OUT_PW_L: track 20.8 -> 14.5 mm
- net LINK_OUT_CV_L: track 18.4 -> 12.0 mm
- net LINK_OUT_FM_L: track 22.7 -> 16.9 mm
- net /Outputs and sin/LINK_OUT_SAW: track 43.7 -> 44.2 mm
