File: Hardware/PCB/herovco/herovco.kicad_pcb (KiCad board)
At the start: 2 copper layers, 269 x 172 mm, 163 parts, among them J1 Conn_01x09, J10 Conn_01x03, J11 Conn_01x03, J12 3_pin_Molex_connector, J13 Wire pads, J14 Conn_01x01, J15 Conn_01x01, J16 Conn_01x01, J17 Conn_02x04_Odd_Even, J18 AudioJack2, J19 AudioJack2, J2 Conn_01x03, J20 AudioJack2, J21 AudioJack2, J22 AudioJack2, J23 Synth_power_2x5, J24 AudioJack2, J25 AudioJack2, J26 AudioJack2, J27 AudioJack2, J28 AudioJack2, J3 Conn_01x03, J4 3_pin_Molex_header, J5 Wire pads, J6 Conn_01x01, J7 Conn_01x01, J8 Conn_01x01, J9 Conn_01x09, Q1 2N3904, Q2 2N3904, SW1 SW_Rotary12, SW2 SW_DP3T, U1 TL074, U2 TL072, U3 AS3340A, U4 LM4040BIZ-5, U5 LM4040BIZ-5, U6 L79L05_TO92, U7 TL074

Commit message: schem tweaks
Parts:
- removed J12: 3_pin_Molex_connector, ao_tht:Molex_KK-254_AE-6410-03A_1x03_P2.54mm_Vertical
- removed R32, R33, R34, R35, R36, R37, R38, R39, R40, R41: 10k 1/8W, ao_tht:R_Axial_DIN0207_L6.3mm_D2.5mm_P10.16mm_Horizontal
- removed SW1: SW_Rotary12, ao_tht:Rotary_Switch
Routing:
- net /Octave and sync switches/OCTAVE_P: track 22.6 -> 0.00 mm
- net Net-(R32-Pad1): track 21.3 -> 0.00 mm
- net /Octave and sync switches/+5V_REF_P: track 18.5 -> 0.00 mm
- net Net-(R35-Pad1): track 18.4 -> 0.00 mm
- net Net-(R37-Pad1): track 17.6 -> 0.00 mm
- net Net-(R40-Pad1): track 17.5 -> 0.00 mm
- net Net-(R34-Pad1): track 14.2 -> 0.00 mm
- net Net-(R33-Pad1): track 13.8 -> 0.00 mm
- net /Octave and sync switches/-5V_REF_P: track 13.1 -> 0.00 mm
- net Net-(R39-Pad1): track 11.8 -> 0.00 mm
- net Net-(R38-Pad1): track 11.8 -> 0.00 mm
- net Net-(R36-Pad1): track 11.7 -> 0.00 mm
Other:
- board text removed: "Panel mounted"

Commit message: Convert jack footprints to slotted; clean up silkscreen; add silkscreen notes to match resistors
Parts:
- J18, J19, J20, J21, J22, J24, J25, J26, J27, J28: footprint ao_tht:Jack_6.35mm_PJ_629HAN -> ao_tht:Jack_6.35mm_PJ_629HAN_slots
Other:
- board text added: "Match these 2 resistors"
- board text added: "Match these 4 resistors"
- board text added: "Octave switch with 10 matched resistors added"
- board text removed: "Octave switch"

Commit message: Correct slide switch footprint; use TO-92 wide for regulator
Parts:
- U6: footprint Package_TO_SOT_THT:TO-92_Inline -> ao_tht:TO-92_Inline_Wide
- moved U6 2.58 mm to (135.8, 36.8)
- moved SW2 2.50 mm to (12.3, 121.3)
Connections:
- SW2 pad 1: /Octave and sync switches/HARD_SYNCA_P -> /Octave and sync switches/SOFT_SYNC_OFF_P
- SW2 pad 2: /Octave and sync switches/SYNCA_P -> /Octave and sync switches/SOFT_SYNCA_P
- SW2 pad 3: unconnected-(SW2-Pad3) -> /Octave and sync switches/SOFT_SYNC_OFF_P
- SW2 pad 4: /Octave and sync switches/SOFT_SYNCA_P -> unconnected-(SW2-Pad4)
- SW2 pad 5: /Octave and sync switches/SOFT_SYNC_OFF_P -> /Octave and sync switches/HARD_SYNCA_P
- SW2 pad 6: /Octave and sync switches/SOFT_SYNCA_P -> /Octave and sync switches/SYNCA_P
- SW2 pad 7: /Octave and sync switches/SOFT_SYNC_OFF_P -> unconnected-(SW2-Pad7)
- SW2 pad 8: unconnected-(SW2-Pad8) -> /Octave and sync switches/SOFT_SYNCA_P
Routing:
- net -12V: track 163.5 -> 164.5 mm

Commit message: 5 mm pitch for 330 pF
Parts:
- C18, C19: footprint ao_tht:C_Disc_D3.0mm_W1.6mm_P2.50mm -> ao_tht:C_Disc_D5.0mm_W2.5mm_P5.00mm
- moved C18 2.46 mm to (229.9, 120.7)
Routing:
- net /Outputs and sin/LINK_OUT_SAW: track 44.2 -> 44.9 mm
