File: Hardware/PCB/herovco/herovco.kicad_sch (KiCad schematic)
At the start: 9 parts, among them J1 Conn_01x09, J2 Conn_01x07, J3 Conn_01x06, J4 3_pin_Molex_header, J5 Conn_01x09, J6 Conn_01x07, J7 Conn_01x06, J8 3_pin_Molex_connector, J9 Conn_02x04_Odd_Even

Commit message: Change pot symbols and fix orientation, other small tweaks
Changed lines of the file:
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@@
     )
   )
-  (symbol (lib_id "ao_symbols:3_pin_Molex_header") (at 114.3 138.43 0)
+  (symbol (lib_id "ao_symbols:3_pin_Molex_header") (at 114.3 138.43 0) (unit 1)
     (in_bom yes) (on_board yes)
     (property "Reference" "J4" (id 0) (at 119.38 137.16 90)
@@
     (pin "3")
   )
-  (symbol (lib_id "Connector_Generic:Conn_01x06") (at 114.3 106.68 0)
+  (symbol (lib_id "Connector_Generic:Conn_01x06") (at 114.3 106.68 0) (unit 1)
     (in_bom yes) (on_board yes)
     (property "Reference" "J3" (id 0) (at 119.38 107.95 90)
@@
     (pin "6")
   )
-  (symbol (lib_id "Connector_Generic:Conn_01x07") (at 114.3 88.9 0)
+  (symbol (lib_id "Connector_Generic:Conn_01x07") (at 114.3 88.9 0) (unit 1)
     (in_bom yes) (on_board yes)
     (property "Reference" "J2" (id 0) (at 119.38 88.9 90))
@@
     (pin "7")
   )
-  (symbol (lib_id "Connector_Generic:Conn_01x09") (at 114.3 58.42 0)
+  (symbol (lib_id "Connector_Generic:Conn_01x09") (at 114.3 58.42 0) (unit 1)
     (in_bom yes) (on_board yes)
     (property "Reference" "J1" (id 0) (at 119.38 58.42 90))
@@
     (pin "9")
   )
-  (symbol (lib_id "Connector_Generic:Conn_01x09") (at 137.16 58.42 0) (mirror y)
+  (symbol (lib_id "Connector_Generic:Conn_01x09") (at 137.16 58.42 0) (mirror y) (unit 1)
     (in_bom yes) (on_board yes)
     (property "Reference" "J5" (id 0) (at 132.08 58.42 90))
@@
     (pin "9")
   )
-  (symbol (lib_id "Connector_Generic:Conn_02x04_Odd_Even") (at 222.25 88.9 0)
+  (symbol (lib_id "Connector_Generic:Conn_02x04_Odd_Even") (at 222.25 88.9 0) (unit 1)
     (in_bom yes) (on_board yes)
     (property "Reference" "J9" (id 0) (at 223.52 80.8482 0))
@@
     (pin "8")
   )
-  (symbol (lib_id "power:GND1") (at 232.41 95.25 0) (mirror y)
+  (symbol (lib_id "power:GND1") (at 232.41 95.25 0) (mirror y) (unit 1)
     (in_bom yes) (on_board yes)
     (property "Reference" "#PWR01" (id 0) (at 232.41 101.6 0)
@@
     (pin "1")
   )
-  (symbol (lib_id "Connector_Generic:Conn_01x06") (at 137.16 106.68 0) (mirror y)
+  (symbol (lib_id "Connector_Generic:Conn_01x06") (at 137.16 106.68 0) (mirror y) (unit 1)
     (in_bom yes) (on_board yes)
     (property "Reference" "J7" (id 0) (at 132.08 107.95 90)
@@
     (pin "6")
   )
-  (symbol (lib_id "Connector_Generic:Conn_01x07") (at 137.16 88.9 0) (mirror y)
+  (symbol (lib_id "Connector_Generic:Conn_01x07") (at 137.16 88.9 0) (mirror y) (unit 1)
     (in_bom yes) (on_board yes)
     (property "Reference" "J6" (id 0) (at 132.08 88.9 90))
@@
     (pin "7")
   )
-  (symbol (lib_id "ao_symbols:3_pin_Molex_connector") (at 137.16 138.43 0) (mirror y)
+  (symbol (lib_id "ao_symbols:3_pin_Molex_connector") (at 137.16 138.43 0) (mirror y) (unit 1)
     (in_bom yes) (on_board yes)
     (property "Reference" "J8" (id 0) (at 132.08 138.43 90))
@@
       (effects (font (size 1.27 1.27)) (justify right))
     )
-    (pin "+8V_REF" input (at 95.25 124.46 0)
+    (pin "+8V_REF" output (at 95.25 124.46 0)
       (effects (font (size 1.27 1.27)) (justify right))
     )
@@
       (effects (font (size 1.27 1.27)) (justify left top))
     )
-    (pin "OCTAVE_P" input (at 160.02 135.89 180)
-      (effects (font (size 1.27 1.27)) (justify left))
-    )
     (pin "+8V_REF_P" input (at 160.02 138.43 180)
       (effects (font (size 1.27 1.27)) (justify left))
     )
     (pin "0V" input (at 160.02 140.97 180)
+      (effects (font (size 1.27 1.27)) (justify left))
+    )
+    (pin "OCTAVE_P" output (at 160.02 135.89 180)
       (effects (font (size 1.27 1.27)) (justify left))
     )
@@
       (effects (font (size 1.27 1.27)) (justify left top))
     )
-    (pin "SIN_S_CW_S" input (at 160.02 93.98 180)
-      (effects (font (size 1.27 1.27)) (justify left))
-    )
-    (pin "SIN_S_CCW_S" input (at 160.02 88.9 180)
-      (effects (font (size 1.27 1.27)) (justify left))
-    )
-    (pin "SIN_S_W_S" input (at 160.02 91.44 180)
-      (effects (font (size 1.27 1.27)) (justify left))
-    )
-    (pin "SIN_R_W_S" input (at 160.02 96.52 180)
-      (effects (font (size 1.27 1.27)) (justify left))
-    )
-    (pin "SIN_R_CCW_S" input (at 160.02 86.36 180)
+    (pin "SIN_S_CW_S" output (at 160.02 93.98 180)
+      (effects (font (size 1.27 1.27)) (justify left))
+    )
+    (pin "SIN_S_CCW_S" output (at 160.02 88.9 180)
+      (effects (font (size 1.27 1.27)) (justify left))
+    )
+    (pin "SIN_S_W_S" output (at 160.02 91.44 180)
+      (effects (font (size 1.27 1.27)) (justify left))
+    )
+    (pin "SIN_R_W_S" output (at 160.02 96.52 180)
+      (effects (font (size 1.27 1.27)) (justify left))
+    )
+    (pin "SIN_R_CCW_S" output (at 160.02 86.36 180)
       (effects (font (size 1.27 1.27)) (justify left))
     )
@@
       (effects (font (size 1.27 1.27)) (justify left))
     )
-    (pin "GND_BACK" input (at 160.02 48.26 180)
-      (effects (font (size 1.27 1.27)) (justify left))
-    )
-    (pin "+12V_BACK" input (at 160.02 53.34 180)
-      (effects (font (size 1.27 1.27)) (justify left))
-    )
-    (pin "-12V_BACK" input (at 160.02 50.8 180)
+    (pin "GND_BACK" output (at 160.02 48.26 180)
+      (effects (font (size 1.27 1.27)) (justify left))
+    )
+    (pin "+12V_BACK" output (at 160.02 53.34 180)
+      (effects (font (size 1.27 1.27)) (justify left))
+    )
+    (pin "-12V_BACK" output (at 160.02 50.8 180)
       (effects (font (size 1.27 1.27)) (justify left))
     )
@@
     )
     (path "/00000000-0000-0000-0000-000061942543/00000000-0000-0000-0000-000060939e16"
-      (reference "C2") (unit 1) (value "10nF") (footprint "ao_tht:C_Rect_L7.2mm_W2.5mm_P5.00mm_FKS2_FKP2_MKS2_MKP2")
+      (reference "C2") (unit 1) (value "10nF") (footprint "ao_tht:C_Disc_D3.0mm_W1.6mm_P2.50mm")
     )
     (path "/00000000-0000-0000-0000-000061942543/00000000-0000-0000-0000-00005f157032"
@@
     )
     (path "/00000000-0000-0000-0000-000061942543/00000000-0000-0000-0000-000060f756fe"
-      (reference "C6") (unit 1) (value "1nF") (footprint "ao_tht:C_Rect_L7.2mm_W2.5mm_P5.00mm_FKS2_FKP2_MKS2_MKP2")
+      (reference "C6") (unit 1) (value "1nF") (footprint "ao_tht:C_Disc_D3.0mm_W1.6mm_P2.50mm")
     )
     (path "/00000000-0000-0000-0000-000061942543/00000000-0000-0000-0000-00006181e495"
-      (reference "C7") (unit 1) (value "10nF") (footprint "ao_tht:C_Rect_L7.2mm_W2.5mm_P5.00mm_FKS2_FKP2_MKS2_MKP2")
+      (reference "C7") (unit 1) (value "10nF") (footprint "ao_tht:C_Disc_D3.0mm_W1.6mm_P2.50mm")
     )
     (path "/00000000-0000-0000-0000-000061942543/00000000-0000-0000-0000-000060f0a6ec"
-      (reference "C8") (unit 1) (value "10nF") (footprint "ao_tht:C_Rect_L7.2mm_W2.5mm_P5.00mm_FKS2_FKP2_MKS2_MKP2")
+      (reference "C8") (unit 1) (value "10nF") (footprint "ao_tht:C_Disc_D3.0mm_W1.6mm_P2.50mm")
     )
     (path "/00000000-0000-0000-0000-000061942543/00000000-0000-0000-0000-0000615ab5be"
@@
     )
     (path "/00000000-0000-0000-0000-000061a0b1ab/00000000-0000-0000-0000-00005f5271a5"
-      (reference "C16") (unit 1) (value "10uF") (footprint "ao_tht:CP_Radial_D5.0mm_P2.00mm")
+      (reference "C16") (unit 1) (value "10uF") (footprint "ao_tht:CP_Radial_D6.3mm_P2.50mm")
     )
     (path "/00000000-0000-0000-0000-000061a0b1ab/00000000-0000-0000-0000-00005f5271ab"
-      (reference "C17") (unit 1) (value "10uF") (footprint "ao_tht:CP_Radial_D5.0mm_P2.00mm")
+      (reference "C17") (unit 1) (value "10uF") (footprint "ao_tht:CP_Radial_D6.3mm_P2.50mm")
     )
     (path "/00000000-0000-0000-0000-000061942543/00000000-0000-0000-0000-00006181739b"
@@
     )
     (path "/00000000-0000-0000-0000-000061942543/00000000-0000-0000-0000-0000616604b5"
-      (reference "D2") (unit 1) (value "1N4732A") (footprint "ao_tht:D_DO-41_SOD81_P10.16mm_Horizontal")
+      (reference "D2") (unit 1) (value "1N4732A") (footprint "Diode_THT:D_DO-41_SOD81_P10.16mm_Horizontal")
     )
     (path "/00000000-0000-0000-0000-000061a0b1ab/00000000-0000-0000-0000-00005f776ff5"
@@
     )
     (path "/00000000-0000-0000-0000-000061942543/00000000-0000-0000-0000-000061a3d1dc"
-      (reference "U4") (unit 1) (value "TL431LP") (footprint "ao_tht:TO-92_Inline_Wide")
+      (reference "U4") (unit 1) (value "TL431LP") (footprint "Package_TO_SOT_THT:TO-92_Inline")
     )
     (path "/00000000-0000-0000-0000-000061942543/00000000-0000-0000-0000-000061817387"
-      (reference "U5") (unit 1) (value "L79L05_TO92") (footprint "ao_tht:TO-92_Inline_Wide")
+      (reference "U5") (unit 1) (value "L79L05_TO92") (footprint "Package_TO_SOT_THT:TO-92_Inline")
     )
     (path "/00000000-0000-0000-0000-0000619fd1d7/00000000-0000-0000-0000-000062fc82dc"

Commit message: Pre-breadboard updates
Connections:
- net Front PCB/+8V_REF: now also J4.3 (Pin_3); no longer J4.2 (Pin_2)
- net Front PCB/OCTAVE: now also J4.2 (Pin_2); no longer J4.1 (Pin_1)
- net Octave switch/+8V_REF_P: now also J8.3 (Pin_3); no longer J8.2 (Pin_2)
- net Octave switch/0V: now also J8.1 (Pin_1); no longer J8.3 (Pin_3)
- net Octave switch/OCTAVE_P: now also J8.2 (Pin_2); no longer J8.1 (Pin_1)
- net Front PCB/GND_FRONT renamed GND
- net GND: now also J4.1 (Pin_1); no longer J4.3 (Pin_3)
Other:
- moved on the sheet: J4, J8

Commit message: rm Zener, change adj ref to fixed and modify octave switch and fine tune accordingly
Connections:
- net Front PCB/+8V_REF renamed Front PCB/+10V_REF
- net Octave switch/+8V_REF_P renamed Octave switch/+10V_REF_P
Other:
- sheet Front PCB ports: added +10V_REF; removed +8V_REF
- sheet Octave switch ports: added +10V_REF_P; removed +8V_REF_P

Commit message: Sync input revision
Parts:
- added J10: 4_pin_Molex_connector, ao_tht:Molex_KK-254_AE-6410-04A_1x04_P2.54mm_Vertical, symbol Connector_Generic:Conn_01x04
- added J5: 4_pin_Molex_header, ao_tht:Molex_KK-254_AE-6410-04A_1x04_P2.54mm_Vertical, symbol Connector_Generic:Conn_01x04
- renumbered J9 to J11, J5 to J6, J6 to J7, J7 to J8, J8 to J9
Connections:
- new net Front PCB/HARD_SYNCA: J5.4 (Pin_4)
- new net Front PCB/SOFT_SYNCA: J5.2 (Pin_2)
- new net Front PCB/SOFT_SYNC_OFF: J5.3 (Pin_3)
- new net Front PCB/SYNCA: J5.1 (Pin_1)
- new net Octave and sync switches/HARD_SYNCA_P: J10.4 (Pin_4)
- new net Octave and sync switches/SOFT_SYNCA_P: J10.2 (Pin_2)
- new net Octave and sync switches/SOFT_SYNC_OFF_P: J10.3 (Pin_3)
- new net Octave and sync switches/SYNCA_P: J10.1 (Pin_1)
Other:
- sheet Octave switch renamed Octave and sync switches
- sheet Front PCB ports: added HARD_SYNCA, SOFT_SYNCA, SOFT_SYNC_OFF, SYNCA; removed none
- sheet Octave and sync switches ports: added HARD_SYNCA_P, SOFT_SYNCA_P, SOFT_SYNC_OFF_P, SYNCA_P; removed none
- moved on the sheet: J4

Commit message: Big panel and PCB revisions
Parts:
- removed J3: Conn_01x06, Connector_PinHeader_2.54mm:PinHeader_1x06_P2.54mm_Vertical, symbol Connector_Generic:Conn_01x06
- removed J8: Conn_01x06, Connector_PinSocket_2.54mm:PinSocket_1x06_P2.54mm_Vertical, symbol Connector_Generic:Conn_01x06
- added J10, J9: Conn_01x03, Connector_PinSocket_2.54mm:PinSocket_1x03_P2.54mm_Vertical, symbol Connector_Generic:Conn_01x03
- added J3, J4: Conn_01x03, Connector_PinHeader_2.54mm:PinHeader_1x03_P2.54mm_Vertical, symbol Connector_Generic:Conn_01x03
- J12: renamed from J10; footprint ao_tht:Molex_KK-254_AE-6410-04A_1x04_P2.54mm_Vertical -> Connector_Molex:Molex_KK-254_AE-6410-04A_1x04_P2.54mm_Vertical
- J6: renamed from J5; footprint ao_tht:Molex_KK-254_AE-6410-04A_1x04_P2.54mm_Vertical -> Connector_Molex:Molex_KK-254_AE-6410-04A_1x04_P2.54mm_Vertical
- renumbered J9 to J11, J11 to J13, J4 to J5, J6 to J7, J7 to J8
Connections:
- net Front PCB/LINK_OUT_CV: now also J4.3 (Pin_3)
- net Front PCB/LINK_OUT_FM: now also J4.1 (Pin_1)
- net Front PCB/LINK_OUT_PW: now also J4.2 (Pin_2)
- net Front PCB/PULSE_OUT: now also J3.2 (Pin_2)
- net Front PCB/SAW_OUT: now also J3.3 (Pin_3)
- net Front PCB/TRIANGLE_OUT: now also J3.1 (Pin_1)
- net LINK_OUT_CV_L: now also J10.3 (Pin_3)
- net LINK_OUT_FM_L: now also J10.1 (Pin_1)
- net LINK_OUT_PW_L: now also J10.2 (Pin_2)
- net Outputs and sin/PULSE_OUT_S: now also J9.2 (Pin_2)
- net Outputs and sin/SAW_OUT_S: now also J9.3 (Pin_3)
- net Outputs and sin/TRIANGLE_OUT_S: now also J9.1 (Pin_1)

Commit message: Sch cleanup, switch footprint
Connections:
- net Front PCB/+12V_FRONT renamed +12V
- net Front PCB/-12V_FRONT renamed -12V
- net Jacks, power, etc/+12V_BACK renamed +12V_1
- net Jacks, power, etc/-12V_BACK renamed -12V_1
Other:
- sheet Front PCB ports: added none; removed +12V_FRONT, -12V_FRONT, GND_FRONT
- sheet Jacks, power, etc ports: added none; removed +12V_BACK, -12V_BACK, GND_BACK
- sheet Outputs and sin ports: added none; removed GND_BACK
