File: Hardware/PCB/herovco/herovco.kicad_sch (KiCad schematic)
At the start: 17 parts, among them J1 Conn_01x09, J10 Conn_01x03, J11 Conn_01x03, J12 3_pin_Molex_connector, J13 Wire pads, J14 Conn_01x01, J15 Conn_01x01, J16 Conn_01x01, J17 Conn_02x04_Odd_Even, J2 Conn_01x03, J3 Conn_01x03, J4 3_pin_Molex_header, J5 Wire pads, J6 Conn_01x01, J7 Conn_01x01, J8 Conn_01x01, J9 Conn_01x09

Commit message: Initial BOM; DNF the test points; README typo
Parts:
- J13, J14, J15, J16, J5, J6, J7, J8: Config (none) -> DNF
Changed lines of the file:
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@@
+      (effects (font (size 1.27 1.27)) hide)
+    )
+    (property "Config" "DNF" (id 4) (at 114.3 137.16 0)
       (effects (font (size 1.27 1.27)) hide)
     )
@@
       (effects (font (size 1.27 1.27)) hide)
     )
+    (property "Config" "DNF" (id 4) (at 137.16 139.7 0)
+      (effects (font (size 1.27 1.27)) hide)
+    )
     (pin "1")
   )
@@
       (effects (font (size 1.27 1.27)) hide)
     )
+    (property "Config" "DNF" (id 4) (at 137.16 142.24 0)
+      (effects (font (size 1.27 1.27)) hide)
+    )
     (pin "1")
   )
@@
       (effects (font (size 1.27 1.27)) hide)
     )
+    (property "Config" "DNF" (id 4) (at 114.3 139.7 0)
+      (effects (font (size 1.27 1.27)) hide)
+    )
     (pin "1")
   )
@@
     )
     (property "Datasheet" "~" (id 3) (at 137.16 137.16 0)
+      (effects (font (size 1.27 1.27)) hide)
+    )
+    (property "Config" "DNF" (id 4) (at 137.16 137.16 0)
       (effects (font (size 1.27 1.27)) hide)
     )
@@
       (effects (font (size 1.27 1.27)) hide)
     )
+    (property "Config" "DNF" (id 4) (at 114.3 142.24 0)
+      (effects (font (size 1.27 1.27)) hide)
+    )
     (pin "1")
   )
@@
     )
     (property "Datasheet" "~" (id 3) (at 137.16 144.78 0)
+      (effects (font (size 1.27 1.27)) hide)
+    )
+    (property "Config" "DNF" (id 4) (at 137.16 144.78 0)
       (effects (font (size 1.27 1.27)) hide)
     )
@@
       (effects (font (size 1.27 1.27)) hide)
     )
+    (property "Config" "DNF" (id 4) (at 114.3 144.78 0)
+      (effects (font (size 1.27 1.27)) hide)
+    )
