File: Hardware/PCB/herovco/herovco_front.kicad_sch (KiCad schematic)
At the start: 71 parts, among them SW2 SW_SPDT_MSM, U1 TL074, U2 AS3340A, U3 TL072, U4 TL431LP, U5 L79L05_TO92

Commit message: Change pot symbols and fix orientation, other small tweaks
Parts:
- C2, C6, C7, C8: footprint ao_tht:C_Rect_L7.2mm_W2.5mm_P5.00mm_FKS2_FKP2_MKS2_MKP2 -> ao_tht:C_Disc_D3.0mm_W1.6mm_P2.50mm
- D2: footprint ao_tht:D_DO-41_SOD81_P10.16mm_Horizontal -> Diode_THT:D_DO-41_SOD81_P10.16mm_Horizontal
- RV1, RV10, RV11, RV3, RV4: symbol Device:R_POT -> ao_symbols:R_POT; Vendor (none) -> Tayda
- U4, U5: footprint ao_tht:TO-92_Inline_Wide -> Package_TO_SOT_THT:TO-92_Inline
Connections:
- net +12V: now also U1.4 (V+)
- net -12V: now also U1.11 (V-)
Other:
- note added: "Sine amplitude"
- note removed: "Sin amplitude"

Commit message: Pre-breadboard updates
Parts:
- B1: Config (none) -> DNF
- R9: value 3M -> 10M
- RV12, RV13, RV2, RV5, RV6, RV7, RV8, RV9: footprint ao_tht:Potentiometer_Bourns_3296W_Vertical_screw_centered -> ao_tht:Potentiometer_Bourns_3296W_Vertical_standard; symbol Device:R_POT_TRIM -> ao_symbols:R_POT_TRIM_3296W; Vendor (none) -> Tayda
- SW2: symbol Switch:SW_SPDT_MSM -> ao_symbols:SW_SPDT_MSM; SKU (none) -> A-3187; Vendor (none) -> Tayda
- U1: symbol Amplifier_Operational:TL074 -> ao_symbols:TL074; SKU (none) -> A-1138; Vendor (none) -> Tayda
Other:
- note added: "I did some tests that indicated 3M is better than 10M for suppressing high frequency oscillations, but in later tests 10M looked OK and 3M had a bad effect on minimum pulse width. 1M killed PW range totally. But Henry uses 1M + 1 nF to ground, for better fall time and to suppress oscillations respectively. I don't understand seeming inconsistency."
- note added: "TRACKING"
- note removed: "I did some tests that indicated 3M is better than 10M for suppressing high frequency oscillations, but in later tests 10M looked OK and 3M had a bad effect on minimum pulse width. I don't understand seeming inconsistency."

Commit message: rm Zener, change adj ref to fixed and modify octave switch and fine tune accordingly
Parts:
- removed D2: 1N4732A, Diode_THT:D_DO-41_SOD81_P10.16mm_Horizontal, symbol Diode:1N47xxA
- removed R28: 8.2k, ao_tht:R_Axial_DIN0207_L6.3mm_D2.5mm_P10.16mm_Horizontal, symbol ao_symbols:R
- removed R29: 1k, ao_tht:R_Axial_DIN0207_L6.3mm_D2.5mm_P10.16mm_Horizontal, symbol ao_symbols:R
- removed RV7: 10k, ao_tht:Potentiometer_Bourns_3296W_Vertical_standard, symbol ao_symbols:R_POT_TRIM_3296W
- removed TP1: TestPoint, TestPoint:TestPoint_Pad_2.5x2.5mm, symbol Connector:TestPoint
- removed U4: TL431LP, Package_TO_SOT_THT:TO-92_Inline, symbol Reference_Voltage:TL431LP
- added C18: 10nF, ao_tht:C_Disc_D3.0mm_W1.6mm_P2.50mm, symbol ao_symbols:C
- added R64: 470R, ao_tht:R_Axial_DIN0207_L6.3mm_D2.5mm_P10.16mm_Horizontal, symbol ao_symbols:R
- added U?: LM4040LP-10, ao_tht:TO-92_Inline_Wide, symbol ao_symbols:LM4040LP-10
- R10: value 300k -> 200k
- RV1: value 100k -> 50k
- RV12, RV13, RV2, RV5, RV6, RV8, RV9: footprint ao_tht:Potentiometer_Bourns_3296W_Vertical_standard -> ao_tht:Potentiometer_Bourns_3296W_Vertical_screw_centered
Connections:
- net CV_NODE: now also R64.1
- net GND: now also C6.1, C18.2, U?.3 (A); no longer C6.2
- net at U2.11 (Cap): now also C6.2; no longer C6.1
- net +8V_REF renamed +10V_REF
- net +10V_REF: now also U?.2 (K)
- new net: C18.1, R64.2
Other:
- note added: "+10 V REFERENCE"
- note added: "For VCC=12V, PWM_IN value for 100% PW is typically 4.0 V, maximum 4.3 V. With PWMIN=0, PULSE_WIDTH ±12 V becomes ∓5 V at op amp output. With PULSE_WIDTH=0, PWM_IN ±5 V becomes ∓5 V at op amp output. Either way LINK_OUT_PW becomes ±5 V. (Larger range if both CVs are nonzero.) At top of trimmer V is 5.5 to 0 V. Adjust trimmer to get correct upper limit."
- note removed: "+8V REFERENCE"
- note removed: "For VCC=12V, PWM_IN value for 100% PW is typically 4.0 V, maximum 4.3 V. With PWMIN=0, PULSE_WIDTH ±12 V becomes ∓5 V at op amp output. With PULSE_WIDTH=0, PWM_IN ±5 V becomes ∓5 V at op amp output. Either way LINK_OUT_PW becomes ±5 V. At top of trimmer V is 5.5 to 0 V. Adjust trimmer to get correct upper limit. Zener clamps to 4.7 to 0 V."
- moved on the sheet: C6, C8, R21, R22, R23, R25, R26, R27, R30, TP2, TP3, TP4

Commit message: rm Zener, change adj ref to fixed, cont'd
Parts:
- gave numbers to parts that had none: 1
Changed lines of the file:
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@@
   (symbol (lib_id "ao_symbols:LM4040LP-10") (at 152.4 59.69 90) (unit 1)
     (in_bom yes) (on_board yes) (fields_autoplaced)
-    (property "Reference" "U?" (id 0) (at 154.4066 58.7815 90)
+    (property "Reference" "U4" (id 0) (at 154.4066 58.7815 90)
       (effects (font (size 1.27 1.27)) (justify right))
     )

Commit message: Panel updates; reannotate; correct PCB errors
Parts:
- renumbered C9 to C10, C10 to C11, C11 to C12, C18 to C4, C4 to C5, C5 to C6, C6 to C7, C7 to C8, C8 to C9, R9 to R1, R18 to R10, R19 to R11, R64 to R12, R20 to R13, R21 to R14, R22 to R15, R23 to R16, R24 to R17, R25 to R18, R26 to R19, R10 to R2, R27 to R20, R30 to R21, R31 to R22, R32 to R23, R33 to R24, R34 to R25, R35 to R26, R36 to R27, R37 to R28, R11 to R3, R12 to R4, R13 to R5, R14 to R6, R15 to R7, R16 to R8, R17 to R9, RV9 to RV10, RV12 to RV11, RV13 to RV12, RV10 to RV7, RV11 to RV8, RV8 to RV9, SW2 to SW1, TP2 to TP1, TP3 to TP2, TP4 to TP3

Commit message: Sync input revision
Parts:
- removed SW1: SW_SPDT_MSM, ao_tht:SPDT-toggle-switch-1M-series, symbol ao_symbols:SW_SPDT_MSM
- added C12: 100nF, ao_tht:C_Disc_D3.0mm_W1.6mm_P2.50mm, symbol ao_symbols:C
- added D1: 1N4148, ao_tht:D_DO-35_SOD27_P7.62mm_Horizontal, symbol ao_symbols:1N4148
- added R17: 5.6k, ao_tht:R_Axial_DIN0207_L6.3mm_D2.5mm_P10.16mm_Horizontal, symbol ao_symbols:R
- added R18: 47k, ao_tht:R_Axial_DIN0207_L6.3mm_D2.5mm_P10.16mm_Horizontal, symbol ao_symbols:R
- added R23: 10k, ao_tht:R_Axial_DIN0207_L6.3mm_D2.5mm_P10.16mm_Horizontal, symbol ao_symbols:R
- C7: renamed from C2; value 10nF -> 100nF
- R1: value 10M -> 1M
- renumbered C8 to C10, C9 to C11, C12 to C13, C5 to C2, C6 to C3, C10 to C4, C11 to C5, C3 to C6, C4 to C8, C7 to C9, D1 to D2, R17 to R19, R18 to R20, R19 to R21, R20 to R22, R21 to R24, R22 to R25, R23 to R26, R24 to R27, R25 to R28, R26 to R29, R27 to R30, R28 to R31, U3 to U2, U2 to U3
Connections:
- net GND: now also C12.1, R23.1
- net HARD_SYNC: now also D1.2 (A)
- net SOFT_SYNC: now also R18.1
- net SYNCA: now reaches C7.1
- new net: D1.1 (K), R17.1, R23.2
- new net HARD_SYNCA: R17.2
- new net SOFT_SYNCA: R18.2
- new net SOFT_SYNC_OFF: C12.2
Other:
- note added: "Regulated -5V is recommended by Alfa, and tests show it mostly suppresses PW frequency shift."
- note removed: "I did some tests that indicated 3M is better than 10M for suppressing high frequency oscillations, but in later tests 10M looked OK and 3M had a bad effect on minimum pulse width. 1M killed PW range totally. But Henry uses 1M + 1 nF to ground, for better fall time and to suppress oscillations respectively. I don't understand seeming inconsistency."
- note removed: "In Sidekick: LINK CV goes through 100k to CV_NODE (summed inside 3340) LINK FM goes through 10nF + 1M to LIN_FM (summed inside 3340) LINK PW goes through 100k to PWM summing amp (summed outside 3340) LINK SAW goes to SYNC"
- note removed: "Regulated -5V is recommended by Alfa, and tests show it mostly or entirely suppresses PW frequency shift."
- moved on the sheet: C2, C3, C4, C5, C7, U1E, U2C

Commit message: Big panel and PCB revisions
Parts:
- C10, C11, C12, C13, C7, C8: footprint ao_tht:C_Disc_D3.0mm_W1.6mm_P2.50mm -> ao_tht:C_Rect_L7.2mm_W2.5mm_P5.00mm_FKS2_FKP2_MKS2_MKP2
- C9: footprint ao_tht:C_Disc_D3.0mm_W1.6mm_P2.50mm -> Capacitor_THT:C_Rect_L7.2mm_W4.5mm_P5.00mm_FKS2_FKP2_MKS2_MKP2
- GRAF1: footprint herovco_panel:herovco_panel_holes -> herovco:herovco_panel_behind
Changed lines of the file:
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@@
     (property "Reference" "C7" (id 0) (at 99.06 173.9392 90))
     (property "Value" "100nF" (id 1) (at 99.06 176.2506 90))
-    (property "Footprint" "ao_tht:C_Disc_D3.0mm_W1.6mm_P2.50mm" (id 2) (at 95.25 181.3052 0)
+    (property "Footprint" "ao_tht:C_Rect_L7.2mm_W2.5mm_P5.00mm_FKS2_FKP2_MKS2_MKP2" (id 2) (at 95.25 181.3052 0)
       (effects (font (size 1.27 1.27)) hide)
     )
@@
       (effects (font (size 1.27 1.27)) (justify left))
     )
-    (property "Footprint" "ao_tht:C_Disc_D3.0mm_W1.6mm_P2.50mm" (id 2) (at 126.6952 63.5 0)
+    (property "Footprint" "ao_tht:C_Rect_L7.2mm_W2.5mm_P5.00mm_FKS2_FKP2_MKS2_MKP2" (id 2) (at 126.6952 63.5 0)
       (effects (font (size 1.27 1.27)) hide)
     )
@@
       (effects (font (size 1.27 1.27)) (justify left))
     )
-    (property "Footprint" "ao_tht:C_Disc_D3.0mm_W1.6mm_P2.50mm" (id 2) (at 120.3452 38.1 0)
+    (property "Footprint" "Capacitor_THT:C_Rect_L7.2mm_W4.5mm_P5.00mm_FKS2_FKP2_MKS2_MKP2" (id 2) (at 120.3452 38.1 0)
       (effects (font (size 1.27 1.27)) hide)
     )
@@
       (effects (font (size 1.27 1.27)) (justify left))
     )
-    (property "Footprint" "ao_tht:C_Disc_D3.0mm_W1.6mm_P2.50mm" (id 2) (at 211.7852 46.99 0)
+    (property "Footprint" "ao_tht:C_Rect_L7.2mm_W2.5mm_P5.00mm_FKS2_FKP2_MKS2_MKP2" (id 2) (at 211.7852 46.99 0)
       (effects (font (size 1.27 1.27)) hide)
     )
@@
     (property "Reference" "C10" (id 0) (at 121.92 78.6892 90))
     (property "Value" "10nF" (id 1) (at 121.92 81.0006 90))
-    (property "Footprint" "ao_tht:C_Disc_D3.0mm_W1.6mm_P2.50mm" (id 2) (at 118.11 86.0552 0)
+    (property "Footprint" "ao_tht:C_Rect_L7.2mm_W2.5mm_P5.00mm_FKS2_FKP2_MKS2_MKP2" (id 2) (at 118.11 86.0552 0)
       (effects (font (size 1.27 1.27)) hide)
     )
@@
       (effects (font (size 1.27 1.27)) (justify left))
     )
-    (property "Footprint" "herovco_panel:herovco_panel_holes" (id 2) (at 22.86 186.69 0)
+    (property "Footprint" "herovco:herovco_panel_behind" (id 2) (at 22.86 186.69 0)
       (effects (font (size 1.27 1.27)) hide)
     )
@@
       (effects (font (size 1.27 1.27)) (justify left))
     )
-    (property "Footprint" "ao_tht:C_Disc_D3.0mm_W1.6mm_P2.50mm" (id 2) (at 105.1052 67.31 0)
+    (property "Footprint" "ao_tht:C_Rect_L7.2mm_W2.5mm_P5.00mm_FKS2_FKP2_MKS2_MKP2" (id 2) (at 105.1052 67.31 0)
       (effects (font (size 1.27 1.27)) hide)
     )
@@
     (property "Reference" "C12" (id 0) (at 134.62 186.6392 90))
     (property "Value" "100nF" (id 1) (at 134.62 188.9506 90))
-    (property "Footprint" "ao_tht:C_Disc_D3.0mm_W1.6mm_P2.50mm" (id 2) (at 130.81 194.0052 0)
-      (effects (font (size 1.27 1.27)) hide)
-    )
+    (property "Footprint" "ao_tht:C_Rect_L7.2mm_W2.5mm_P5.00mm_FKS2_FKP2_MKS2_MKP2" (id 2) (at 130.81 194.0052 0)
+      (effects (font (size 1.27 1.27)) hide)
+    )

Commit message: Sch cleanup, switch footprint
Other:
- moved on the sheet: TP1, TP2, TP3
