File: Hardware/PCB/herovco/herovco_front.kicad_sch (KiCad schematic)
At the start: 71 parts, among them U1 TL074, U2 TL072, U3 AS3340A, U4 LM4040LP-10, U5 L79L05_TO92

Commit message: Sine trimmers to back board, misc accumulated tweaks
Parts:
- removed RV10, RV9: 50k, ao_tht:Potentiometer_Bourns_3296W_Vertical_screw_centered, symbol ao_symbols:R_POT_TRIM_3296W
- removed RV11: 5k, ao_tht:Potentiometer_Bourns_3296W_Vertical_screw_centered, symbol ao_symbols:R_POT_TRIM_3296W
Other:
- note added: "Make this 470k?"
- note removed: "SINE TRIMMERS"
- note removed: "Sine amplitude"
- note removed: "Sine round"
- note removed: "Sine symmetry"

Commit message: Schematics tweaks, silk and fab cleanup, layout PDFs, panel revisions
Parts:
- removed R2: 200k, ao_tht:R_Axial_DIN0207_L6.3mm_D2.5mm_P10.16mm_Horizontal, symbol ao_symbols:R
- added R24: 1k, ao_tht:R_Axial_DIN0207_L6.3mm_D2.5mm_P10.16mm_Horizontal, symbol ao_symbols:R
- added TP2: +5VREF, ao_tht:TestPoint_THTPad_D1.5mm_Drill0.7mm, symbol ao_symbols:TestPoint
- added TP4: -5VREF, ao_tht:TestPoint_THTPad_D1.5mm_Drill0.7mm, symbol ao_symbols:TestPoint
- added TP6: -5V, ao_tht:TestPoint_THTPad_D1.5mm_Drill0.7mm, symbol ao_symbols:TestPoint
- added U5: LM4040BIZ-5, ao_tht:TO-92_Inline_Wide, symbol ao_symbols:LM4040LP-5
- R20: renamed from R21; value 100k -> 47k
- RV1: value 50k -> 100k
- RV6: value 100k -> 20k
- TP5: renamed from TP3; footprint ao_tht:TestPoint_THTPad_1.5x1.5mm_Drill0.7mm -> ao_tht:TestPoint_THTPad_D1.5mm_Drill0.7mm
- U4: value LM4040LP-10 -> LM4040BIZ-5; symbol ao_symbols:LM4040LP-10 -> ao_symbols:LM4040LP-5
- renumbered R11 to R10, R12 to R11, R13 to R12, R14 to R13, R15 to R14, R16 to R15, R17 to R16, R18 to R17, R19 to R18, R20 to R19, R3 to R2, R22 to R21, R23 to R22, R24 to R23, R4 to R3, R5 to R4, R6 to R5, R7 to R6, R9 to R7, R10 to R9, RV12 to RV9, TP2 to TP3, U5 to U6
Connections:
- net +10V_REF is gone; now on net +5V_REF: R23.2, RV6.3, U4.2 (K)
- net -12V: now also R24.2
- net -5V: now also TP6.1
- net FINE_TUNE: now also R7.2; no longer R8.2
- net FREQ_CV: now also R8.2; no longer R7.2
- net GND: now also U5.2 (K); no longer RV1.1
- net +5V_REF: now reaches RV1.3
- net +5V_REF: now also TP2.1
- new net -5V_REF: R24.1, RV1.1, TP4.1, U5.3 (A)
Other:
- note added: "-5V reg"
- note added: "PWM max limit"
- note added: "Thomas Henry claims 1M between pins 4 and 5 improves pulse wave fall time and 1 nF cap from pin 5 to ground suppresses falling edge oscillations. What I see is 1M suppresses oscillations, does not affect fall time, and 1 nF makes fall time significantly worse. Must be something else going on I guess."
- note added: "±5 V REFERENCES"
- note removed: "+10 V REFERENCE"
- note removed: "-5V"
- moved on the sheet: C13, D2, R7, R8, U4, U6

Commit message: schem tweaks
Other:
- note added: "-5V REGULATOR"
- note removed: "-5V reg"
- note removed: "Can dispense with this op amp if there's a better use for it somewhere else"
- moved on the sheet: C13, D2, TP6, U6

Commit message: Initial BOM; DNF the test points; README typo
Parts:
- TP1, TP3, TP5: Config (none) -> DNF
Changed lines of the file:
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@@
+      (effects (font (size 1.27 1.27)) hide)
+    )
+    (property "Config" "DNF" (id 4) (at 158.75 91.44 0)
       (effects (font (size 1.27 1.27)) hide)
     )
@@
       (effects (font (size 1.27 1.27)) hide)
     )
+    (property "Config" "DNF" (id 4) (at 181.61 91.44 0)
+      (effects (font (size 1.27 1.27)) hide)
+    )
     (pin "1")
   )
@@
       (effects (font (size 1.27 1.27)) hide)
     )
+    (property "Config" "DNF" (id 4) (at 204.47 91.44 0)
+      (effects (font (size 1.27 1.27)) hide)
+    )

Commit message: Correct slide switch footprint; use TO-92 wide for regulator
Parts:
- U6: footprint Package_TO_SOT_THT:TO-92_Inline -> ao_tht:TO-92_Inline_Wide
Changed lines of the file:
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@@
     (property "Reference" "U6" (id 0) (at 241.3 47.1932 0))
     (property "Value" "L79L05_TO92" (id 1) (at 241.3 49.5046 0))
-    (property "Footprint" "Package_TO_SOT_THT:TO-92_Inline" (id 2) (at 241.3 48.26 0)
+    (property "Footprint" "ao_tht:TO-92_Inline_Wide" (id 2) (at 241.3 48.26 0)
       (effects (font (size 1.27 1.27) italic) hide)
     )

Commit message: Use uninverted PW CV
Connections:
- net LINK_OUT_PW: now also R30.2
- net at R27.2, R28.1, U2.1: no longer R30.2
Other:
- note added: "For VCC=12V, PWM_IN value for 100% PW is typically 4.0 V, maximum 4.3 V. With PWMIN=0, PULSE_WIDTH ±12 V becomes ∓5 V at op amp output. With PULSE_WIDTH=0, PWM_IN ±5 V becomes ∓5 V at op amp output. Either way LINK_OUT_PW becomes ±5 V. (Larger range if both CVs are nonzero.) At top of trimmer V is 0 to 5.5 V. Adjust trimmer to get correct upper limit."
- note removed: "For VCC=12V, PWM_IN value for 100% PW is typically 4.0 V, maximum 4.3 V. With PWMIN=0, PULSE_WIDTH ±12 V becomes ∓5 V at op amp output. With PULSE_WIDTH=0, PWM_IN ±5 V becomes ∓5 V at op amp output. Either way LINK_OUT_PW becomes ±5 V. (Larger range if both CVs are nonzero.) At top of trimmer V is 5.5 to 0 V. Adjust trimmer to get correct upper limit."
- moved on the sheet: C12, C7, D1, R16, R17, R22, R27, R29, R30, R31, RV9, U2B

Commit message: Revert "Use uninverted PW CV"
This reverts commit afeb33e5ee15cb89f0e577c33928166723912ed3.
Connections:
- net LINK_OUT_PW: no longer R30.2
- net at R27.2, R28.1, U2.1: now also R30.2
Other:
- note added: "For VCC=12V, PWM_IN value for 100% PW is typically 4.0 V, maximum 4.3 V. With PWMIN=0, PULSE_WIDTH ±12 V becomes ∓5 V at op amp output. With PULSE_WIDTH=0, PWM_IN ±5 V becomes ∓5 V at op amp output. Either way LINK_OUT_PW becomes ±5 V. (Larger range if both CVs are nonzero.) At top of trimmer V is 5.5 to 0 V. Adjust trimmer to get correct upper limit."
- note removed: "For VCC=12V, PWM_IN value for 100% PW is typically 4.0 V, maximum 4.3 V. With PWMIN=0, PULSE_WIDTH ±12 V becomes ∓5 V at op amp output. With PULSE_WIDTH=0, PWM_IN ±5 V becomes ∓5 V at op amp output. Either way LINK_OUT_PW becomes ±5 V. (Larger range if both CVs are nonzero.) At top of trimmer V is 0 to 5.5 V. Adjust trimmer to get correct upper limit."
- moved on the sheet: C12, C7, D1, R16, R17, R22, R27, R29, R30, R31, RV9, U2B
