File: Hardware/PCB/herovco/herovco_front.kicad_sch (KiCad schematic)
At the start: 72 parts, among them U1 TL074, U2 TL072, U3 AS3340A, U4 LM4040BIZ-5, U5 LM4040BIZ-5, U6 L79L05_TO92

Commit message: Post prototype updates
Parts:
- C10, C11, C13, C8: SKU (none) -> A-559
- C12, C7: SKU (none) -> A-564
- C9: SKU (none) -> FKP2G011001D00HSSD; Vendor Tayda -> Digi-Key
- RV1, RV3, RV4, RV7, RV8: SKU (none) -> A-1848 or A-5513
- RV2: SKU (none) -> A-586
- RV5, RV6: SKU (none) -> A-592
- RV9: SKU (none) -> A-598
- U3: Vendor (none) -> CabinTech Global
- U4, U5: SKU (none) -> LM4040BIZ-5/NOPB-ND; Vendor (none) -> Digi-Key
- U6: SKU (none) -> A-4676; Vendor (none) -> Tayda

Commit message: 20k trimmers to 10k
Parts:
- RV5, RV6: value 20k -> 10k
Other:
- note removed: "Make this 470k?"
Changed lines of the file:
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@@
     (effects (font (size 1.27 1.27)) (justify left bottom))
-  )
-  (text "Make this 470k?" (at 130.81 116.84 0)
-    (effects (font (size 2.032 2.032)) (justify left bottom))
   )
   (label "PULSE_WIDTH" (at 175.26 124.46 0)
@@
     (in_bom yes) (on_board yes)
     (property "Reference" "RV5" (id 0) (at 116.84 112.8522 90))
-    (property "Value" "20k" (id 1) (at 116.84 115.1636 90))
+    (property "Value" "10k" (id 1) (at 116.84 115.1636 90))
     (property "Footprint" "ao_tht:Potentiometer_Bourns_3296W_Vertical_screw_centered" (id 2) (at 116.84 118.11 0)
       (effects (font (size 1.27 1.27)) hide)
@@
     (in_bom yes) (on_board yes)
     (property "Reference" "RV6" (id 0) (at 116.84 126.8222 90))
-    (property "Value" "20k" (id 1) (at 116.84 129.1336 90))
+    (property "Value" "10k" (id 1) (at 116.84 129.1336 90))
     (property "Footprint" "ao_tht:Potentiometer_Bourns_3296W_Vertical_screw_centered" (id 2) (at 116.84 132.08 0)
       (effects (font (size 1.27 1.27)) hide)
