File: Hardware/PCB/herovco/octave.kicad_sch (KiCad schematic)
At the start: 9 parts, among them SW1 SW_Rotary12

Commit message: Change pot symbols and fix orientation, other small tweaks
Changed lines of the file:
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@@
   (no_connect (at 147.32 82.55))
   (no_connect (at 147.32 77.47))
-  (wire (pts (xy 100.33 93.98) (xy 124.46 93.98))
+  (wire (pts (xy 102.87 93.98) (xy 124.46 93.98))
     (stroke (width 0) (type default) (color 0 0 0 0))
   )
@@
   )
   (polyline (pts (xy 125.73 129.54) (xy 113.03 129.54))
-    (stroke (width 0) (type default) (color 0 0 0 0))
+    (stroke (width 0) (type default) (color 194 0 194 1))
   )
   (wire (pts (xy 140.97 97.79) (xy 147.32 97.79))
@@
     (stroke (width 0) (type default) (color 0 0 0 0))
   )
-  (wire (pts (xy 100.33 91.44) (xy 123.19 91.44))
+  (wire (pts (xy 102.87 91.44) (xy 123.19 91.44))
     (stroke (width 0) (type default) (color 0 0 0 0))
   )
@@
   )
   (polyline (pts (xy 135.89 60.96) (xy 135.89 129.54))
-    (stroke (width 0) (type default) (color 0 0 0 0))
+    (stroke (width 0) (type default) (color 194 0 194 1))
   )
   (wire (pts (xy 140.97 92.71) (xy 140.97 97.79))
@@
   )
   (polyline (pts (xy 135.89 129.54) (xy 151.13 129.54))
-    (stroke (width 0) (type default) (color 0 0 0 0))
+    (stroke (width 0) (type default) (color 194 0 194 1))
   )
   (polyline (pts (xy 151.13 134.62) (xy 113.03 134.62))
-    (stroke (width 0) (type default) (color 0 0 0 0))
+    (stroke (width 0) (type default) (color 194 0 194 1))
   )
   (wire (pts (xy 143.51 77.47) (xy 143.51 90.17))
@@
     (stroke (width 0) (type default) (color 0 0 0 0))
   )
-  (wire (pts (xy 100.33 96.52) (xy 123.19 96.52))
+  (wire (pts (xy 102.87 96.52) (xy 123.19 96.52))
     (stroke (width 0) (type default) (color 0 0 0 0))
   )
@@
   )
   (polyline (pts (xy 125.73 60.96) (xy 125.73 129.54))
-    (stroke (width 0) (type default) (color 0 0 0 0))
+    (stroke (width 0) (type default) (color 194 0 194 1))
   )
   (polyline (pts (xy 113.03 129.54) (xy 113.03 134.62))
-    (stroke (width 0) (type default) (color 0 0 0 0))
+    (stroke (width 0) (type default) (color 194 0 194 1))
   )
   (polyline (pts (xy 85.09 140.97) (xy 179.07 140.97))
@@
   )
   (polyline (pts (xy 151.13 129.54) (xy 151.13 134.62))
-    (stroke (width 0) (type default) (color 0 0 0 0))
+    (stroke (width 0) (type default) (color 194 0 194 1))
   )
   (polyline (pts (xy 125.73 60.96) (xy 135.89 60.96))
-    (stroke (width 0) (type default) (color 0 0 0 0))
+    (stroke (width 0) (type default) (color 194 0 194 1))
   )
   (polyline (pts (xy 85.09 52.07) (xy 179.07 52.07))
@@
     (effects (font (size 1.27 1.27)) (justify left bottom))
   )
-  (hierarchical_label "0V" (shape input) (at 107.95 96.52 270)
+  (hierarchical_label "0V" (shape input) (at 102.87 96.52 180)
     (effects (font (size 1.27 1.27)) (justify right))
   )
-  (hierarchical_label "OCTAVE_P" (shape input) (at 102.87 91.44 270)
+  (hierarchical_label "OCTAVE_P" (shape output) (at 102.87 91.44 180)
     (effects (font (size 1.27 1.27)) (justify right))
   )
-  (hierarchical_label "+8V_REF_P" (shape input) (at 105.41 93.98 270)
+  (hierarchical_label "+8V_REF_P" (shape input) (at 102.87 93.98 180)
     (effects (font (size 1.27 1.27)) (justify right))
   )
-  (symbol (lib_id "Switch:SW_Rotary12") (at 157.48 92.71 180)
+  (symbol (lib_id "Switch:SW_Rotary12") (at 157.48 92.71 180) (unit 1)
     (in_bom yes) (on_board yes)
     (property "Reference" "SW1" (id 0) (at 160.02 71.755 0))
@@
     (pin "9")
   )
-  (symbol (lib_id "ao_symbols:R") (at 130.81 66.04 0) (mirror x)
+  (symbol (lib_id "ao_symbols:R") (at 130.81 66.04 0) (mirror x) (unit 1)
     (in_bom yes) (on_board yes)
     (property "Reference" "R1" (id 0) (at 132.08 64.135 0)
@@
     (pin "2")
   )
-  (symbol (lib_id "ao_symbols:R") (at 130.81 73.66 0) (mirror x)
+  (symbol (lib_id "ao_symbols:R") (at 130.81 73.66 0) (mirror x) (unit 1)
     (in_bom yes) (on_board yes)
     (property "Reference" "R2" (id 0) (at 132.08 71.755 0)
@@
     (pin "2")
   )
-  (symbol (lib_id "ao_symbols:R") (at 130.81 81.28 0) (mirror x)
+  (symbol (lib_id "ao_symbols:R") (at 130.81 81.28 0) (mirror x) (unit 1)
     (in_bom yes) (on_board yes)
     (property "Reference" "R3" (id 0) (at 132.08 79.375 0)
@@
     (pin "2")
   )
-  (symbol (lib_id "ao_symbols:R") (at 130.81 88.9 0) (mirror x)
+  (symbol (lib_id "ao_symbols:R") (at 130.81 88.9 0) (mirror x) (unit 1)
     (in_bom yes) (on_board yes)
     (property "Reference" "R4" (id 0) (at 132.08 86.995 0)
@@
     (pin "2")
   )
-  (symbol (lib_id "ao_symbols:R") (at 130.81 96.52 0) (mirror x)
+  (symbol (lib_id "ao_symbols:R") (at 130.81 96.52 0) (mirror x) (unit 1)
     (in_bom yes) (on_board yes)
     (property "Reference" "R5" (id 0) (at 132.08 94.615 0)
@@
     (pin "2")
   )
-  (symbol (lib_id "ao_symbols:R") (at 130.81 104.14 0) (mirror x)
+  (symbol (lib_id "ao_symbols:R") (at 130.81 104.14 0) (mirror x) (unit 1)
     (in_bom yes) (on_board yes)
     (property "Reference" "R6" (id 0) (at 132.08 102.235 0)
@@
     (pin "2")
   )
-  (symbol (lib_id "ao_symbols:R") (at 130.81 111.76 0) (mirror x)
+  (symbol (lib_id "ao_symbols:R") (at 130.81 111.76 0) (mirror x) (unit 1)
     (in_bom yes) (on_board yes)
     (property "Reference" "R7" (id 0) (at 132.08 109.855 0)
@@
     (pin "2")
   )
-  (symbol (lib_id "ao_symbols:R") (at 130.81 119.38 0) (mirror x)
+  (symbol (lib_id "ao_symbols:R") (at 130.81 119.38 0) (mirror x) (unit 1)
     (in_bom yes) (on_board yes)
     (property "Reference" "R8" (id 0) (at 132.08 117.475 0)

Commit message: Pre-breadboard updates
Parts:
- SW1: symbol Switch:SW_Rotary12 -> ao_symbols:SW_Rotary12; SKU (none) -> A-1893; Vendor (none) -> Tayda
Changed lines of the file:
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@@
     (comment 1 "or neighboring rights to this work. Published from United States.")
     (comment 2 "To the extent possible under law, Richard Holmes has waived all copyright and related ")
-    (comment 3 "Based mainly on Kassutronics VCO 3340")
+    (comment 3 "Partly based on designs by Kassutronics, Thomas Henry, and LMNC")
   )
   (junction (at 130.81 92.71) (diameter 0) (color 0 0 0 0)
@@
     (effects (font (size 1.27 1.27)) (justify right))
   )
-  (symbol (lib_id "Switch:SW_Rotary12") (at 157.48 92.71 180) (unit 1)
+  (symbol (lib_id "ao_symbols:SW_Rotary12") (at 157.48 92.71 180) (unit 1)
     (in_bom yes) (on_board yes)
     (property "Reference" "SW1" (id 0) (at 160.02 71.755 0))
@@
       (effects (font (size 1.27 1.27)) hide)
     )
+    (property "Vendor" "Tayda" (id 4) (at 157.48 92.71 0)
+      (effects (font (size 1.27 1.27)) hide)
+    )
+    (property "SKU" "A-1893" (id 5) (at 157.48 92.71 0)
+      (effects (font (size 1.27 1.27)) hide)
+    )

Commit message: rm Zener, change adj ref to fixed and modify octave switch and fine tune accordingly
Parts:
- added R? (x2): 10k 1/8W, ao_tht:R_Axial_DIN0207_L6.3mm_D2.5mm_P10.16mm_Horizontal, symbol ao_symbols:R
Connections:
- net at SW1.10: now also R?.1, R?.2
- net +10V_REF_P: now reaches SW1.11
- net +10V_REF_P: now also R?.2
- net +8V_REF_P: no longer names the net of R1.2, SW1.9
- net +8V_REF_P: now also R?.1
- no-connect marks 3 -> 1
Other:
- note removed: "Octave switch"
- moved on the sheet: R1, R2, R3, R4, R5, R6, R7, R8, SW1

Commit message: rm Zener, change adj ref to fixed, cont'd
Parts:
- gave numbers to parts that had none: 2
Changed lines of the file:
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@@
   (symbol (lib_id "ao_symbols:R") (at 119.38 67.31 0) (mirror x) (unit 1)
     (in_bom yes) (on_board yes)
-    (property "Reference" "R?" (id 0) (at 120.65 65.405 0)
+    (property "Reference" "R28" (id 0) (at 120.65 65.405 0)
       (effects (font (size 1.27 1.27)) (justify left))
     )
@@
   (symbol (lib_id "ao_symbols:R") (at 119.38 74.93 0) (mirror x) (unit 1)
     (in_bom yes) (on_board yes)
-    (property "Reference" "R?" (id 0) (at 120.65 73.025 0)
+    (property "Reference" "R29" (id 0) (at 120.65 73.025 0)
       (effects (font (size 1.27 1.27)) (justify left))
     )

Commit message: Panel updates; reannotate; correct PCB errors
Parts:
- renumbered R28 to R29, R29 to R30, R1 to R31, R2 to R32, R3 to R33, R4 to R34, R5 to R35, R6 to R36, R7 to R37, R8 to R38, SW1 to SW2
Changed lines of the file:
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@@
   (symbol (lib_id "ao_symbols:SW_Rotary12") (at 151.13 109.22 180) (unit 1)
     (in_bom yes) (on_board yes)
-    (property "Reference" "SW1" (id 0) (at 153.67 88.265 0))
+    (property "Reference" "SW2" (id 0) (at 153.67 88.265 0))
     (property "Value" "SW_Rotary12" (id 1) (at 153.67 90.5764 0))
     (property "Footprint" "ao_tht:Rotary_Switch" (id 2) (at 156.21 127 0)
@@
   (symbol (lib_id "ao_symbols:R") (at 119.38 82.55 0) (mirror x) (unit 1)
     (in_bom yes) (on_board yes)
-    (property "Reference" "R1" (id 0) (at 120.65 80.645 0)
+    (property "Reference" "R31" (id 0) (at 120.65 80.645 0)
       (effects (font (size 1.27 1.27)) (justify left))
     )
@@
   (symbol (lib_id "ao_symbols:R") (at 119.38 90.17 0) (mirror x) (unit 1)
     (in_bom yes) (on_board yes)
-    (property "Reference" "R2" (id 0) (at 120.65 88.265 0)
+    (property "Reference" "R32" (id 0) (at 120.65 88.265 0)
       (effects (font (size 1.27 1.27)) (justify left))
     )
@@
   (symbol (lib_id "ao_symbols:R") (at 119.38 97.79 0) (mirror x) (unit 1)
     (in_bom yes) (on_board yes)
-    (property "Reference" "R3" (id 0) (at 120.65 95.885 0)
+    (property "Reference" "R33" (id 0) (at 120.65 95.885 0)
       (effects (font (size 1.27 1.27)) (justify left))
     )
@@
   (symbol (lib_id "ao_symbols:R") (at 119.38 105.41 0) (mirror x) (unit 1)
     (in_bom yes) (on_board yes)
-    (property "Reference" "R4" (id 0) (at 120.65 103.505 0)
+    (property "Reference" "R34" (id 0) (at 120.65 103.505 0)
       (effects (font (size 1.27 1.27)) (justify left))
     )
@@
   (symbol (lib_id "ao_symbols:R") (at 119.38 113.03 0) (mirror x) (unit 1)
     (in_bom yes) (on_board yes)
-    (property "Reference" "R5" (id 0) (at 120.65 111.125 0)
+    (property "Reference" "R35" (id 0) (at 120.65 111.125 0)
       (effects (font (size 1.27 1.27)) (justify left))
     )
@@
   (symbol (lib_id "ao_symbols:R") (at 119.38 120.65 0) (mirror x) (unit 1)
     (in_bom yes) (on_board yes)
-    (property "Reference" "R6" (id 0) (at 120.65 118.745 0)
+    (property "Reference" "R36" (id 0) (at 120.65 118.745 0)
       (effects (font (size 1.27 1.27)) (justify left))
     )
@@
   (symbol (lib_id "ao_symbols:R") (at 119.38 128.27 0) (mirror x) (unit 1)
     (in_bom yes) (on_board yes)
-    (property "Reference" "R7" (id 0) (at 120.65 126.365 0)
+    (property "Reference" "R37" (id 0) (at 120.65 126.365 0)
       (effects (font (size 1.27 1.27)) (justify left))
     )
@@
   (symbol (lib_id "ao_symbols:R") (at 119.38 135.89 0) (mirror x) (unit 1)
     (in_bom yes) (on_board yes)
-    (property "Reference" "R8" (id 0) (at 120.65 133.985 0)
+    (property "Reference" "R38" (id 0) (at 120.65 133.985 0)
       (effects (font (size 1.27 1.27)) (justify left))
     )
@@
   (symbol (lib_id "ao_symbols:R") (at 119.38 67.31 0) (mirror x) (unit 1)
     (in_bom yes) (on_board yes)
-    (property "Reference" "R28" (id 0) (at 120.65 65.405 0)
+    (property "Reference" "R29" (id 0) (at 120.65 65.405 0)
       (effects (font (size 1.27 1.27)) (justify left))
     )
@@
   (symbol (lib_id "ao_symbols:R") (at 119.38 74.93 0) (mirror x) (unit 1)
     (in_bom yes) (on_board yes)
-    (property "Reference" "R29" (id 0) (at 120.65 73.025 0)
-      (effects (font (size 1.27 1.27)) (justify left))
-    )
+    (property "Reference" "R30" (id 0) (at 120.65 73.025 0)
+      (effects (font (size 1.27 1.27)) (justify left))
+    )

Commit message: Sync input revision
Parts:
- added SW2: SW_DP3T, symbol Switch:SW_DP3T
- renumbered R29 to R32, R30 to R33, R31 to R34, R32 to R35, R33 to R36, R34 to R37, R35 to R38, R36 to R39, R37 to R40, R38 to R41, SW2 to SW1
Connections:
- new net HARD_SYNCA_P: SW2.1
- new net SOFT_SYNCA_P: SW2.4, SW2.7
- new net SOFT_SYNC_OFF_P: SW2.5, SW2.6
- new net SYNCA_P: SW2.3
- no-connect marks 1 -> 3
Other:
- note added: "SYNC SWITCH"
Changed lines of the file:
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@@
   (junction (at 119.38 116.84) (diameter 0) (color 0 0 0 0)
   )
+  (junction (at 215.9 101.6) (diameter 0) (color 0 0 0 0)
+  )
   (junction (at 119.38 71.12) (diameter 0) (color 0 0 0 0)
   )
@@
   (junction (at 119.38 86.36) (diameter 0) (color 0 0 0 0)
   )
+  (junction (at 229.87 110.49) (diameter 0) (color 0 0 0 0)
+  )
   (junction (at 119.38 132.08) (diameter 0) (color 0 0 0 0)
   )
   (junction (at 119.38 124.46) (diameter 0) (color 0 0 0 0)
   )
+  (no_connect (at 227.33 115.57))
   (no_connect (at 140.97 93.98))
+  (no_connect (at 214.63 99.06))
   (wire (pts (xy 110.49 63.5) (xy 119.38 63.5))
     (stroke (width 0) (type default) (color 0 0 0 0))
@@
     (stroke (width 0) (type default) (color 0 0 0 0))
   )
+  (wire (pts (xy 217.17 113.03) (xy 215.9 113.03))
+    (stroke (width 0) (type default) (color 0 0 0 0))
+  )
   (wire (pts (xy 170.18 109.22) (xy 166.37 109.22))
     (stroke (width 0) (type default) (color 0 0 0 0))
@@
     (stroke (width 0) (type default) (color 0 0 0 0))
   )
+  (wire (pts (xy 232.41 110.49) (xy 229.87 110.49))
+    (stroke (width 0) (type default) (color 0 0 0 0))
+  )
+  (wire (pts (xy 227.33 113.03) (xy 229.87 113.03))
+    (stroke (width 0) (type default) (color 0 0 0 0))
+  )
   (wire (pts (xy 132.08 124.46) (xy 132.08 119.38))
     (stroke (width 0) (type default) (color 0 0 0 0))
@@
     (stroke (width 0) (type default) (color 0 0 0 0))
   )
+  (polyline (pts (xy 189.23 52.07) (xy 189.23 124.46))
+    (stroke (width 0) (type default) (color 0 0 0 0))
+  )
+  (polyline (pts (xy 257.81 52.07) (xy 257.81 124.46))
+    (stroke (width 0) (type default) (color 0 0 0 0))
+  )
   (polyline (pts (xy 184.15 52.07) (xy 184.15 156.21))
     (stroke (width 0) (type default) (color 0 0 0 0))
@@
     (stroke (width 0) (type default) (color 0 0 0 0))
   )
+  (wire (pts (xy 229.87 110.49) (xy 227.33 110.49))
+    (stroke (width 0) (type default) (color 0 0 0 0))
+  )
   (wire (pts (xy 134.62 139.7) (xy 134.62 124.46))
     (stroke (width 0) (type default) (color 0 0 0 0))
@@
     (stroke (width 0) (type default) (color 0 0 0 0))
   )
+  (wire (pts (xy 218.44 96.52) (xy 214.63 96.52))
+    (stroke (width 0) (type default) (color 0 0 0 0))
+  )
   (wire (pts (xy 119.38 86.36) (xy 133.35 86.36))
     (stroke (width 0) (type default) (color 0 0 0 0))
   )
+  (wire (pts (xy 215.9 113.03) (xy 215.9 101.6))
+    (stroke (width 0) (type default) (color 0 0 0 0))
+  )
+  (wire (pts (xy 224.79 101.6) (xy 215.9 101.6))
+    (stroke (width 0) (type default) (color 0 0 0 0))
+  )
   (wire (pts (xy 119.38 109.22) (xy 129.54 109.22))
     (stroke (width 0) (type default) (color 0 0 0 0))
@@
     (stroke (width 0) (type default) (color 0 0 0 0))
   )
+  (wire (pts (xy 215.9 101.6) (xy 214.63 101.6))
+    (stroke (width 0) (type default) (color 0 0 0 0))
+  )
+  (wire (pts (xy 229.87 113.03) (xy 229.87 110.49))
+    (stroke (width 0) (type default) (color 0 0 0 0))
+  )
   (wire (pts (xy 133.35 86.36) (xy 133.35 104.14))
     (stroke (width 0) (type default) (color 0 0 0 0))
@@
     (stroke (width 0) (type default) (color 0 0 0 0))
   )
+  (polyline (pts (xy 189.23 52.07) (xy 257.81 52.07))
+    (stroke (width 0) (type default) (color 0 0 0 0))
+  )
   (wire (pts (xy 137.16 96.52) (xy 140.97 96.52))
     (stroke (width 0) (type default) (color 0 0 0 0))
@@
   (polyline (pts (xy 101.6 146.05) (xy 101.6 151.13))
     (stroke (width 0) (type default) (color 194 0 194 1))
+  )
+  (polyline (pts (xy 257.81 124.46) (xy 189.23 124.46))
+    (stroke (width 0) (type default) (color 0 0 0 0))
   )
   (polyline (pts (xy 85.09 156.21) (xy 184.15 156.21))
@@
     (effects (font (size 1.27 1.27)) (justify left bottom))
   )
+  (text "SYNC\nSWITCH" (at 203.2 72.39 0)
+    (effects (font (size 3.81 3.81)) (justify left bottom))
+  )
   (text "OCTAVE\nSWITCH" (at 146.05 72.39 0)
     (effects (font (size 3.81 3.81)) (justify left bottom))
@@
     (effects (font (size 1.27 1.27)) (justify left bottom))
   )
+  (text "Panel mounted" (at 203.2 78.74 0)
+    (effects (font (size 1.27 1.27)) (justify left bottom))
+  )
   (hierarchical_label "0V" (shape input) (at 110.49 139.7 180)
     (effects (font (size 1.27 1.27)) (justify right))
@@
     (effects (font (size 1.27 1.27)) (justify left))
   )
+  (hierarchical_label "SOFT_SYNC_OFF_P" (shape output) (at 232.41 110.49 0)
+    (effects (font (size 1.27 1.27)) (justify left))
+  )
+  (hierarchical_label "SYNCA_P" (shape input) (at 204.47 99.06 180)
+    (effects (font (size 1.27 1.27)) (justify right))
+  )
+  (hierarchical_label "HARD_SYNCA_P" (shape output) (at 218.44 96.52 0)
+    (effects (font (size 1.27 1.27)) (justify left))
+  )
   (hierarchical_label "+10V_REF_P" (shape input) (at 110.49 63.5 180)
     (effects (font (size 1.27 1.27)) (justify right))
   )
+  (hierarchical_label "SOFT_SYNCA_P" (shape output) (at 224.79 101.6 0)
+    (effects (font (size 1.27 1.27)) (justify left))
+  )
   (symbol (lib_id "ao_symbols:SW_Rotary12") (at 151.13 109.22 180) (unit 1)
     (in_bom yes) (on_board yes)
-    (property "Reference" "SW2" (id 0) (at 153.67 88.265 0))
+    (property "Reference" "SW1" (id 0) (at 153.67 88.265 0))
     (property "Value" "SW_Rotary12" (id 1) (at 153.67 90.5764 0))
     (property "Footprint" "ao_tht:Rotary_Switch" (id 2) (at 156.21 127 0)
@@
   (symbol (lib_id "ao_symbols:R") (at 119.38 82.55 0) (mirror x) (unit 1)
     (in_bom yes) (on_board yes)
-    (property "Reference" "R31" (id 0) (at 120.65 80.645 0)
+    (property "Reference" "R34" (id 0) (at 120.65 80.645 0)
       (effects (font (size 1.27 1.27)) (justify left))
     )
@@
   (symbol (lib_id "ao_symbols:R") (at 119.38 90.17 0) (mirror x) (unit 1)
     (in_bom yes) (on_board yes)
-    (property "Reference" "R32" (id 0) (at 120.65 88.265 0)
+    (property "Reference" "R35" (id 0) (at 120.65 88.265 0)
       (effects (font (size 1.27 1.27)) (justify left))
     )
@@
   (symbol (lib_id "ao_symbols:R") (at 119.38 97.79 0) (mirror x) (unit 1)
     (in_bom yes) (on_board yes)
-    (property "Reference" "R33" (id 0) (at 120.65 95.885 0)
+    (property "Reference" "R36" (id 0) (at 120.65 95.885 0)
       (effects (font (size 1.27 1.27)) (justify left))
     )
@@
   (symbol (lib_id "ao_symbols:R") (at 119.38 105.41 0) (mirror x) (unit 1)
     (in_bom yes) (on_board yes)
-    (property "Reference" "R34" (id 0) (at 120.65 103.505 0)
+    (property "Reference" "R37" (id 0) (at 120.65 103.505 0)
       (effects (font (size 1.27 1.27)) (justify left))
     )
@@
   (symbol (lib_id "ao_symbols:R") (at 119.38 113.03 0) (mirror x) (unit 1)
     (in_bom yes) (on_board yes)
-    (property "Reference" "R35" (id 0) (at 120.65 111.125 0)
+    (property "Reference" "R38" (id 0) (at 120.65 111.125 0)
       (effects (font (size 1.27 1.27)) (justify left))
     )
@@
   (symbol (lib_id "ao_symbols:R") (at 119.38 120.65 0) (mirror x) (unit 1)
     (in_bom yes) (on_board yes)
-    (property "Reference" "R36" (id 0) (at 120.65 118.745 0)
+    (property "Reference" "R39" (id 0) (at 120.65 118.745 0)
       (effects (font (size 1.27 1.27)) (justify left))
     )
@@
   (symbol (lib_id "ao_symbols:R") (at 119.38 128.27 0) (mirror x) (unit 1)
     (in_bom yes) (on_board yes)
-    (property "Reference" "R37" (id 0) (at 120.65 126.365 0)
+    (property "Reference" "R40" (id 0) (at 120.65 126.365 0)
       (effects (font (size 1.27 1.27)) (justify left))
     )
@@
   (symbol (lib_id "ao_symbols:R") (at 119.38 135.89 0) (mirror x) (unit 1)
     (in_bom yes) (on_board yes)
-    (property "Reference" "R38" (id 0) (at 120.65 133.985 0)
+    (property "Reference" "R41" (id 0) (at 120.65 133.985 0)
       (effects (font (size 1.27 1.27)) (justify left))
     )
@@
   (symbol (lib_id "ao_symbols:R") (at 119.38 67.31 0) (mirror x) (unit 1)
     (in_bom yes) (on_board yes)
-    (property "Reference" "R29" (id 0) (at 120.65 65.405 0)
+    (property "Reference" "R32" (id 0) (at 120.65 65.405 0)
       (effects (font (size 1.27 1.27)) (justify left))
     )
@@
     (pin "2")
   )
+  (symbol (lib_name "SW_DP3T_1") (lib_id "Switch:SW_DP3T") (at 209.55 99.06 0) (unit 1)
+    (in_bom yes) (on_board yes) (fields_autoplaced)
+    (property "Reference" "SW2" (id 0) (at 209.55 92.2233 0))
+    (property "Value" "SW_DP3T" (id 1) (at 209.55 94.9984 0))
+    (property "Footprint" "" (id 2) (at 193.675 94.615 0)
+      (effects (font (size 1.27 1.27)) hide)
+    )
+    (property "Datasheet" "~" (id 3) (at 193.675 94.615 0)
+      (effects (font (size 1.27 1.27)) hide)
+    )
+    (property "Manufacturer" "CW Industries" (id 4) (at 209.55 99.06 0)
+      (effects (font (size 1.27 1.27)) hide)
+    )
+    (property "Part" "G-1128S-0055" (id 5) (at 209.55 99.06 0)
+      (effects (font (size 1.27 1.27)) hide)
+    )
+    (pin "1")
+    (pin "2")
+    (pin "3")
+    (pin "4")
+  )
   (symbol (lib_id "ao_symbols:R") (at 119.38 74.93 0) (mirror x) (unit 1)
     (in_bom yes) (on_board yes)
-    (property "Reference" "R30" (id 0) (at 120.65 73.025 0)
+    (property "Reference" "R33" (id 0) (at 120.65 73.025 0)
       (effects (font (size 1.27 1.27)) (justify left))
     )
@@
     (pin "2")
   )
+  (symbol (lib_id "Switch:SW_DP3T") (at 222.25 113.03 0) (unit 2)
+    (in_bom yes) (on_board yes) (fields_autoplaced)
+    (property "Reference" "SW2" (id 0) (at 222.25 106.1933 0))
+    (property "Value" "SW_DP3T" (id 1) (at 222.25 108.9684 0))
+    (property "Footprint" "" (id 2) (at 206.375 108.585 0)
+      (effects (font (size 1.27 1.27)) hide)
+    )
+    (property "Datasheet" "~" (id 3) (at 206.375 108.585 0)
+      (effects (font (size 1.27 1.27)) hide)
+    )
+    (pin "5")
+    (pin "6")
+    (pin "7")
+    (pin "8")
+  )
 )

Commit message: Big panel and PCB revisions
Parts:
- SW2: footprint (none) -> ao_tht:Heatsink_17x17mm_A-5093
Changed lines of the file:
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@@
     (property "Reference" "SW2" (id 0) (at 209.55 92.2233 0))
     (property "Value" "SW_DP3T" (id 1) (at 209.55 94.9984 0))
-    (property "Footprint" "" (id 2) (at 193.675 94.615 0)
+    (property "Footprint" "ao_tht:Heatsink_17x17mm_A-5093" (id 2) (at 193.675 94.615 0)
       (effects (font (size 1.27 1.27)) hide)
     )
@@
     (property "Reference" "SW2" (id 0) (at 222.25 106.1933 0))
     (property "Value" "SW_DP3T" (id 1) (at 222.25 108.9684 0))
-    (property "Footprint" "" (id 2) (at 206.375 108.585 0)
+    (property "Footprint" "ao_tht:Heatsink_17x17mm_A-5093" (id 2) (at 206.375 108.585 0)
       (effects (font (size 1.27 1.27)) hide)
     )

Commit message: Sch cleanup, switch footprint
Parts:
- removed SW2: SW_DP3T, ao_tht:Heatsink_17x17mm_A-5093, symbol Switch:SW_DP3T
- added SW2: SW_DP3T, herovco:G-1128S_DP3T, symbol herovco:SW_DP3T
Connections:
- net HARD_SYNCA_P: now also SW2.1
- net SOFT_SYNCA_P: now also SW2.4, SW2.7
- net SOFT_SYNC_OFF_P: now also SW2.5, SW2.6
- net SYNCA_P: now also SW2.3
Other:
- moved on the sheet: R32, R33, R34, R35, R36, R37, R38, R39, R40, R41, SW1
