File: Hardware/PCB/herovco/octave.kicad_sch (KiCad schematic)
At the start: 12 parts, among them SW1 SW_Rotary12, SW2 SW_DP3T

Commit message: Different sync switch, other tweaks
Parts:
- added B3: Board, ao_tht:Board_Marker, symbol ao_symbols:Board
- SW2: footprint herovco:G-1128S_DP3T -> herovco:SW_CK_OS203012MU5QP1_DP3T; Manufacturer CW Industries -> C&K; Part G-1128S-0055 -> OS203012MU5QP1‎; SKU SW334-ND -> CKN9554-ND
Connections:
- net SOFT_SYNCA_P: now also SW2.6; no longer SW2.7
- net SOFT_SYNC_OFF_P: now also SW2.7; no longer SW2.6
- net SYNCA_P: now also SW2.2; no longer SW2.3
Changed lines of the file:
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@@
     (pin "2")
   )
-  (symbol (lib_id "herovco:SW_DP3T") (at 175.26 99.06 0) (unit 1)
+  (symbol (lib_name "SW_DP3T_1") (lib_id "herovco:SW_DP3T") (at 175.26 99.06 0) (unit 1)
     (in_bom yes) (on_board yes) (fields_autoplaced)
     (property "Reference" "SW2" (id 0) (at 175.26 92.2233 0))
     (property "Value" "SW_DP3T" (id 1) (at 175.26 94.9984 0))
-    (property "Footprint" "herovco:G-1128S_DP3T" (id 2) (at 159.385 94.615 0)
+    (property "Footprint" "herovco:SW_CK_OS203012MU5QP1_DP3T" (id 2) (at 159.385 94.615 0)
       (effects (font (size 1.27 1.27)) hide)
     )
@@
       (effects (font (size 1.27 1.27)) hide)
     )
-    (property "Manufacturer" "CW Industries" (id 4) (at 175.26 99.06 0)
+    (property "Manufacturer" "C&K" (id 4) (at 175.26 99.06 0)
       (effects (font (size 1.27 1.27)) hide)
     )
-    (property "Part" "G-1128S-0055" (id 5) (at 175.26 99.06 0)
+    (property "Part" "OS203012MU5QP1‎" (id 5) (at 175.26 99.06 0)
       (effects (font (size 1.27 1.27)) hide)
     )
@@
       (effects (font (size 1.27 1.27)) hide)
     )
-    (property "SKU" "SW334-ND" (id 7) (at 175.26 99.06 0)
+    (property "SKU" "CKN9554-ND" (id 7) (at 175.26 99.06 0)
       (effects (font (size 1.27 1.27)) hide)
     )
@@
     (property "Reference" "SW2" (id 0) (at 187.96 106.1933 0))
     (property "Value" "SW_DP3T" (id 1) (at 187.96 108.9684 0))
-    (property "Footprint" "herovco:G-1128S_DP3T" (id 2) (at 172.085 108.585 0)
+    (property "Footprint" "herovco:SW_CK_OS203012MU5QP1_DP3T" (id 2) (at 172.085 108.585 0)
       (effects (font (size 1.27 1.27)) hide)
     )
@@
       (effects (font (size 1.27 1.27)) hide)
     )
-    (property "Manufacturer" "CW Industries" (id 4) (at 187.96 113.03 0)
+    (property "Manufacturer" "C&K" (id 4) (at 187.96 113.03 0)
       (effects (font (size 1.27 1.27)) hide)
     )
-    (property "Part" "G-1128S-0055" (id 5) (at 187.96 113.03 0)
+    (property "Part" "OS203012MU5QP1‎" (id 5) (at 187.96 113.03 0)
       (effects (font (size 1.27 1.27)) hide)
     )
@@
       (effects (font (size 1.27 1.27)) hide)
     )
-    (property "SKU" "SW334-ND" (id 7) (at 187.96 113.03 0)
+    (property "SKU" "CKN9554-ND" (id 7) (at 187.96 113.03 0)
       (effects (font (size 1.27 1.27)) hide)
     )
@@
     (pin "8")
   )
+  (symbol (lib_id "ao_symbols:Board") (at 209.55 72.39 0) (unit 1)
+    (in_bom yes) (on_board yes) (fields_autoplaced)
+    (property "Reference" "B3" (id 0) (at 215.265 71.4815 0)
+      (effects (font (size 1.27 1.27)) (justify left))
+    )
+    (property "Value" "Board" (id 1) (at 215.265 74.2566 0)
+      (effects (font (size 1.27 1.27)) (justify left))
+    )
+    (property "Footprint" "ao_tht:Board_Marker" (id 2) (at 209.55 72.39 0)
+      (effects (font (size 1.27 1.27)) hide)
+    )
+    (property "Datasheet" "" (id 3) (at 209.55 72.39 0)
+      (effects (font (size 1.27 1.27)) hide)
+    )
+    (property "Config" "DNF" (id 4) (at 209.55 72.39 0)
+      (effects (font (size 1.27 1.27)) hide)
+    )
+  )
 )

Commit message: Schematics tweaks, silk and fab cleanup, layout PDFs, panel revisions
Connections:
- net +10V_REF_P renamed +5V_REF_P
- net 0V renamed -5V_REF_P
Changed lines of the file:
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@@
     (effects (font (size 1.27 1.27)) (justify left bottom))
-  )
-  (hierarchical_label "0V" (shape input) (at 76.2 139.7 180)
-    (effects (font (size 1.27 1.27)) (justify right))
   )
   (hierarchical_label "OCTAVE_P" (shape output) (at 135.89 109.22 0)
     (effects (font (size 1.27 1.27)) (justify left))
+  )
+  (hierarchical_label "+5V_REF_P" (shape input) (at 76.2 63.5 180)
+    (effects (font (size 1.27 1.27)) (justify right))
+  )
+  (hierarchical_label "-5V_REF_P" (shape input) (at 76.2 139.7 180)
+    (effects (font (size 1.27 1.27)) (justify right))
   )
   (hierarchical_label "SOFT_SYNC_OFF_P" (shape output) (at 198.12 110.49 0)
@@
     (effects (font (size 1.27 1.27)) (justify left))
   )
-  (hierarchical_label "+10V_REF_P" (shape input) (at 76.2 63.5 180)
-    (effects (font (size 1.27 1.27)) (justify right))
-  )
   (hierarchical_label "SOFT_SYNCA_P" (shape output) (at 190.5 101.6 0)

Commit message: 100k in octave switch; rotary footprint; note stuff to fix
Parts:
- R32, R33, R34, R35, R36, R37, R38, R39, R40, R41: value 10k 1/8W -> 100k 1/8W
Changed lines of the file:
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@@
       (effects (font (size 1.27 1.27)) (justify left))
     )
-    (property "Value" "10k 1/8W" (id 1) (at 86.36 82.55 0)
+    (property "Value" "100k 1/8W" (id 1) (at 86.36 82.55 0)
       (effects (font (size 1.27 1.27)) (justify left))
     )
@@
       (effects (font (size 1.27 1.27)) (justify left))
     )
-    (property "Value" "10k 1/8W" (id 1) (at 86.36 90.17 0)
+    (property "Value" "100k 1/8W" (id 1) (at 86.36 90.17 0)
       (effects (font (size 1.27 1.27)) (justify left))
     )
@@
       (effects (font (size 1.27 1.27)) (justify left))
     )
-    (property "Value" "10k 1/8W" (id 1) (at 86.36 97.79 0)
+    (property "Value" "100k 1/8W" (id 1) (at 86.36 97.79 0)
       (effects (font (size 1.27 1.27)) (justify left))
     )
@@
       (effects (font (size 1.27 1.27)) (justify left))
     )
-    (property "Value" "10k 1/8W" (id 1) (at 86.36 105.41 0)
+    (property "Value" "100k 1/8W" (id 1) (at 86.36 105.41 0)
       (effects (font (size 1.27 1.27)) (justify left))
     )
@@
       (effects (font (size 1.27 1.27)) (justify left))
     )
-    (property "Value" "10k 1/8W" (id 1) (at 86.36 113.03 0)
+    (property "Value" "100k 1/8W" (id 1) (at 86.36 113.03 0)
       (effects (font (size 1.27 1.27)) (justify left))
     )
@@
       (effects (font (size 1.27 1.27)) (justify left))
     )
-    (property "Value" "10k 1/8W" (id 1) (at 86.36 120.65 0)
+    (property "Value" "100k 1/8W" (id 1) (at 86.36 120.65 0)
       (effects (font (size 1.27 1.27)) (justify left))
     )
@@
       (effects (font (size 1.27 1.27)) (justify left))
     )
-    (property "Value" "10k 1/8W" (id 1) (at 86.36 128.27 0)
+    (property "Value" "100k 1/8W" (id 1) (at 86.36 128.27 0)
       (effects (font (size 1.27 1.27)) (justify left))
     )
@@
       (effects (font (size 1.27 1.27)) (justify left))
     )
-    (property "Value" "10k 1/8W" (id 1) (at 86.36 135.89 0)
+    (property "Value" "100k 1/8W" (id 1) (at 86.36 135.89 0)
       (effects (font (size 1.27 1.27)) (justify left))
     )
@@
       (effects (font (size 1.27 1.27)) (justify left))
     )
-    (property "Value" "10k 1/8W" (id 1) (at 86.36 67.31 0)
+    (property "Value" "100k 1/8W" (id 1) (at 86.36 67.31 0)
       (effects (font (size 1.27 1.27)) (justify left))
     )
@@
       (effects (font (size 1.27 1.27)) (justify left))
     )
-    (property "Value" "10k 1/8W" (id 1) (at 86.36 74.93 0)
-      (effects (font (size 1.27 1.27)) (justify left))
-    )
+    (property "Value" "100k 1/8W" (id 1) (at 86.36 74.93 0)
+      (effects (font (size 1.27 1.27)) (justify left))
+    )

Commit message: Correct slide switch footprint; use TO-92 wide for regulator
Connections:
- net HARD_SYNCA_P: now also SW2.5; no longer SW2.1
- net SOFT_SYNCA_P: now also SW2.2, SW2.8; no longer SW2.4, SW2.6
- net SOFT_SYNC_OFF_P: now also SW2.1, SW2.3; no longer SW2.5, SW2.7
- net SYNCA_P: now also SW2.6; no longer SW2.2
Other:
- moved on the sheet: SW2A, SW2B
Changed lines of the file:
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@@
     (pin "2")
   )
-  (symbol (lib_name "SW_DP3T_1") (lib_id "herovco:SW_DP3T") (at 175.26 99.06 0) (unit 1)
+  (symbol (lib_name "SW_DP3T_1") (lib_id "herovco:SW_DP3T") (at 187.96 113.03 0) (unit 1)
     (in_bom yes) (on_board yes) (fields_autoplaced)
-    (property "Reference" "SW2" (id 0) (at 175.26 92.2233 0))
-    (property "Value" "SW_DP3T" (id 1) (at 175.26 94.9984 0))
-    (property "Footprint" "herovco:SW_CK_OS203012MU5QP1_DP3T" (id 2) (at 159.385 94.615 0)
+    (property "Reference" "SW2" (id 0) (at 187.96 106.1933 0))
+    (property "Value" "SW_DP3T" (id 1) (at 187.96 108.9684 0))
+    (property "Footprint" "herovco:SW_CK_OS203012MU5QP1_DP3T" (id 2) (at 172.085 108.585 0)
       (effects (font (size 1.27 1.27)) hide)
     )
-    (property "Datasheet" "~" (id 3) (at 159.385 94.615 0)
+    (property "Datasheet" "~" (id 3) (at 172.085 108.585 0)
       (effects (font (size 1.27 1.27)) hide)
     )
-    (property "Manufacturer" "C&K" (id 4) (at 175.26 99.06 0)
+    (property "Manufacturer" "C&K" (id 4) (at 187.96 113.03 0)
       (effects (font (size 1.27 1.27)) hide)
     )
-    (property "Part" "OS203012MU5QP1‎" (id 5) (at 175.26 99.06 0)
+    (property "Part" "OS203012MU5QP1‎" (id 5) (at 187.96 113.03 0)
       (effects (font (size 1.27 1.27)) hide)
     )
-    (property "Vendor" "Digi-Key" (id 6) (at 175.26 99.06 0)
+    (property "Vendor" "Digi-Key" (id 6) (at 187.96 113.03 0)
       (effects (font (size 1.27 1.27)) hide)
     )
-    (property "SKU" "CKN9554-ND" (id 7) (at 175.26 99.06 0)
+    (property "SKU" "CKN9554-ND" (id 7) (at 187.96 113.03 0)
       (effects (font (size 1.27 1.27)) hide)
     )
@@
     (pin "2")
   )
-  (symbol (lib_id "herovco:SW_DP3T") (at 187.96 113.03 0) (unit 2)
+  (symbol (lib_id "herovco:SW_DP3T") (at 175.26 99.06 0) (unit 2)
     (in_bom yes) (on_board yes) (fields_autoplaced)
-    (property "Reference" "SW2" (id 0) (at 187.96 106.1933 0))
-    (property "Value" "SW_DP3T" (id 1) (at 187.96 108.9684 0))
-    (property "Footprint" "herovco:SW_CK_OS203012MU5QP1_DP3T" (id 2) (at 172.085 108.585 0)
+    (property "Reference" "SW2" (id 0) (at 175.26 92.2233 0))
+    (property "Value" "SW_DP3T" (id 1) (at 175.26 94.9984 0))
+    (property "Footprint" "herovco:SW_CK_OS203012MU5QP1_DP3T" (id 2) (at 159.385 94.615 0)
       (effects (font (size 1.27 1.27)) hide)
     )
-    (property "Datasheet" "~" (id 3) (at 172.085 108.585 0)
+    (property "Datasheet" "~" (id 3) (at 159.385 94.615 0)
       (effects (font (size 1.27 1.27)) hide)
     )
-    (property "Manufacturer" "C&K" (id 4) (at 187.96 113.03 0)
+    (property "Manufacturer" "C&K" (id 4) (at 175.26 99.06 0)
       (effects (font (size 1.27 1.27)) hide)
     )
-    (property "Part" "OS203012MU5QP1‎" (id 5) (at 187.96 113.03 0)
+    (property "Part" "OS203012MU5QP1‎" (id 5) (at 175.26 99.06 0)
       (effects (font (size 1.27 1.27)) hide)
     )
-    (property "Vendor" "Digi-Key" (id 6) (at 187.96 113.03 0)
+    (property "Vendor" "Digi-Key" (id 6) (at 175.26 99.06 0)
       (effects (font (size 1.27 1.27)) hide)
     )
-    (property "SKU" "CKN9554-ND" (id 7) (at 187.96 113.03 0)
+    (property "SKU" "CKN9554-ND" (id 7) (at 175.26 99.06 0)
       (effects (font (size 1.27 1.27)) hide)
     )

Commit message: 10k resistors in octave switch
Parts:
- R32, R33, R34, R35, R36, R37, R38, R39, R40, R41: value 100k 1/8W -> 10k 1/8W
Changed lines of the file:
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@@
       (effects (font (size 1.27 1.27)) (justify left))
     )
-    (property "Value" "100k 1/8W" (id 1) (at 86.36 82.55 0)
+    (property "Value" "10k 1/8W" (id 1) (at 86.36 82.55 0)
       (effects (font (size 1.27 1.27)) (justify left))
     )
@@
       (effects (font (size 1.27 1.27)) (justify left))
     )
-    (property "Value" "100k 1/8W" (id 1) (at 86.36 90.17 0)
+    (property "Value" "10k 1/8W" (id 1) (at 86.36 90.17 0)
       (effects (font (size 1.27 1.27)) (justify left))
     )
@@
       (effects (font (size 1.27 1.27)) (justify left))
     )
-    (property "Value" "100k 1/8W" (id 1) (at 86.36 97.79 0)
+    (property "Value" "10k 1/8W" (id 1) (at 86.36 97.79 0)
       (effects (font (size 1.27 1.27)) (justify left))
     )
@@
       (effects (font (size 1.27 1.27)) (justify left))
     )
-    (property "Value" "100k 1/8W" (id 1) (at 86.36 105.41 0)
+    (property "Value" "10k 1/8W" (id 1) (at 86.36 105.41 0)
       (effects (font (size 1.27 1.27)) (justify left))
     )
@@
       (effects (font (size 1.27 1.27)) (justify left))
     )
-    (property "Value" "100k 1/8W" (id 1) (at 86.36 113.03 0)
+    (property "Value" "10k 1/8W" (id 1) (at 86.36 113.03 0)
       (effects (font (size 1.27 1.27)) (justify left))
     )
@@
       (effects (font (size 1.27 1.27)) (justify left))
     )
-    (property "Value" "100k 1/8W" (id 1) (at 86.36 120.65 0)
+    (property "Value" "10k 1/8W" (id 1) (at 86.36 120.65 0)
       (effects (font (size 1.27 1.27)) (justify left))
     )
@@
       (effects (font (size 1.27 1.27)) (justify left))
     )
-    (property "Value" "100k 1/8W" (id 1) (at 86.36 128.27 0)
+    (property "Value" "10k 1/8W" (id 1) (at 86.36 128.27 0)
       (effects (font (size 1.27 1.27)) (justify left))
     )
@@
       (effects (font (size 1.27 1.27)) (justify left))
     )
-    (property "Value" "100k 1/8W" (id 1) (at 86.36 135.89 0)
+    (property "Value" "10k 1/8W" (id 1) (at 86.36 135.89 0)
       (effects (font (size 1.27 1.27)) (justify left))
     )
@@
       (effects (font (size 1.27 1.27)) (justify left))
     )
-    (property "Value" "100k 1/8W" (id 1) (at 86.36 67.31 0)
+    (property "Value" "10k 1/8W" (id 1) (at 86.36 67.31 0)
       (effects (font (size 1.27 1.27)) (justify left))
     )
@@
       (effects (font (size 1.27 1.27)) (justify left))
     )
-    (property "Value" "100k 1/8W" (id 1) (at 86.36 74.93 0)
-      (effects (font (size 1.27 1.27)) (justify left))
-    )
+    (property "Value" "10k 1/8W" (id 1) (at 86.36 74.93 0)
+      (effects (font (size 1.27 1.27)) (justify left))
+    )
