File: Hardware/PCB/herovco/jackspower.kicad_sch (KiCad schematic)
At the start: 25 parts, among them J10 AudioJack2, J11 AudioJack2, J12 AudioJack2, J13 AudioJack2, J14 AudioJack2, J15 Synth_power_2x5, J16 AudioJack2, J17 AudioJack2, J18 AudioJack2, J19 AudioJack2, J20 AudioJack2

Commit message: Change pot symbols and fix orientation, other small tweaks
Parts:
- C16, C17: footprint ao_tht:CP_Radial_D5.0mm_P2.00mm -> ao_tht:CP_Radial_D6.3mm_P2.50mm
- J15: SKU (none) -> A-2939; Vendor (none) -> Tayda
Changed lines of the file:
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@@
     (pin "1")
   )
-  (symbol (lib_id "ao_symbols:CP") (at 163.83 137.16 0)
+  (symbol (lib_id "ao_symbols:CP") (at 163.83 137.16 0) (unit 1)
     (in_bom yes) (on_board yes)
     (property "Reference" "C16" (id 0) (at 166.8272 135.9916 0)
@@
       (effects (font (size 1.27 1.27)) (justify left))
     )
-    (property "Footprint" "ao_tht:CP_Radial_D5.0mm_P2.00mm" (id 2) (at 164.7952 140.97 0)
+    (property "Footprint" "ao_tht:CP_Radial_D6.3mm_P2.50mm" (id 2) (at 164.7952 140.97 0)
       (effects (font (size 1.27 1.27)) hide)
     )
@@
     (pin "2")
   )
-  (symbol (lib_id "ao_symbols:CP") (at 163.83 144.78 0)
+  (symbol (lib_id "ao_symbols:CP") (at 163.83 144.78 0) (unit 1)
     (in_bom yes) (on_board yes)
     (property "Reference" "C17" (id 0) (at 166.8272 143.6116 0)
@@
       (effects (font (size 1.27 1.27)) (justify left))
     )
-    (property "Footprint" "ao_tht:CP_Radial_D5.0mm_P2.00mm" (id 2) (at 164.7952 148.59 0)
+    (property "Footprint" "ao_tht:CP_Radial_D6.3mm_P2.50mm" (id 2) (at 164.7952 148.59 0)
       (effects (font (size 1.27 1.27)) hide)
     )
@@
     (property "Datasheet" "" (id 3) (at 97.155 140.97 0)
       (effects (font (size 1.524 1.524)) hide)
+    )
+    (property "Vendor" "Tayda" (id 4) (at 97.155 140.97 0)
+      (effects (font (size 1.27 1.27)) hide)
+    )
+    (property "SKU" "A-2939" (id 5) (at 97.155 140.97 0)
+      (effects (font (size 1.27 1.27)) hide)
     )
     (pin "1")
@@
     (pin "2")
   )
-  (symbol (lib_id "Diode:1N5817") (at 123.19 135.89 180) (unit 1)
+  (symbol (lib_name "1N5817_1") (lib_id "Diode:1N5817") (at 123.19 135.89 180) (unit 1)
     (in_bom yes) (on_board yes)
     (property "Reference" "D3" (id 0) (at 123.19 130.3782 0))
@@
     (pin "1")
   )
-  (symbol (lib_id "ao_symbols:+12V_1") (at 143.51 135.89 0)
+  (symbol (lib_id "ao_symbols:+12V_1") (at 143.51 135.89 0) (unit 1)
     (in_bom yes) (on_board yes)
     (property "Reference" "#PWR073" (id 0) (at 143.51 139.7 0)
@@
     (pin "1")
   )
-  (symbol (lib_id "ao_symbols:+12V_1") (at 163.83 133.35 0)
+  (symbol (lib_id "ao_symbols:+12V_1") (at 163.83 133.35 0) (unit 1)
     (in_bom yes) (on_board yes)
     (property "Reference" "#PWR076" (id 0) (at 163.83 137.16 0)
@@
     (pin "1")
   )
-  (symbol (lib_id "ao_symbols:-12V_1") (at 143.51 146.05 0)
+  (symbol (lib_id "ao_symbols:-12V_1") (at 143.51 146.05 0) (unit 1)
     (in_bom yes) (on_board yes)
     (property "Reference" "#PWR074" (id 0) (at 143.51 143.51 0)
@@
     (pin "1")
   )
-  (symbol (lib_id "ao_symbols:-12V_1") (at 163.83 148.59 180)
+  (symbol (lib_id "ao_symbols:-12V_1") (at 163.83 148.59 180) (unit 1)
     (in_bom yes) (on_board yes)
     (property "Reference" "#PWR077" (id 0) (at 163.83 151.13 0)
@@
     (pin "1")
   )
-  (symbol (lib_id "ao_symbols:+12V_1") (at 104.14 160.02 90)
+  (symbol (lib_id "ao_symbols:+12V_1") (at 104.14 160.02 90) (unit 1)
     (in_bom yes) (on_board yes)
     (property "Reference" "#PWR078" (id 0) (at 107.95 160.02 0)
@@
     (pin "1")
   )
-  (symbol (lib_id "ao_symbols:-12V_1") (at 123.19 160.02 90)
+  (symbol (lib_id "ao_symbols:-12V_1") (at 123.19 160.02 90) (unit 1)
     (in_bom yes) (on_board yes)
     (property "Reference" "#PWR079" (id 0) (at 120.65 160.02 0)
@@
     (pin "1")
   )
-  (symbol (lib_id "ao_symbols:+12V_1") (at 35.56 60.96 0)
+  (symbol (lib_id "ao_symbols:+12V_1") (at 35.56 60.96 0) (unit 1)
     (in_bom yes) (on_board yes)
     (property "Reference" "#PWR059" (id 0) (at 35.56 64.77 0)
@@
     (pin "1")
   )
-  (symbol (lib_id "ao_symbols:-12V_1") (at 35.56 71.12 0)
+  (symbol (lib_id "ao_symbols:-12V_1") (at 35.56 71.12 0) (unit 1)
     (in_bom yes) (on_board yes)
     (property "Reference" "#PWR060" (id 0) (at 35.56 68.58 0)

Commit message: Pre-breadboard updates
Parts:
- B2: Config (none) -> DNF
- D3, D4: footprint Diode_THT:D_DO-41_SOD81_P10.16mm_Horizontal -> ao_tht:D_DO-41_SOD81_P10.16mm_Horizontal; symbol Diode:1N5817 -> ao_symbols:1N5817; SKU (none) -> A-159; Vendor (none) -> Tayda
- J10, J11, J12, J13, J14, J16, J17, J18, J19, J20: footprint ao_tht:Jack_6.35mm_PJ_629HAN_slots -> ao_tht:Jack_6.35mm_PJ_629HAN; symbol Connector:AudioJack2 -> ao_symbols:AudioJack2; SKU (none) -> A-1121; Vendor (none) -> Tayda
Other:
- note removed: "HEADERS"
- moved on the sheet: TP5, TP6, TP7

Commit message: Panel updates; reannotate; correct PCB errors
Parts:
- renumbered C16 to C13, C17 to C14, D3 to D2, D4 to D3, TP5 to TP4, TP6 to TP5, TP7 to TP6
Changed lines of the file:
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@@
   (symbol (lib_id "power:GND1") (at 119.38 44.45 0) (unit 1)
     (in_bom yes) (on_board yes)
-    (property "Reference" "#PWR068" (id 0) (at 119.38 50.8 0)
+    (property "Reference" "#PWR051" (id 0) (at 119.38 50.8 0)
       (effects (font (size 1.27 1.27)) hide)
     )
@@
   (symbol (lib_id "power:GND1") (at 119.38 56.515 0) (unit 1)
     (in_bom yes) (on_board yes)
-    (property "Reference" "#PWR069" (id 0) (at 119.38 62.865 0)
+    (property "Reference" "#PWR052" (id 0) (at 119.38 62.865 0)
       (effects (font (size 1.27 1.27)) hide)
     )
@@
   (symbol (lib_id "power:GND1") (at 119.38 68.58 0) (unit 1)
     (in_bom yes) (on_board yes)
-    (property "Reference" "#PWR070" (id 0) (at 119.38 74.93 0)
+    (property "Reference" "#PWR053" (id 0) (at 119.38 74.93 0)
       (effects (font (size 1.27 1.27)) hide)
     )
@@
   (symbol (lib_id "power:GND1") (at 119.38 80.645 0) (unit 1)
     (in_bom yes) (on_board yes)
-    (property "Reference" "#PWR071" (id 0) (at 119.38 86.995 0)
+    (property "Reference" "#PWR054" (id 0) (at 119.38 86.995 0)
       (effects (font (size 1.27 1.27)) hide)
     )
@@
   (symbol (lib_id "power:GND1") (at 95.25 44.45 0) (mirror y) (unit 1)
     (in_bom yes) (on_board yes)
-    (property "Reference" "#PWR062" (id 0) (at 95.25 50.8 0)
+    (property "Reference" "#PWR044" (id 0) (at 95.25 50.8 0)
       (effects (font (size 1.27 1.27)) hide)
     )
@@
   (symbol (lib_id "power:GND1") (at 95.25 56.515 0) (mirror y) (unit 1)
     (in_bom yes) (on_board yes)
-    (property "Reference" "#PWR063" (id 0) (at 95.25 62.865 0)
+    (property "Reference" "#PWR045" (id 0) (at 95.25 62.865 0)
       (effects (font (size 1.27 1.27)) hide)
     )
@@
   (symbol (lib_id "power:GND1") (at 95.25 68.58 0) (mirror y) (unit 1)
     (in_bom yes) (on_board yes)
-    (property "Reference" "#PWR064" (id 0) (at 95.25 74.93 0)
+    (property "Reference" "#PWR046" (id 0) (at 95.25 74.93 0)
       (effects (font (size 1.27 1.27)) hide)
     )
@@
   (symbol (lib_id "power:GND1") (at 95.25 80.645 0) (mirror y) (unit 1)
     (in_bom yes) (on_board yes)
-    (property "Reference" "#PWR065" (id 0) (at 95.25 86.995 0)
+    (property "Reference" "#PWR047" (id 0) (at 95.25 86.995 0)
       (effects (font (size 1.27 1.27)) hide)
     )
@@
   (symbol (lib_id "power:GND1") (at 95.25 92.71 0) (mirror y) (unit 1)
     (in_bom yes) (on_board yes)
-    (property "Reference" "#PWR066" (id 0) (at 95.25 99.06 0)
+    (property "Reference" "#PWR048" (id 0) (at 95.25 99.06 0)
       (effects (font (size 1.27 1.27)) hide)
     )
@@
   (symbol (lib_id "ao_symbols:CP") (at 163.83 137.16 0) (unit 1)
     (in_bom yes) (on_board yes)
-    (property "Reference" "C16" (id 0) (at 166.8272 135.9916 0)
+    (property "Reference" "C13" (id 0) (at 166.8272 135.9916 0)
       (effects (font (size 1.27 1.27)) (justify left))
     )
@@
   (symbol (lib_id "ao_symbols:CP") (at 163.83 144.78 0) (unit 1)
     (in_bom yes) (on_board yes)
-    (property "Reference" "C17" (id 0) (at 166.8272 143.6116 0)
+    (property "Reference" "C14" (id 0) (at 166.8272 143.6116 0)
       (effects (font (size 1.27 1.27)) (justify left))
     )
@@
   (symbol (lib_id "ao_symbols:1N5817") (at 123.19 146.05 0) (unit 1)
     (in_bom yes) (on_board yes)
-    (property "Reference" "D4" (id 0) (at 123.19 140.5382 0))
+    (property "Reference" "D3" (id 0) (at 123.19 140.5382 0))
     (property "Value" "1N5817" (id 1) (at 123.19 142.8496 0))
     (property "Footprint" "ao_tht:D_DO-41_SOD81_P10.16mm_Horizontal" (id 2) (at 123.19 150.495 0)
@@
   (symbol (lib_id "ao_symbols:1N5817") (at 123.19 135.89 180) (unit 1)
     (in_bom yes) (on_board yes)
-    (property "Reference" "D3" (id 0) (at 123.19 130.3782 0))
+    (property "Reference" "D2" (id 0) (at 123.19 130.3782 0))
     (property "Value" "1N5817" (id 1) (at 123.19 132.6896 0))
     (property "Footprint" "ao_tht:D_DO-41_SOD81_P10.16mm_Horizontal" (id 2) (at 123.19 131.445 0)
@@
   (symbol (lib_id "power:GND1") (at 133.35 93.345 0) (mirror y) (unit 1)
     (in_bom yes) (on_board yes)
-    (property "Reference" "#PWR072" (id 0) (at 133.35 99.695 0)
+    (property "Reference" "#PWR056" (id 0) (at 133.35 99.695 0)
       (effects (font (size 1.27 1.27)) hide)
     )
@@
   (symbol (lib_id "power:GND1") (at 78.74 140.97 270) (mirror x) (unit 1)
     (in_bom yes) (on_board yes)
-    (property "Reference" "#PWR061" (id 0) (at 72.39 140.97 0)
+    (property "Reference" "#PWR043" (id 0) (at 72.39 140.97 0)
       (effects (font (size 1.27 1.27)) hide)
     )
@@
   (symbol (lib_id "power:GND1") (at 108.585 140.97 90) (mirror x) (unit 1)
     (in_bom yes) (on_board yes)
-    (property "Reference" "#PWR067" (id 0) (at 114.935 140.97 0)
+    (property "Reference" "#PWR050" (id 0) (at 114.935 140.97 0)
       (effects (font (size 1.27 1.27)) hide)
     )
@@
   (symbol (lib_id "power:GND1") (at 156.21 142.24 0) (mirror y) (unit 1)
     (in_bom yes) (on_board yes)
-    (property "Reference" "#PWR075" (id 0) (at 156.21 148.59 0)
+    (property "Reference" "#PWR060" (id 0) (at 156.21 148.59 0)
       (effects (font (size 1.27 1.27)) hide)
     )
@@
   (symbol (lib_id "ao_symbols:+12V_1") (at 143.51 135.89 0) (unit 1)
     (in_bom yes) (on_board yes)
-    (property "Reference" "#PWR073" (id 0) (at 143.51 139.7 0)
+    (property "Reference" "#PWR058" (id 0) (at 143.51 139.7 0)
       (effects (font (size 1.27 1.27)) hide)
     )
@@
   (symbol (lib_id "ao_symbols:+12V_1") (at 163.83 133.35 0) (unit 1)
     (in_bom yes) (on_board yes)
-    (property "Reference" "#PWR076" (id 0) (at 163.83 137.16 0)
+    (property "Reference" "#PWR061" (id 0) (at 163.83 137.16 0)
       (effects (font (size 1.27 1.27)) hide)
     )
@@
   (symbol (lib_id "ao_symbols:-12V_1") (at 143.51 146.05 0) (unit 1)
     (in_bom yes) (on_board yes)
-    (property "Reference" "#PWR074" (id 0) (at 143.51 143.51 0)
+    (property "Reference" "#PWR059" (id 0) (at 143.51 143.51 0)
       (effects (font (size 1.27 1.27)) hide)
     )
@@
   (symbol (lib_id "ao_symbols:-12V_1") (at 163.83 148.59 180) (unit 1)
     (in_bom yes) (on_board yes)
-    (property "Reference" "#PWR077" (id 0) (at 163.83 151.13 0)
+    (property "Reference" "#PWR062" (id 0) (at 163.83 151.13 0)
       (effects (font (size 1.27 1.27)) hide)
     )
@@
   (symbol (lib_id "Connector:TestPoint") (at 104.14 156.21 0) (unit 1)
     (in_bom yes) (on_board yes)
-    (property "Reference" "TP5" (id 0) (at 105.6132 153.2128 0)
+    (property "Reference" "TP4" (id 0) (at 105.6132 153.2128 0)
       (effects (font (size 1.27 1.27)) (justify left))
     )
@@
   (symbol (lib_id "Connector:TestPoint") (at 123.19 156.21 0) (unit 1)
     (in_bom yes) (on_board yes)
-    (property "Reference" "TP6" (id 0) (at 124.6632 153.2128 0)
+    (property "Reference" "TP5" (id 0) (at 124.6632 153.2128 0)
       (effects (font (size 1.27 1.27)) (justify left))
     )
@@
   (symbol (lib_id "Connector:TestPoint") (at 142.24 156.21 0) (unit 1)
     (in_bom yes) (on_board yes)
-    (property "Reference" "TP7" (id 0) (at 143.7132 153.2128 0)
+    (property "Reference" "TP6" (id 0) (at 143.7132 153.2128 0)
       (effects (font (size 1.27 1.27)) (justify left))
     )
@@
   (symbol (lib_id "ao_symbols:+12V_1") (at 104.14 156.21 90) (unit 1)
     (in_bom yes) (on_board yes)
-    (property "Reference" "#PWR078" (id 0) (at 107.95 156.21 0)
+    (property "Reference" "#PWR049" (id 0) (at 107.95 156.21 0)
       (effects (font (size 1.27 1.27)) hide)
     )
@@
   (symbol (lib_id "ao_symbols:-12V_1") (at 123.19 156.21 90) (unit 1)
     (in_bom yes) (on_board yes)
-    (property "Reference" "#PWR079" (id 0) (at 120.65 156.21 0)
+    (property "Reference" "#PWR055" (id 0) (at 120.65 156.21 0)
       (effects (font (size 1.27 1.27)) hide)
     )
@@
   (symbol (lib_id "power:GND1") (at 142.24 156.21 270) (mirror x) (unit 1)
     (in_bom yes) (on_board yes)
-    (property "Reference" "#PWR080" (id 0) (at 135.89 156.21 0)
-      (effects (font (size 1.27 1.27)) hide)
-    )
+    (property "Reference" "#PWR057" (id 0) (at 135.89 156.21 0)
+      (effects (font (size 1.27 1.27)) hide)
+    )

Commit message: Sync input revision
Parts:
- renumbered C13 to C14, C14 to C15, D2 to D3, D3 to D4, J10 to J12, J11 to J13, J12 to J14, J13 to J15, J14 to J16, J15 to J17, J16 to J18, J17 to J19, J18 to J20, J19 to J21, J20 to J22

Commit message: Big panel and PCB revisions
Parts:
- renumbered J12 to J14, J13 to J15, J14 to J16, J15 to J17, J16 to J18, J17 to J19, J18 to J20, J19 to J21, J20 to J22, J21 to J23, J22 to J24
Changed lines of the file:
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@@
   (symbol (lib_id "ao_symbols:AudioJack2") (at 125.73 40.64 180) (unit 1)
     (in_bom yes) (on_board yes)
-    (property "Reference" "J18" (id 0) (at 130.302 40.2082 0)
+    (property "Reference" "J20" (id 0) (at 130.302 40.2082 0)
       (effects (font (size 1.27 1.27)) (justify right))
     )
@@
   (symbol (lib_id "ao_symbols:AudioJack2") (at 125.73 52.705 180) (unit 1)
     (in_bom yes) (on_board yes)
-    (property "Reference" "J19" (id 0) (at 130.302 52.2732 0)
+    (property "Reference" "J21" (id 0) (at 130.302 52.2732 0)
       (effects (font (size 1.27 1.27)) (justify right))
     )
@@
   (symbol (lib_id "ao_symbols:AudioJack2") (at 125.73 64.77 180) (unit 1)
     (in_bom yes) (on_board yes)
-    (property "Reference" "J20" (id 0) (at 130.302 64.3382 0)
+    (property "Reference" "J22" (id 0) (at 130.302 64.3382 0)
       (effects (font (size 1.27 1.27)) (justify right))
     )
@@
   (symbol (lib_id "ao_symbols:AudioJack2") (at 125.73 76.835 180) (unit 1)
     (in_bom yes) (on_board yes)
-    (property "Reference" "J21" (id 0) (at 130.302 76.4032 0)
+    (property "Reference" "J23" (id 0) (at 130.302 76.4032 0)
       (effects (font (size 1.27 1.27)) (justify right))
     )
@@
   (symbol (lib_id "ao_symbols:AudioJack2") (at 88.9 40.64 0) (mirror x) (unit 1)
     (in_bom yes) (on_board yes)
-    (property "Reference" "J12" (id 0) (at 84.328 40.2082 0)
+    (property "Reference" "J14" (id 0) (at 84.328 40.2082 0)
       (effects (font (size 1.27 1.27)) (justify right))
     )
@@
   (symbol (lib_id "ao_symbols:AudioJack2") (at 88.9 52.705 0) (mirror x) (unit 1)
     (in_bom yes) (on_board yes)
-    (property "Reference" "J13" (id 0) (at 84.328 52.2732 0)
+    (property "Reference" "J15" (id 0) (at 84.328 52.2732 0)
       (effects (font (size 1.27 1.27)) (justify right))
     )
@@
   (symbol (lib_id "ao_symbols:AudioJack2") (at 88.9 64.77 0) (mirror x) (unit 1)
     (in_bom yes) (on_board yes)
-    (property "Reference" "J14" (id 0) (at 84.328 64.3382 0)
+    (property "Reference" "J16" (id 0) (at 84.328 64.3382 0)
       (effects (font (size 1.27 1.27)) (justify right))
     )
@@
   (symbol (lib_id "ao_symbols:AudioJack2") (at 88.9 76.835 0) (mirror x) (unit 1)
     (in_bom yes) (on_board yes)
-    (property "Reference" "J15" (id 0) (at 84.328 76.4032 0)
+    (property "Reference" "J17" (id 0) (at 84.328 76.4032 0)
       (effects (font (size 1.27 1.27)) (justify right))
     )
@@
   (symbol (lib_id "ao_symbols:AudioJack2") (at 88.9 88.9 0) (mirror x) (unit 1)
     (in_bom yes) (on_board yes)
-    (property "Reference" "J16" (id 0) (at 84.328 88.4682 0)
+    (property "Reference" "J18" (id 0) (at 84.328 88.4682 0)
       (effects (font (size 1.27 1.27)) (justify right))
     )
@@
   (symbol (lib_id "ao_symbols:Synth_power_2x5") (at 97.155 140.97 0) (unit 1)
     (in_bom yes) (on_board yes)
-    (property "Reference" "J17" (id 0) (at 97.155 129.6162 0)
+    (property "Reference" "J19" (id 0) (at 97.155 129.6162 0)
       (effects (font (size 1.524 1.524)))
     )
@@
   (symbol (lib_id "ao_symbols:AudioJack2") (at 127 89.535 0) (mirror x) (unit 1)
     (in_bom yes) (on_board yes)
-    (property "Reference" "J22" (id 0) (at 122.428 89.1032 0)
-      (effects (font (size 1.27 1.27)) (justify right))
-    )
+    (property "Reference" "J24" (id 0) (at 122.428 89.1032 0)
+      (effects (font (size 1.27 1.27)) (justify right))
+    )
