File: Hardware/PCB/herovco/jackspower.kicad_sch (KiCad schematic)
At the start: 25 parts, among them J14 AudioJack2, J15 AudioJack2, J16 AudioJack2, J17 AudioJack2, J18 AudioJack2, J19 Synth_power_2x5, J20 AudioJack2, J21 AudioJack2, J22 AudioJack2, J23 AudioJack2, J24 AudioJack2

Commit message: Sch cleanup, switch footprint
Changed lines of the file:
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@@
     (stroke (width 0) (type default) (color 0 0 0 0))
   )
-  (polyline (pts (xy 67.31 170.18) (xy 175.26 170.18))
+  (polyline (pts (xy 67.31 162.56) (xy 175.26 162.56))
     (stroke (width 0) (type default) (color 0 0 0 0))
   )
@@
     (stroke (width 0) (type default) (color 0 0 0 0))
   )
-  (polyline (pts (xy 67.31 25.4) (xy 67.31 170.18))
+  (polyline (pts (xy 67.31 25.4) (xy 67.31 162.56))
     (stroke (width 0) (type default) (color 0 0 0 0))
   )
@@
     (stroke (width 0) (type default) (color 0 0 0 0))
   )
-  (polyline (pts (xy 175.26 113.03) (xy 175.26 170.18))
+  (polyline (pts (xy 175.26 113.03) (xy 175.26 162.56))
     (stroke (width 0) (type default) (color 0 0 0 0))
   )
@@
     )
   )
-  (hierarchical_label "-12V_BACK" (shape input) (at 123.19 156.21 270)
-    (effects (font (size 1.27 1.27)) (justify right))
-  )
   (hierarchical_label "V_OCT_J" (shape output) (at 95.25 88.9 0)
     (effects (font (size 1.27 1.27)) (justify left))
@@
     (effects (font (size 1.27 1.27)) (justify right))
   )
-  (hierarchical_label "GND_BACK" (shape input) (at 142.24 156.21 270)
-    (effects (font (size 1.27 1.27)) (justify right))
-  )
   (hierarchical_label "PWMIN_J" (shape output) (at 95.25 40.64 0)
     (effects (font (size 1.27 1.27)) (justify left))
@@
     (effects (font (size 1.27 1.27)) (justify left))
   )
-  (hierarchical_label "+12V_BACK" (shape input) (at 104.14 156.21 270)
-    (effects (font (size 1.27 1.27)) (justify right))
-  )
   (hierarchical_label "V_OCT2_J" (shape output) (at 133.35 89.535 0)
     (effects (font (size 1.27 1.27)) (justify left))
@@
   (symbol (lib_id "power:GND1") (at 119.38 44.45 0) (unit 1)
     (in_bom yes) (on_board yes)
-    (property "Reference" "#PWR053" (id 0) (at 119.38 50.8 0)
+    (property "Reference" "#PWR057" (id 0) (at 119.38 50.8 0)
       (effects (font (size 1.27 1.27)) hide)
     )
@@
   (symbol (lib_id "power:GND1") (at 119.38 56.515 0) (unit 1)
     (in_bom yes) (on_board yes)
-    (property "Reference" "#PWR054" (id 0) (at 119.38 62.865 0)
+    (property "Reference" "#PWR058" (id 0) (at 119.38 62.865 0)
       (effects (font (size 1.27 1.27)) hide)
     )
@@
   (symbol (lib_id "power:GND1") (at 119.38 68.58 0) (unit 1)
     (in_bom yes) (on_board yes)
-    (property "Reference" "#PWR055" (id 0) (at 119.38 74.93 0)
+    (property "Reference" "#PWR059" (id 0) (at 119.38 74.93 0)
       (effects (font (size 1.27 1.27)) hide)
     )
@@
   (symbol (lib_id "power:GND1") (at 119.38 80.645 0) (unit 1)
     (in_bom yes) (on_board yes)
-    (property "Reference" "#PWR056" (id 0) (at 119.38 86.995 0)
+    (property "Reference" "#PWR060" (id 0) (at 119.38 86.995 0)
       (effects (font (size 1.27 1.27)) hide)
     )
@@
   (symbol (lib_id "power:GND1") (at 95.25 44.45 0) (mirror y) (unit 1)
     (in_bom yes) (on_board yes)
-    (property "Reference" "#PWR046" (id 0) (at 95.25 50.8 0)
+    (property "Reference" "#PWR050" (id 0) (at 95.25 50.8 0)
       (effects (font (size 1.27 1.27)) hide)
     )
@@
   (symbol (lib_id "power:GND1") (at 95.25 56.515 0) (mirror y) (unit 1)
     (in_bom yes) (on_board yes)
-    (property "Reference" "#PWR047" (id 0) (at 95.25 62.865 0)
+    (property "Reference" "#PWR051" (id 0) (at 95.25 62.865 0)
       (effects (font (size 1.27 1.27)) hide)
     )
@@
   (symbol (lib_id "power:GND1") (at 95.25 68.58 0) (mirror y) (unit 1)
     (in_bom yes) (on_board yes)
-    (property "Reference" "#PWR048" (id 0) (at 95.25 74.93 0)
+    (property "Reference" "#PWR052" (id 0) (at 95.25 74.93 0)
       (effects (font (size 1.27 1.27)) hide)
     )
@@
   (symbol (lib_id "power:GND1") (at 95.25 80.645 0) (mirror y) (unit 1)
     (in_bom yes) (on_board yes)
-    (property "Reference" "#PWR049" (id 0) (at 95.25 86.995 0)
+    (property "Reference" "#PWR053" (id 0) (at 95.25 86.995 0)
       (effects (font (size 1.27 1.27)) hide)
     )
@@
   (symbol (lib_id "power:GND1") (at 95.25 92.71 0) (mirror y) (unit 1)
     (in_bom yes) (on_board yes)
-    (property "Reference" "#PWR050" (id 0) (at 95.25 99.06 0)
+    (property "Reference" "#PWR054" (id 0) (at 95.25 99.06 0)
       (effects (font (size 1.27 1.27)) hide)
     )
@@
   (symbol (lib_id "power:GND1") (at 133.35 93.345 0) (mirror y) (unit 1)
     (in_bom yes) (on_board yes)
-    (property "Reference" "#PWR058" (id 0) (at 133.35 99.695 0)
+    (property "Reference" "#PWR062" (id 0) (at 133.35 99.695 0)
       (effects (font (size 1.27 1.27)) hide)
     )
@@
   (symbol (lib_id "power:GND1") (at 78.74 140.97 270) (mirror x) (unit 1)
     (in_bom yes) (on_board yes)
-    (property "Reference" "#PWR045" (id 0) (at 72.39 140.97 0)
+    (property "Reference" "#PWR049" (id 0) (at 72.39 140.97 0)
       (effects (font (size 1.27 1.27)) hide)
     )
@@
   (symbol (lib_id "power:GND1") (at 108.585 140.97 90) (mirror x) (unit 1)
     (in_bom yes) (on_board yes)
-    (property "Reference" "#PWR052" (id 0) (at 114.935 140.97 0)
+    (property "Reference" "#PWR056" (id 0) (at 114.935 140.97 0)
       (effects (font (size 1.27 1.27)) hide)
     )
@@
   (symbol (lib_id "power:GND1") (at 156.21 142.24 0) (mirror y) (unit 1)
     (in_bom yes) (on_board yes)
-    (property "Reference" "#PWR062" (id 0) (at 156.21 148.59 0)
+    (property "Reference" "#PWR066" (id 0) (at 156.21 148.59 0)
       (effects (font (size 1.27 1.27)) hide)
     )
@@
   (symbol (lib_id "ao_symbols:+12V_1") (at 143.51 135.89 0) (unit 1)
     (in_bom yes) (on_board yes)
-    (property "Reference" "#PWR060" (id 0) (at 143.51 139.7 0)
+    (property "Reference" "#PWR064" (id 0) (at 143.51 139.7 0)
       (effects (font (size 1.27 1.27)) hide)
     )
@@
   (symbol (lib_id "ao_symbols:+12V_1") (at 163.83 133.35 0) (unit 1)
     (in_bom yes) (on_board yes)
-    (property "Reference" "#PWR063" (id 0) (at 163.83 137.16 0)
+    (property "Reference" "#PWR067" (id 0) (at 163.83 137.16 0)
       (effects (font (size 1.27 1.27)) hide)
     )
@@
   (symbol (lib_id "ao_symbols:-12V_1") (at 143.51 146.05 0) (unit 1)
     (in_bom yes) (on_board yes)
-    (property "Reference" "#PWR061" (id 0) (at 143.51 143.51 0)
+    (property "Reference" "#PWR065" (id 0) (at 143.51 143.51 0)
       (effects (font (size 1.27 1.27)) hide)
     )
@@
   (symbol (lib_id "ao_symbols:-12V_1") (at 163.83 148.59 180) (unit 1)
     (in_bom yes) (on_board yes)
-    (property "Reference" "#PWR064" (id 0) (at 163.83 151.13 0)
+    (property "Reference" "#PWR068" (id 0) (at 163.83 151.13 0)
       (effects (font (size 1.27 1.27)) hide)
     )
@@
   (symbol (lib_id "ao_symbols:+12V_1") (at 104.14 156.21 90) (unit 1)
     (in_bom yes) (on_board yes)
-    (property "Reference" "#PWR051" (id 0) (at 107.95 156.21 0)
+    (property "Reference" "#PWR055" (id 0) (at 107.95 156.21 0)
       (effects (font (size 1.27 1.27)) hide)
     )
@@
   (symbol (lib_id "ao_symbols:-12V_1") (at 123.19 156.21 90) (unit 1)
     (in_bom yes) (on_board yes)
-    (property "Reference" "#PWR057" (id 0) (at 120.65 156.21 0)
+    (property "Reference" "#PWR061" (id 0) (at 120.65 156.21 0)
       (effects (font (size 1.27 1.27)) hide)
     )
@@
   (symbol (lib_id "power:GND1") (at 142.24 156.21 270) (mirror x) (unit 1)
     (in_bom yes) (on_board yes)
-    (property "Reference" "#PWR059" (id 0) (at 135.89 156.21 0)
-      (effects (font (size 1.27 1.27)) hide)
-    )
+    (property "Reference" "#PWR063" (id 0) (at 135.89 156.21 0)
+      (effects (font (size 1.27 1.27)) hide)
+    )

Commit message: Different sync switch, other tweaks
Parts:
- renumbered J14 to J20, J15 to J21, J16 to J22, J17 to J23, J18 to J24, J19 to J25, J20 to J26, J21 to J27, J22 to J28, J23 to J29, J24 to J30
Changed lines of the file:
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@@
   (symbol (lib_id "ao_symbols:AudioJack2") (at 125.73 40.64 180) (unit 1)
     (in_bom yes) (on_board yes)
-    (property "Reference" "J20" (id 0) (at 130.302 40.2082 0)
+    (property "Reference" "J26" (id 0) (at 130.302 40.2082 0)
       (effects (font (size 1.27 1.27)) (justify right))
     )
@@
   (symbol (lib_id "ao_symbols:AudioJack2") (at 125.73 52.705 180) (unit 1)
     (in_bom yes) (on_board yes)
-    (property "Reference" "J21" (id 0) (at 130.302 52.2732 0)
+    (property "Reference" "J27" (id 0) (at 130.302 52.2732 0)
       (effects (font (size 1.27 1.27)) (justify right))
     )
@@
   (symbol (lib_id "ao_symbols:AudioJack2") (at 125.73 64.77 180) (unit 1)
     (in_bom yes) (on_board yes)
-    (property "Reference" "J22" (id 0) (at 130.302 64.3382 0)
+    (property "Reference" "J28" (id 0) (at 130.302 64.3382 0)
       (effects (font (size 1.27 1.27)) (justify right))
     )
@@
   (symbol (lib_id "ao_symbols:AudioJack2") (at 125.73 76.835 180) (unit 1)
     (in_bom yes) (on_board yes)
-    (property "Reference" "J23" (id 0) (at 130.302 76.4032 0)
+    (property "Reference" "J29" (id 0) (at 130.302 76.4032 0)
       (effects (font (size 1.27 1.27)) (justify right))
     )
@@
   (symbol (lib_id "ao_symbols:AudioJack2") (at 88.9 40.64 0) (mirror x) (unit 1)
     (in_bom yes) (on_board yes)
-    (property "Reference" "J14" (id 0) (at 84.328 40.2082 0)
+    (property "Reference" "J20" (id 0) (at 84.328 40.2082 0)
       (effects (font (size 1.27 1.27)) (justify right))
     )
@@
   (symbol (lib_id "ao_symbols:AudioJack2") (at 88.9 52.705 0) (mirror x) (unit 1)
     (in_bom yes) (on_board yes)
-    (property "Reference" "J15" (id 0) (at 84.328 52.2732 0)
+    (property "Reference" "J21" (id 0) (at 84.328 52.2732 0)
       (effects (font (size 1.27 1.27)) (justify right))
     )
@@
   (symbol (lib_id "ao_symbols:AudioJack2") (at 88.9 64.77 0) (mirror x) (unit 1)
     (in_bom yes) (on_board yes)
-    (property "Reference" "J16" (id 0) (at 84.328 64.3382 0)
+    (property "Reference" "J22" (id 0) (at 84.328 64.3382 0)
       (effects (font (size 1.27 1.27)) (justify right))
     )
@@
   (symbol (lib_id "ao_symbols:AudioJack2") (at 88.9 76.835 0) (mirror x) (unit 1)
     (in_bom yes) (on_board yes)
-    (property "Reference" "J17" (id 0) (at 84.328 76.4032 0)
+    (property "Reference" "J23" (id 0) (at 84.328 76.4032 0)
       (effects (font (size 1.27 1.27)) (justify right))
     )
@@
   (symbol (lib_id "ao_symbols:AudioJack2") (at 88.9 88.9 0) (mirror x) (unit 1)
     (in_bom yes) (on_board yes)
-    (property "Reference" "J18" (id 0) (at 84.328 88.4682 0)
+    (property "Reference" "J24" (id 0) (at 84.328 88.4682 0)
       (effects (font (size 1.27 1.27)) (justify right))
     )
@@
   (symbol (lib_id "ao_symbols:Synth_power_2x5") (at 97.155 140.97 0) (unit 1)
     (in_bom yes) (on_board yes)
-    (property "Reference" "J19" (id 0) (at 97.155 129.6162 0)
+    (property "Reference" "J25" (id 0) (at 97.155 129.6162 0)
       (effects (font (size 1.524 1.524)))
     )
@@
   (symbol (lib_id "ao_symbols:AudioJack2") (at 127 89.535 0) (mirror x) (unit 1)
     (in_bom yes) (on_board yes)
-    (property "Reference" "J24" (id 0) (at 122.428 89.1032 0)
-      (effects (font (size 1.27 1.27)) (justify right))
-    )
+    (property "Reference" "J30" (id 0) (at 122.428 89.1032 0)
+      (effects (font (size 1.27 1.27)) (justify right))
+    )

Commit message: Schematics tweaks, silk and fab cleanup, layout PDFs, panel revisions
Parts:
- renumbered J20 to J18, J21 to J19, J22 to J20, J23 to J21, J24 to J22, J25 to J23, J26 to J24, J27 to J25, J28 to J26, J29 to J27, J30 to J28, TP4 to TP7, TP5 to TP8, TP6 to TP9
Changed lines of the file:
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@@
   (symbol (lib_id "ao_symbols:AudioJack2") (at 125.73 40.64 180) (unit 1)
     (in_bom yes) (on_board yes)
-    (property "Reference" "J26" (id 0) (at 130.302 40.2082 0)
+    (property "Reference" "J24" (id 0) (at 130.302 40.2082 0)
       (effects (font (size 1.27 1.27)) (justify right))
     )
@@
   (symbol (lib_id "ao_symbols:AudioJack2") (at 125.73 52.705 180) (unit 1)
     (in_bom yes) (on_board yes)
-    (property "Reference" "J27" (id 0) (at 130.302 52.2732 0)
+    (property "Reference" "J25" (id 0) (at 130.302 52.2732 0)
       (effects (font (size 1.27 1.27)) (justify right))
     )
@@
   (symbol (lib_id "ao_symbols:AudioJack2") (at 125.73 64.77 180) (unit 1)
     (in_bom yes) (on_board yes)
-    (property "Reference" "J28" (id 0) (at 130.302 64.3382 0)
+    (property "Reference" "J26" (id 0) (at 130.302 64.3382 0)
       (effects (font (size 1.27 1.27)) (justify right))
     )
@@
   (symbol (lib_id "ao_symbols:AudioJack2") (at 125.73 76.835 180) (unit 1)
     (in_bom yes) (on_board yes)
-    (property "Reference" "J29" (id 0) (at 130.302 76.4032 0)
+    (property "Reference" "J27" (id 0) (at 130.302 76.4032 0)
       (effects (font (size 1.27 1.27)) (justify right))
     )
@@
   (symbol (lib_id "ao_symbols:AudioJack2") (at 88.9 40.64 0) (mirror x) (unit 1)
     (in_bom yes) (on_board yes)
-    (property "Reference" "J20" (id 0) (at 84.328 40.2082 0)
+    (property "Reference" "J18" (id 0) (at 84.328 40.2082 0)
       (effects (font (size 1.27 1.27)) (justify right))
     )
@@
   (symbol (lib_id "ao_symbols:AudioJack2") (at 88.9 52.705 0) (mirror x) (unit 1)
     (in_bom yes) (on_board yes)
-    (property "Reference" "J21" (id 0) (at 84.328 52.2732 0)
+    (property "Reference" "J19" (id 0) (at 84.328 52.2732 0)
       (effects (font (size 1.27 1.27)) (justify right))
     )
@@
   (symbol (lib_id "ao_symbols:AudioJack2") (at 88.9 64.77 0) (mirror x) (unit 1)
     (in_bom yes) (on_board yes)
-    (property "Reference" "J22" (id 0) (at 84.328 64.3382 0)
+    (property "Reference" "J20" (id 0) (at 84.328 64.3382 0)
       (effects (font (size 1.27 1.27)) (justify right))
     )
@@
   (symbol (lib_id "ao_symbols:AudioJack2") (at 88.9 76.835 0) (mirror x) (unit 1)
     (in_bom yes) (on_board yes)
-    (property "Reference" "J23" (id 0) (at 84.328 76.4032 0)
+    (property "Reference" "J21" (id 0) (at 84.328 76.4032 0)
       (effects (font (size 1.27 1.27)) (justify right))
     )
@@
   (symbol (lib_id "ao_symbols:AudioJack2") (at 88.9 88.9 0) (mirror x) (unit 1)
     (in_bom yes) (on_board yes)
-    (property "Reference" "J24" (id 0) (at 84.328 88.4682 0)
+    (property "Reference" "J22" (id 0) (at 84.328 88.4682 0)
       (effects (font (size 1.27 1.27)) (justify right))
     )
@@
   (symbol (lib_id "ao_symbols:Synth_power_2x5") (at 97.155 140.97 0) (unit 1)
     (in_bom yes) (on_board yes)
-    (property "Reference" "J25" (id 0) (at 97.155 129.6162 0)
+    (property "Reference" "J23" (id 0) (at 97.155 129.6162 0)
       (effects (font (size 1.524 1.524)))
     )
@@
   (symbol (lib_id "ao_symbols:AudioJack2") (at 127 89.535 0) (mirror x) (unit 1)
     (in_bom yes) (on_board yes)
-    (property "Reference" "J30" (id 0) (at 122.428 89.1032 0)
+    (property "Reference" "J28" (id 0) (at 122.428 89.1032 0)
       (effects (font (size 1.27 1.27)) (justify right))
     )
@@
   (symbol (lib_id "Connector:TestPoint") (at 104.14 156.21 0) (unit 1)
     (in_bom yes) (on_board yes)
-    (property "Reference" "TP4" (id 0) (at 105.6132 153.2128 0)
+    (property "Reference" "TP7" (id 0) (at 105.6132 153.2128 0)
       (effects (font (size 1.27 1.27)) (justify left))
     )
@@
   (symbol (lib_id "Connector:TestPoint") (at 123.19 156.21 0) (unit 1)
     (in_bom yes) (on_board yes)
-    (property "Reference" "TP5" (id 0) (at 124.6632 153.2128 0)
+    (property "Reference" "TP8" (id 0) (at 124.6632 153.2128 0)
       (effects (font (size 1.27 1.27)) (justify left))
     )
@@
   (symbol (lib_id "Connector:TestPoint") (at 142.24 156.21 0) (unit 1)
     (in_bom yes) (on_board yes)
-    (property "Reference" "TP6" (id 0) (at 143.7132 153.2128 0)
-      (effects (font (size 1.27 1.27)) (justify left))
-    )
+    (property "Reference" "TP9" (id 0) (at 143.7132 153.2128 0)
+      (effects (font (size 1.27 1.27)) (justify left))
+    )
