File: Hardware/PCB/herovco/jackspower.kicad_sch (KiCad schematic)
At the start: 25 parts, among them J18 AudioJack2, J19 AudioJack2, J20 AudioJack2, J21 AudioJack2, J22 AudioJack2, J23 Synth_power_2x5, J24 AudioJack2, J25 AudioJack2, J26 AudioJack2, J27 AudioJack2, J28 AudioJack2

Commit message: Initial BOM; DNF the test points; README typo
Parts:
- TP7, TP8, TP9: Config (none) -> DNF
Changed lines of the file:
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@@
+      (effects (font (size 1.27 1.27)) hide)
+    )
+    (property "Config" "DNF" (id 4) (at 104.14 156.21 0)
       (effects (font (size 1.27 1.27)) hide)
     )
@@
       (effects (font (size 1.27 1.27)) hide)
     )
+    (property "Config" "DNF" (id 4) (at 123.19 156.21 0)
+      (effects (font (size 1.27 1.27)) hide)
+    )
     (pin "1")
   )
@@
       (effects (font (size 1.27 1.27)) hide)
     )
+    (property "Config" "DNF" (id 4) (at 142.24 156.21 0)
+      (effects (font (size 1.27 1.27)) hide)
+    )

Commit message: Convert jack footprints to slotted; clean up silkscreen; add silkscreen notes to match resistors
Parts:
- J18, J19, J20, J21, J22, J24, J25, J26, J27, J28: footprint ao_tht:Jack_6.35mm_PJ_629HAN -> ao_tht:Jack_6.35mm_PJ_629HAN_slots
Changed lines of the file:
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@@
       (effects (font (size 1.27 1.27)) (justify right))
     )
-    (property "Footprint" "ao_tht:Jack_6.35mm_PJ_629HAN" (id 2) (at 125.73 40.64 0)
+    (property "Footprint" "ao_tht:Jack_6.35mm_PJ_629HAN_slots" (id 2) (at 125.73 40.64 0)
       (effects (font (size 1.27 1.27)) hide)
     )
@@
       (effects (font (size 1.27 1.27)) (justify right))
     )
-    (property "Footprint" "ao_tht:Jack_6.35mm_PJ_629HAN" (id 2) (at 125.73 52.705 0)
+    (property "Footprint" "ao_tht:Jack_6.35mm_PJ_629HAN_slots" (id 2) (at 125.73 52.705 0)
       (effects (font (size 1.27 1.27)) hide)
     )
@@
       (effects (font (size 1.27 1.27)) (justify right))
     )
-    (property "Footprint" "ao_tht:Jack_6.35mm_PJ_629HAN" (id 2) (at 125.73 64.77 0)
+    (property "Footprint" "ao_tht:Jack_6.35mm_PJ_629HAN_slots" (id 2) (at 125.73 64.77 0)
       (effects (font (size 1.27 1.27)) hide)
     )
@@
       (effects (font (size 1.27 1.27)) (justify right))
     )
-    (property "Footprint" "ao_tht:Jack_6.35mm_PJ_629HAN" (id 2) (at 125.73 76.835 0)
+    (property "Footprint" "ao_tht:Jack_6.35mm_PJ_629HAN_slots" (id 2) (at 125.73 76.835 0)
       (effects (font (size 1.27 1.27)) hide)
     )
@@
       (effects (font (size 1.27 1.27)) (justify right))
     )
-    (property "Footprint" "ao_tht:Jack_6.35mm_PJ_629HAN" (id 2) (at 88.9 40.64 0)
+    (property "Footprint" "ao_tht:Jack_6.35mm_PJ_629HAN_slots" (id 2) (at 88.9 40.64 0)
       (effects (font (size 1.27 1.27)) hide)
     )
@@
       (effects (font (size 1.27 1.27)) (justify right))
     )
-    (property "Footprint" "ao_tht:Jack_6.35mm_PJ_629HAN" (id 2) (at 88.9 52.705 0)
+    (property "Footprint" "ao_tht:Jack_6.35mm_PJ_629HAN_slots" (id 2) (at 88.9 52.705 0)
       (effects (font (size 1.27 1.27)) hide)
     )
@@
       (effects (font (size 1.27 1.27)) (justify right))
     )
-    (property "Footprint" "ao_tht:Jack_6.35mm_PJ_629HAN" (id 2) (at 88.9 64.77 0)
+    (property "Footprint" "ao_tht:Jack_6.35mm_PJ_629HAN_slots" (id 2) (at 88.9 64.77 0)
       (effects (font (size 1.27 1.27)) hide)
     )
@@
       (effects (font (size 1.27 1.27)) (justify right))
     )
-    (property "Footprint" "ao_tht:Jack_6.35mm_PJ_629HAN" (id 2) (at 88.9 76.835 0)
+    (property "Footprint" "ao_tht:Jack_6.35mm_PJ_629HAN_slots" (id 2) (at 88.9 76.835 0)
       (effects (font (size 1.27 1.27)) hide)
     )
@@
       (effects (font (size 1.27 1.27)) (justify right))
     )
-    (property "Footprint" "ao_tht:Jack_6.35mm_PJ_629HAN" (id 2) (at 88.9 88.9 0)
+    (property "Footprint" "ao_tht:Jack_6.35mm_PJ_629HAN_slots" (id 2) (at 88.9 88.9 0)
       (effects (font (size 1.27 1.27)) hide)
     )
@@
       (effects (font (size 1.27 1.27)) (justify right))
     )
-    (property "Footprint" "ao_tht:Jack_6.35mm_PJ_629HAN" (id 2) (at 127 89.535 0)
-      (effects (font (size 1.27 1.27)) hide)
-    )
+    (property "Footprint" "ao_tht:Jack_6.35mm_PJ_629HAN_slots" (id 2) (at 127 89.535 0)
+      (effects (font (size 1.27 1.27)) hide)
+    )
