File: Hardware/PCB/herovco/herovco_back.kicad_sch (KiCad schematic)
At the start: 34 parts, among them Q1 2N3904, Q2 2N3904, U6 TL074

Commit message: Change pot symbols and fix orientation, other small tweaks
Connections:
- net +12V_1: now also U6.4 (V+)
- net -12V_1: now also U6.11 (V-)
- net GND1: no longer U6.1
Changed lines of the file:
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@@
   (junction (at 213.36 127) (diameter 0) (color 0 0 0 0)
   )
-  (junction (at 85.09 149.86) (diameter 0) (color 0 0 0 0)
-  )
   (junction (at 57.15 74.93) (diameter 0) (color 0 0 0 0)
   )
@@
   )
   (junction (at 231.14 81.28) (diameter 0) (color 0 0 0 0)
-  )
-  (junction (at 85.09 134.62) (diameter 0) (color 0 0 0 0)
   )
   (junction (at 207.01 87.63) (diameter 0) (color 0 0 0 0)
@@
     )
   )
-  (hierarchical_label "SIN_S_CW_S" (shape input) (at 82.55 95.25 0)
+  (hierarchical_label "SIN_S_CW_S" (shape output) (at 82.55 95.25 0)
     (effects (font (size 1.27 1.27)) (justify left))
   )
-  (hierarchical_label "SIN_S_W_S" (shape input) (at 76.2 102.87 180)
+  (hierarchical_label "SIN_S_W_S" (shape output) (at 76.2 102.87 180)
     (effects (font (size 1.27 1.27)) (justify right))
   )
-  (hierarchical_label "SIN_S_CCW_S" (shape input) (at 69.85 95.25 180)
+  (hierarchical_label "SIN_S_CCW_S" (shape output) (at 69.85 95.25 180)
     (effects (font (size 1.27 1.27)) (justify right))
   )
@@
     (effects (font (size 1.27 1.27)) (justify left))
   )
-  (hierarchical_label "SIN_R_CCW_S" (shape input) (at 54.61 74.93 180)
+  (hierarchical_label "SIN_R_CCW_S" (shape output) (at 54.61 74.93 180)
     (effects (font (size 1.27 1.27)) (justify right))
   )
@@
     (effects (font (size 1.27 1.27)) (justify right))
   )
-  (hierarchical_label "SIN_R_W_S" (shape input) (at 40.64 69.85 0)
+  (hierarchical_label "SIN_R_W_S" (shape output) (at 40.64 69.85 0)
     (effects (font (size 1.27 1.27)) (justify left))
   )
@@
     (effects (font (size 1.27 1.27)) (justify right))
   )
-  (symbol (lib_id "Amplifier_Operational:TL074") (at 87.63 142.24 0)
+  (symbol (lib_name "TL074_2") (lib_id "Amplifier_Operational:TL074") (at 87.63 142.24 0) (unit 5)
     (in_bom yes) (on_board yes)
     (property "Reference" "U6" (id 0) (at 86.5632 141.0716 0)
@@
     (pin "2")
   )
-  (symbol (lib_id "ao_symbols:C") (at 95.25 138.43 0)
+  (symbol (lib_id "ao_symbols:C") (at 95.25 138.43 0) (unit 1)
     (in_bom yes) (on_board yes)
     (property "Reference" "C12" (id 0) (at 98.171 137.2616 0)
@@
     (pin "2")
   )
-  (symbol (lib_id "ao_symbols:C") (at 95.25 146.05 0)
+  (symbol (lib_id "ao_symbols:C") (at 95.25 146.05 0) (unit 1)
     (in_bom yes) (on_board yes)
     (property "Reference" "C13" (id 0) (at 98.171 144.8816 0)
@@
     (pin "7")
   )
-  (symbol (lib_id "Amplifier_Operational:TL074") (at 222.25 49.53 0) (unit 3)
+  (symbol (lib_name "TL074_3") (lib_id "Amplifier_Operational:TL074") (at 222.25 49.53 0) (unit 3)
     (in_bom yes) (on_board yes)
     (property "Reference" "U6" (id 0) (at 222.25 40.2082 0))
@@
     (pin "9")
   )
-  (symbol (lib_id "Amplifier_Operational:TL074") (at 222.25 81.28 0) (unit 1)
+  (symbol (lib_name "TL074_4") (lib_id "Amplifier_Operational:TL074") (at 222.25 81.28 0) (unit 1)
     (in_bom yes) (on_board yes)
     (property "Reference" "U6" (id 0) (at 222.25 71.9582 0))
@@
     (pin "2")
   )
-  (symbol (lib_id "Amplifier_Operational:TL074") (at 114.3 66.04 0) (mirror x) (unit 4)
+  (symbol (lib_name "TL074_1") (lib_id "Amplifier_Operational:TL074") (at 114.3 66.04 0) (mirror x) (unit 4)
     (in_bom yes) (on_board yes)
     (property "Reference" "U6" (id 0) (at 116.84 59.69 0))

Commit message: Pre-breadboard updates
Parts:
- R53, R54: symbol Device:R -> ao_symbols:R; Vendor (none) -> Tayda
- U6: symbol Amplifier_Operational:TL074 -> ao_symbols:TL074; SKU (none) -> A-1138; Vendor (none) -> Tayda
Changed lines of the file:
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@@
     (comment 1 "or neighboring rights to this work. Published from United States.")
     (comment 2 "To the extent possible under law, Richard Holmes has waived all copyright and related ")
-    (comment 3 "Based mainly on Kassutronics VCO 3340")
+    (comment 3 "Partly based on designs by Kassutronics, Thomas Henry, and LMNC")
   )
   (junction (at 213.36 92.71) (diameter 0) (color 0 0 0 0)
@@
     (effects (font (size 1.27 1.27)) (justify right))
   )
-  (symbol (lib_name "TL074_2") (lib_id "Amplifier_Operational:TL074") (at 87.63 142.24 0) (unit 5)
+  (symbol (lib_id "ao_symbols:TL074") (at 87.63 142.24 0) (unit 5)
     (in_bom yes) (on_board yes)
     (property "Reference" "U6" (id 0) (at 86.5632 141.0716 0)
@@
     )
     (property "Datasheet" "http://www.ti.com/lit/ds/symlink/tl071.pdf" (id 3) (at 88.9 137.16 0)
+      (effects (font (size 1.27 1.27)) hide)
+    )
+    (property "Vendor" "Tayda" (id 4) (at 87.63 142.24 0)
+      (effects (font (size 1.27 1.27)) hide)
+    )
+    (property "SKU" "A-1138" (id 5) (at 87.63 142.24 0)
       (effects (font (size 1.27 1.27)) hide)
     )
@@
     (pin "1")
   )
-  (symbol (lib_id "Amplifier_Operational:TL074") (at 222.25 115.57 0) (unit 2)
+  (symbol (lib_id "ao_symbols:TL074") (at 222.25 115.57 0) (unit 2)
     (in_bom yes) (on_board yes)
     (property "Reference" "U6" (id 0) (at 222.25 106.2482 0))
@@
       (effects (font (size 1.27 1.27)) hide)
     )
+    (property "Vendor" "Tayda" (id 4) (at 222.25 115.57 0)
+      (effects (font (size 1.27 1.27)) hide)
+    )
+    (property "SKU" "A-1138" (id 5) (at 222.25 115.57 0)
+      (effects (font (size 1.27 1.27)) hide)
+    )
     (pin "5")
     (pin "6")
     (pin "7")
   )
-  (symbol (lib_name "TL074_3") (lib_id "Amplifier_Operational:TL074") (at 222.25 49.53 0) (unit 3)
+  (symbol (lib_id "ao_symbols:TL074") (at 222.25 49.53 0) (unit 3)
     (in_bom yes) (on_board yes)
     (property "Reference" "U6" (id 0) (at 222.25 40.2082 0))
@@
       (effects (font (size 1.27 1.27)) hide)
     )
+    (property "Vendor" "Tayda" (id 4) (at 222.25 49.53 0)
+      (effects (font (size 1.27 1.27)) hide)
+    )
+    (property "SKU" "A-1138" (id 5) (at 222.25 49.53 0)
+      (effects (font (size 1.27 1.27)) hide)
+    )
     (pin "10")
     (pin "8")
     (pin "9")
   )
-  (symbol (lib_name "TL074_4") (lib_id "Amplifier_Operational:TL074") (at 222.25 81.28 0) (unit 1)
+  (symbol (lib_id "ao_symbols:TL074") (at 222.25 81.28 0) (unit 1)
     (in_bom yes) (on_board yes)
     (property "Reference" "U6" (id 0) (at 222.25 71.9582 0))
@@
       (effects (font (size 1.27 1.27)) hide)
     )
+    (property "Vendor" "Tayda" (id 4) (at 222.25 81.28 0)
+      (effects (font (size 1.27 1.27)) hide)
+    )
+    (property "SKU" "A-1138" (id 5) (at 222.25 81.28 0)
+      (effects (font (size 1.27 1.27)) hide)
+    )
     (pin "1")
     (pin "2")
@@
     (pin "2")
   )
-  (symbol (lib_id "Device:R") (at 201.93 87.63 270) (unit 1)
+  (symbol (lib_id "ao_symbols:R") (at 201.93 87.63 270) (unit 1)
     (in_bom yes) (on_board yes)
     (property "Reference" "R53" (id 0) (at 201.93 82.3722 90))
@@
       (effects (font (size 1.27 1.27)) hide)
     )
+    (property "Vendor" "Tayda" (id 4) (at 201.93 87.63 0)
+      (effects (font (size 1.27 1.27)) hide)
+    )
     (pin "1")
     (pin "2")
@@
     (pin "2")
   )
-  (symbol (lib_id "Device:R") (at 201.93 121.92 270) (unit 1)
+  (symbol (lib_id "ao_symbols:R") (at 201.93 121.92 270) (unit 1)
     (in_bom yes) (on_board yes)
     (property "Reference" "R54" (id 0) (at 201.93 116.6622 90))
@@
       (effects (font (size 1.27 1.27)) hide)
     )
+    (property "Vendor" "Tayda" (id 4) (at 201.93 121.92 0)
+      (effects (font (size 1.27 1.27)) hide)
+    )
     (pin "1")
     (pin "2")
@@
     (pin "2")
   )
-  (symbol (lib_name "TL074_1") (lib_id "Amplifier_Operational:TL074") (at 114.3 66.04 0) (mirror x) (unit 4)
+  (symbol (lib_id "ao_symbols:TL074") (at 114.3 66.04 0) (mirror x) (unit 4)
     (in_bom yes) (on_board yes)
     (property "Reference" "U6" (id 0) (at 116.84 59.69 0))
@@
       (effects (font (size 1.27 1.27)) hide)
     )
+    (property "Vendor" "Tayda" (id 4) (at 114.3 66.04 0)
+      (effects (font (size 1.27 1.27)) hide)
+    )
+    (property "SKU" "A-1138" (id 5) (at 114.3 66.04 0)
+      (effects (font (size 1.27 1.27)) hide)
+    )

Commit message: Panel updates; reannotate; correct PCB errors
Parts:
- renumbered C12 to C15, C13 to C16, C14 to C17, C15 to C18, R38 to R39, R39 to R40, R40 to R41, R41 to R42, R42 to R43, R43 to R44, R44 to R45, R45 to R46, R46 to R47, R47 to R48, R48 to R49, R49 to R50, R50 to R51, R51 to R52, R52 to R53, R53 to R54, R54 to R55, R55 to R56, R56 to R57, R57 to R58, R58 to R59, R59 to R60, R60 to R61, R61 to R62, R62 to R63, R63 to R64

Commit message: Sync input revision
Parts:
- renumbered C15 to C16, C16 to C17, C17 to C18, C18 to C19, R39 to R42, R40 to R43, R41 to R44, R42 to R45, R43 to R46, R44 to R47, R45 to R48, R46 to R49, R47 to R50, R48 to R51, R49 to R52, R50 to R53, R51 to R54, R52 to R55, R53 to R56, R54 to R57, R55 to R58, R56 to R59, R57 to R60, R58 to R61, R59 to R62, R60 to R63, R61 to R64, R62 to R65, R63 to R66, R64 to R67

Commit message: Sch cleanup, switch footprint
Changed lines of the file:
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@@
-    (effects (font (size 1.27 1.27)) (justify left))
-  )
-  (hierarchical_label "GND_BACK" (shape input) (at 105.41 81.28 0)
     (effects (font (size 1.27 1.27)) (justify left))
   )
@@
   (symbol (lib_id "power:GND1") (at 106.68 142.24 0) (unit 1)
     (in_bom yes) (on_board yes)
-    (property "Reference" "#PWR072" (id 0) (at 106.68 148.59 0)
+    (property "Reference" "#PWR076" (id 0) (at 106.68 148.59 0)
       (effects (font (size 1.27 1.27)) hide)
     )
@@
   (symbol (lib_id "power:GND1") (at 207.01 66.04 0) (unit 1)
     (in_bom yes) (on_board yes)
-    (property "Reference" "#PWR078" (id 0) (at 207.01 72.39 0)
+    (property "Reference" "#PWR082" (id 0) (at 207.01 72.39 0)
       (effects (font (size 1.27 1.27)) hide)
     )
@@
   (symbol (lib_id "power:GND1") (at 191.77 97.79 0) (unit 1)
     (in_bom yes) (on_board yes)
-    (property "Reference" "#PWR073" (id 0) (at 191.77 104.14 0)
+    (property "Reference" "#PWR077" (id 0) (at 191.77 104.14 0)
       (effects (font (size 1.27 1.27)) hide)
     )
@@
   (symbol (lib_id "power:GND1") (at 207.01 97.79 0) (unit 1)
     (in_bom yes) (on_board yes)
-    (property "Reference" "#PWR079" (id 0) (at 207.01 104.14 0)
+    (property "Reference" "#PWR083" (id 0) (at 207.01 104.14 0)
       (effects (font (size 1.27 1.27)) hide)
     )
@@
   (symbol (lib_id "power:GND1") (at 191.77 132.08 0) (unit 1)
     (in_bom yes) (on_board yes)
-    (property "Reference" "#PWR074" (id 0) (at 191.77 138.43 0)
+    (property "Reference" "#PWR078" (id 0) (at 191.77 138.43 0)
       (effects (font (size 1.27 1.27)) hide)
     )
@@
   (symbol (lib_id "power:GND1") (at 207.01 132.08 0) (unit 1)
     (in_bom yes) (on_board yes)
-    (property "Reference" "#PWR080" (id 0) (at 207.01 138.43 0)
+    (property "Reference" "#PWR084" (id 0) (at 207.01 138.43 0)
       (effects (font (size 1.27 1.27)) hide)
     )
@@
   (symbol (lib_id "ao_symbols:+12V_1") (at 195.58 54.61 0) (unit 1)
     (in_bom yes) (on_board yes)
-    (property "Reference" "#PWR075" (id 0) (at 195.58 58.42 0)
+    (property "Reference" "#PWR079" (id 0) (at 195.58 58.42 0)
       (effects (font (size 1.27 1.27)) hide)
     )
@@
   (symbol (lib_id "ao_symbols:+12V_1") (at 76.2 49.53 0) (unit 1)
     (in_bom yes) (on_board yes)
-    (property "Reference" "#PWR066" (id 0) (at 76.2 53.34 0)
+    (property "Reference" "#PWR070" (id 0) (at 76.2 53.34 0)
       (effects (font (size 1.27 1.27)) hide)
     )
@@
   (symbol (lib_id "ao_symbols:+12V_1") (at 85.09 134.62 0) (unit 1)
     (in_bom yes) (on_board yes)
-    (property "Reference" "#PWR067" (id 0) (at 85.09 138.43 0)
+    (property "Reference" "#PWR071" (id 0) (at 85.09 138.43 0)
       (effects (font (size 1.27 1.27)) hide)
     )
@@
   (symbol (lib_id "ao_symbols:+12V_1") (at 195.58 86.36 0) (unit 1)
     (in_bom yes) (on_board yes)
-    (property "Reference" "#PWR076" (id 0) (at 195.58 90.17 0)
+    (property "Reference" "#PWR080" (id 0) (at 195.58 90.17 0)
       (effects (font (size 1.27 1.27)) hide)
     )
@@
   (symbol (lib_id "ao_symbols:+12V_1") (at 195.58 120.65 0) (unit 1)
     (in_bom yes) (on_board yes)
-    (property "Reference" "#PWR077" (id 0) (at 195.58 124.46 0)
+    (property "Reference" "#PWR081" (id 0) (at 195.58 124.46 0)
       (effects (font (size 1.27 1.27)) hide)
     )
@@
   (symbol (lib_id "power:GND1") (at 105.41 81.28 0) (unit 1)
     (in_bom yes) (on_board yes)
-    (property "Reference" "#PWR071" (id 0) (at 105.41 87.63 0)
+    (property "Reference" "#PWR075" (id 0) (at 105.41 87.63 0)
       (effects (font (size 1.27 1.27)) hide)
     )
@@
   (symbol (lib_id "power:GND1") (at 95.25 87.63 0) (unit 1)
     (in_bom yes) (on_board yes)
-    (property "Reference" "#PWR070" (id 0) (at 95.25 93.98 0)
+    (property "Reference" "#PWR074" (id 0) (at 95.25 93.98 0)
       (effects (font (size 1.27 1.27)) hide)
     )
@@
   (symbol (lib_id "power:GND1") (at 57.15 87.63 0) (unit 1)
     (in_bom yes) (on_board yes)
-    (property "Reference" "#PWR065" (id 0) (at 57.15 93.98 0)
+    (property "Reference" "#PWR069" (id 0) (at 57.15 93.98 0)
       (effects (font (size 1.27 1.27)) hide)
     )
@@
   (symbol (lib_id "ao_symbols:-12V_1") (at 85.09 149.86 180) (unit 1)
     (in_bom yes) (on_board yes)
-    (property "Reference" "#PWR068" (id 0) (at 85.09 152.4 0)
+    (property "Reference" "#PWR072" (id 0) (at 85.09 152.4 0)
       (effects (font (size 1.27 1.27)) hide)
     )
@@
   (symbol (lib_id "ao_symbols:-12V_1") (at 88.9 105.41 180) (unit 1)
     (in_bom yes) (on_board yes)
-    (property "Reference" "#PWR069" (id 0) (at 88.9 107.95 0)
-      (effects (font (size 1.27 1.27)) hide)
-    )
+    (property "Reference" "#PWR073" (id 0) (at 88.9 107.95 0)
+      (effects (font (size 1.27 1.27)) hide)
+    )

Commit message: Sine trimmers to back board, misc accumulated tweaks
Parts:
- added RV10, RV9: 50k, ao_tht:Potentiometer_Bourns_3296W_Vertical_screw_centered, symbol ao_symbols:R_POT_TRIM_3296W
- added RV11: 5k, ao_tht:Potentiometer_Bourns_3296W_Vertical_screw_centered, symbol ao_symbols:R_POT_TRIM_3296W
Connections:
- net GND1: now also RV11.1
- net SIN: now also RV11.2, RV11.3
- net SIN_R_CCW_S: no longer names the net of Q1.2 (B), R43.1
- net SIN_R_CCW_S: now also RV9.1
- net SIN_R_W_S: no longer names the net of R42.1
- net SIN_R_W_S: now also RV9.2, RV9.3
- net SIN_S_CCW_S: no longer names the net of Q1.1 (E), R45.2
- net SIN_S_CCW_S: now also RV10.1
- net SIN_S_CW_S: no longer names the net of Q2.1 (E), R45.1
- net SIN_S_CW_S: now also RV10.3
- net SIN_S_W_S: no longer names the net of R47.2
- net SIN_S_W_S: now also RV10.2
Other:
- note added: "SINE TRIMMERS"
- note added: "Sine amplitude"
- note added: "Sine round"
- note added: "Sine symmetry"

Commit message: Schematics tweaks, silk and fab cleanup, layout PDFs, panel revisions
Parts:
- renumbered RV9 to RV10, RV10 to RV11, RV11 to RV12, U6 to U7
Changed lines of the file:
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@@
   (symbol (lib_id "ao_symbols:TL074") (at 87.63 142.24 0) (unit 5)
     (in_bom yes) (on_board yes)
-    (property "Reference" "U6" (id 0) (at 86.5632 141.0716 0)
+    (property "Reference" "U7" (id 0) (at 86.5632 141.0716 0)
       (effects (font (size 1.27 1.27)) (justify left))
     )
@@
   (symbol (lib_id "power:GND1") (at 207.01 66.04 0) (unit 1)
     (in_bom yes) (on_board yes)
-    (property "Reference" "#PWR082" (id 0) (at 207.01 72.39 0)
+    (property "Reference" "#PWR083" (id 0) (at 207.01 72.39 0)
       (effects (font (size 1.27 1.27)) hide)
     )
@@
   (symbol (lib_id "power:GND1") (at 191.77 97.79 0) (unit 1)
     (in_bom yes) (on_board yes)
-    (property "Reference" "#PWR077" (id 0) (at 191.77 104.14 0)
+    (property "Reference" "#PWR078" (id 0) (at 191.77 104.14 0)
       (effects (font (size 1.27 1.27)) hide)
     )
@@
   (symbol (lib_id "power:GND1") (at 207.01 97.79 0) (unit 1)
     (in_bom yes) (on_board yes)
-    (property "Reference" "#PWR083" (id 0) (at 207.01 104.14 0)
+    (property "Reference" "#PWR084" (id 0) (at 207.01 104.14 0)
       (effects (font (size 1.27 1.27)) hide)
     )
@@
   (symbol (lib_id "power:GND1") (at 191.77 132.08 0) (unit 1)
     (in_bom yes) (on_board yes)
-    (property "Reference" "#PWR078" (id 0) (at 191.77 138.43 0)
+    (property "Reference" "#PWR079" (id 0) (at 191.77 138.43 0)
       (effects (font (size 1.27 1.27)) hide)
     )
@@
   (symbol (lib_id "power:GND1") (at 207.01 132.08 0) (unit 1)
     (in_bom yes) (on_board yes)
-    (property "Reference" "#PWR084" (id 0) (at 207.01 138.43 0)
+    (property "Reference" "#PWR085" (id 0) (at 207.01 138.43 0)
       (effects (font (size 1.27 1.27)) hide)
     )
@@
   (symbol (lib_id "ao_symbols:+12V_1") (at 195.58 54.61 0) (unit 1)
     (in_bom yes) (on_board yes)
-    (property "Reference" "#PWR079" (id 0) (at 195.58 58.42 0)
+    (property "Reference" "#PWR080" (id 0) (at 195.58 58.42 0)
       (effects (font (size 1.27 1.27)) hide)
     )
@@
   (symbol (lib_id "ao_symbols:+12V_1") (at 195.58 86.36 0) (unit 1)
     (in_bom yes) (on_board yes)
-    (property "Reference" "#PWR080" (id 0) (at 195.58 90.17 0)
+    (property "Reference" "#PWR081" (id 0) (at 195.58 90.17 0)
       (effects (font (size 1.27 1.27)) hide)
     )
@@
   (symbol (lib_id "ao_symbols:+12V_1") (at 195.58 120.65 0) (unit 1)
     (in_bom yes) (on_board yes)
-    (property "Reference" "#PWR081" (id 0) (at 195.58 124.46 0)
+    (property "Reference" "#PWR082" (id 0) (at 195.58 124.46 0)
       (effects (font (size 1.27 1.27)) hide)
     )
@@
   (symbol (lib_id "ao_symbols:TL074") (at 222.25 115.57 0) (unit 2)
     (in_bom yes) (on_board yes)
-    (property "Reference" "U6" (id 0) (at 222.25 106.2482 0))
+    (property "Reference" "U7" (id 0) (at 222.25 106.2482 0))
     (property "Value" "TL074" (id 1) (at 222.25 108.5596 0))
     (property "Footprint" "ao_tht:DIP-14_W7.62mm_Socket_LongPads" (id 2) (at 220.98 113.03 0)
@@
   (symbol (lib_id "ao_symbols:TL074") (at 222.25 49.53 0) (unit 3)
     (in_bom yes) (on_board yes)
-    (property "Reference" "U6" (id 0) (at 222.25 40.2082 0))
+    (property "Reference" "U7" (id 0) (at 222.25 40.2082 0))
     (property "Value" "TL074" (id 1) (at 222.25 42.5196 0))
     (property "Footprint" "ao_tht:DIP-14_W7.62mm_Socket_LongPads" (id 2) (at 220.98 46.99 0)
@@
   (symbol (lib_id "ao_symbols:TL074") (at 222.25 81.28 0) (unit 1)
     (in_bom yes) (on_board yes)
-    (property "Reference" "U6" (id 0) (at 222.25 71.9582 0))
+    (property "Reference" "U7" (id 0) (at 222.25 71.9582 0))
     (property "Value" "TL074" (id 1) (at 222.25 74.2696 0))
     (property "Footprint" "ao_tht:DIP-14_W7.62mm_Socket_LongPads" (id 2) (at 220.98 78.74 0)
@@
   (symbol (lib_id "ao_symbols:TL074") (at 114.3 66.04 0) (mirror x) (unit 4)
     (in_bom yes) (on_board yes)
-    (property "Reference" "U6" (id 0) (at 116.84 59.69 0))
+    (property "Reference" "U7" (id 0) (at 116.84 59.69 0))
     (property "Value" "TL074" (id 1) (at 118.11 62.23 0))
     (property "Footprint" "ao_tht:DIP-14_W7.62mm_Socket_LongPads" (id 2) (at 113.03 68.58 0)
@@
   (symbol (lib_id "power:GND1") (at 134.62 82.55 0) (unit 1)
     (in_bom yes) (on_board yes)
-    (property "Reference" "#PWR0101" (id 0) (at 134.62 88.9 0)
+    (property "Reference" "#PWR077" (id 0) (at 134.62 88.9 0)
       (effects (font (size 1.27 1.27)) hide)
     )
@@
   (symbol (lib_id "ao_symbols:R_POT_TRIM_3296W") (at 52.07 69.85 180) (unit 1)
     (in_bom yes) (on_board yes)
-    (property "Reference" "RV9" (id 0) (at 53.848 68.6816 0)
+    (property "Reference" "RV10" (id 0) (at 53.848 68.6816 0)
       (effects (font (size 1.27 1.27)) (justify right))
     )
@@
   (symbol (lib_id "ao_symbols:R_POT_TRIM_3296W") (at 134.62 76.2 0) (mirror x) (unit 1)
     (in_bom yes) (on_board yes)
-    (property "Reference" "RV11" (id 0) (at 132.842 75.0316 0)
+    (property "Reference" "RV12" (id 0) (at 132.842 75.0316 0)
       (effects (font (size 1.27 1.27)) (justify right))
     )
@@
   (symbol (lib_id "ao_symbols:R_POT_TRIM_3296W") (at 76.2 95.25 90) (mirror x) (unit 1)
     (in_bom yes) (on_board yes)
-    (property "Reference" "RV10" (id 0) (at 74.93 90.3986 90)
+    (property "Reference" "RV11" (id 0) (at 74.93 90.3986 90)
       (effects (font (size 1.27 1.27)) (justify right))
     )

Commit message: schem tweaks
Other:
- note removed: "SINE TRIMMERS"
Changed lines of the file:
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@@
     (effects (font (size 1.27 1.27)) (justify left bottom))
-  )
-  (text "SINE\nTRIMMERS" (at 27.94 107.95 0)
-    (effects (font (size 3.81 3.81)) (justify left bottom))
   )
   (text "Kassutronics used 100k feedback resistors and\nsimilarly large values for voltage divider resistors. \nAS3340 datasheet calls for a 51k pulldown \non pin 4, so I reduced the voltage divider \nresistances by a factor ~ (51k/(180k+100k)). \nOp amp resistances were reduced by a factor \nof 10. Then stabilization caps were increased \nmore to make 1/(2πRC) ~ 50kHz."
