File: Hardware/PCB/herovco/herovco_back.kicad_sch (KiCad schematic)
At the start: 36 parts, among them Q1 2N3904, Q2 2N3904, U7 TL074

Commit message: 5 mm pitch for 330 pF
Parts:
- C18, C19: footprint ao_tht:C_Disc_D3.0mm_W1.6mm_P2.50mm -> ao_tht:C_Disc_D5.0mm_W2.5mm_P5.00mm
Changed lines of the file:
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@@
     (property "Reference" "C18" (id 0) (at 222.25 86.3092 90))
     (property "Value" "330pF" (id 1) (at 222.25 88.6206 90))
-    (property "Footprint" "ao_tht:C_Disc_D3.0mm_W1.6mm_P2.50mm" (id 2) (at 218.44 93.6752 0)
+    (property "Footprint" "ao_tht:C_Disc_D5.0mm_W2.5mm_P5.00mm" (id 2) (at 218.44 93.6752 0)
       (effects (font (size 1.27 1.27)) hide)
     )
@@
     (property "Reference" "C19" (id 0) (at 222.25 120.5992 90))
     (property "Value" "330pF" (id 1) (at 222.25 122.9106 90))
-    (property "Footprint" "ao_tht:C_Disc_D3.0mm_W1.6mm_P2.50mm" (id 2) (at 218.44 127.9652 0)
+    (property "Footprint" "ao_tht:C_Disc_D5.0mm_W2.5mm_P5.00mm" (id 2) (at 218.44 127.9652 0)
       (effects (font (size 1.27 1.27)) hide)
     )

Commit message: Post prototype updates
Parts:
- RV10, RV11: SKU (none) -> A-598
- RV12: SKU (none) -> A-597
Changed lines of the file:
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@@
       (effects (font (size 1.27 1.27)) hide)
     )
+    (pin "1")
+    (pin "2")
+    (pin "3")
+    (pin "5")
+    (pin "6")
+    (pin "7")
+    (pin "10")
+    (pin "8")
+    (pin "9")
+    (pin "12")
+    (pin "13")
+    (pin "14")
     (pin "11")
     (pin "4")
@@
       (effects (font (size 1.27 1.27)) hide)
     )
+    (property "Description" "Ceramic capacitor, pitch 2.5 mm" (id 5) (at 95.25 138.43 0)
+      (effects (font (size 1.27 1.27)) hide)
+    )
     (pin "1")
     (pin "2")
@@
     )
     (property "Vendor" "Tayda" (id 4) (at 95.25 146.05 0)
+      (effects (font (size 1.27 1.27)) hide)
+    )
+    (property "Description" "Ceramic capacitor, pitch 2.5 mm" (id 5) (at 95.25 146.05 0)
       (effects (font (size 1.27 1.27)) hide)
     )
@@
       (effects (font (size 1.27 1.27)) hide)
     )
+    (pin "1")
+    (pin "2")
+    (pin "3")
     (pin "5")
     (pin "6")
     (pin "7")
+    (pin "10")
+    (pin "8")
+    (pin "9")
+    (pin "12")
+    (pin "13")
+    (pin "14")
+    (pin "11")
+    (pin "4")
   )
   (symbol (lib_id "ao_symbols:TL074") (at 222.25 49.53 0) (unit 3)
@@
       (effects (font (size 1.27 1.27)) hide)
     )
+    (pin "1")
+    (pin "2")
+    (pin "3")
+    (pin "5")
+    (pin "6")
+    (pin "7")
     (pin "10")
     (pin "8")
     (pin "9")
+    (pin "12")
+    (pin "13")
+    (pin "14")
+    (pin "11")
+    (pin "4")
   )
   (symbol (lib_id "ao_symbols:TL074") (at 222.25 81.28 0) (unit 1)
@@
     (pin "2")
     (pin "3")
+    (pin "5")
+    (pin "6")
+    (pin "7")
+    (pin "10")
+    (pin "8")
+    (pin "9")
+    (pin "12")
+    (pin "13")
+    (pin "14")
+    (pin "11")
+    (pin "4")
   )
   (symbol (lib_id "ao_symbols:R") (at 201.93 55.88 270) (unit 1)
@@
       (effects (font (size 1.27 1.27)) hide)
     )
+    (property "Description" "Ceramic capacitor, pitch 5 mm" (id 5) (at 222.25 92.71 0)
+      (effects (font (size 1.27 1.27)) hide)
+    )
     (pin "1")
     (pin "2")
@@
       (effects (font (size 1.27 1.27)) hide)
     )
+    (property "Description" "Ceramic capacitor, pitch 5 mm" (id 5) (at 222.25 127 0)
+      (effects (font (size 1.27 1.27)) hide)
+    )
     (pin "1")
     (pin "2")
@@
       (effects (font (size 1.27 1.27)) hide)
     )
+    (pin "1")
+    (pin "2")
+    (pin "3")
+    (pin "5")
+    (pin "6")
+    (pin "7")
+    (pin "10")
+    (pin "8")
+    (pin "9")
     (pin "12")
     (pin "13")
     (pin "14")
+    (pin "11")
+    (pin "4")
   )
   (symbol (lib_id "ao_symbols:R") (at 130.81 66.04 270) (unit 1)
@@
       (effects (font (size 1.27 1.27)) hide)
     )
+    (property "Description" "3296W trimmer potentiometer" (id 5) (at 52.07 69.85 0)
+      (effects (font (size 1.27 1.27)) hide)
+    )
+    (property "SKU" "A-598" (id 6) (at 52.07 69.85 0)
+      (effects (font (size 1.27 1.27)) hide)
+    )
     (pin "1")
     (pin "2")
@@
       (effects (font (size 1.27 1.27)) hide)
     )
+    (property "Description" "3296W trimmer potentiometer" (id 5) (at 134.62 76.2 0)
+      (effects (font (size 1.27 1.27)) hide)
+    )
+    (property "SKU" "A-597" (id 6) (at 134.62 76.2 0)
+      (effects (font (size 1.27 1.27)) hide)
+    )
     (pin "1")
     (pin "2")
@@
       (effects (font (size 1.27 1.27)) hide)
     )
+    (property "Description" "3296W trimmer potentiometer" (id 5) (at 76.2 95.25 0)
+      (effects (font (size 1.27 1.27)) hide)
+    )
+    (property "SKU" "A-598" (id 6) (at 76.2 95.25 0)
+      (effects (font (size 1.27 1.27)) hide)
+    )
