File: Hardware/Panel/herovco_panel/herovco_panel.kicad_pcb (KiCad board)
At the start: 2 copper layers, 100 x 200 mm, 31 parts

Commit message: Rear panel labels
Other:
- board text added: "Ctr freq"
- board text added: "Exp FM jack"
- board text added: "Exp FM pot"
- board text added: "Fine tune pot"
- board text added: "HFT"
- board text added: "Hard/soft sync switch"
- board text added: "Lin FM jack"
- board text added: "Lin FM pot"
- board text added: "Octave rotary switch"
- board text added: "PW pot"
- board text added: "PWM jack"
- board text added: "PWM lim"
- board text added: "PWM pot"
- board text added: "Pulse jack"
- board text added: "Saw jack"
- board text added: "Sin amp"
- board text added: "Sin jack"
- board text added: "Sin round"
- board text added: "Sin symm"
- board text added: "Sync jack"
- board text added: "TP1"
- board text added: "Track"
- board text added: "Tri jack"
- board text added: "V/oct 1 jack"
- board text added: "V/oct 2 jack"
- board text added: "Vref"

Commit message: Panel revision, Gerbers
Parts:
- removed the H20 at (110.1, 57.6)
- removed the H21 at (110.1, 47.6)
- removed the H23 at (110.1, 37.6)
- removed H24, H28: Trimmer_Hole, Kosmo_panel:Kosmo_Trimmer_Pot_Hole
- H4: renamed from H9; footprint Kosmo_panel:Kosmo_Switch_Hole -> herovco_panel:Slide switch
- moved H11 20.0 mm to (110.1, 67.6)
- moved H12 20.0 mm to (110.1, 77.6)
- moved H5 20.0 mm to (110.1, 47.6)
- moved H6 20.0 mm to (110.1, 57.6)
- moved H4 2.00 mm to (28.6, 112.6)
- renumbered H16 to H10, H17 to H11, H18 to H12, H19 to H13, H5 to H14, H6 to H15, H22 to H16, H7 to H17, H8 to H18, H25 to H19, H26 to H20, H27 to H21, H11 to H22, H14 to H23, H10 to H3, H12 to H5, H13 to H6, H15 to H7, H3 to H8, H4 to H9
Other:
- net class Default removed
- board text added: "Panel design by Rich Holmes CC0 1.0 Jan 2022 JLCJLCJLCJLC"
- board text removed: "Panel design by Rich Holmes CC0 1.0 ?? 2021 JLCJLCJLCJLC"
- board text removed: "Sin amp"
- board text removed: "Sin round"
- board text removed: "Sin symm"
- board text removed: "TP1"
- board text removed: "Vref"
