File: Hardware/PCB/herovco/Separate PCBs/herovco_back.kicad_pcb (KiCad board)
At the start: 2 copper layers, 94 x 156 mm, 64 parts, among them J10 Conn_01x03, J11 Conn_01x03, J17 Conn_02x04_Odd_Even, J18 AudioJack2, J19 AudioJack2, J20 AudioJack2, J21 AudioJack2, J22 AudioJack2, J23 Synth_power_2x5, J24 AudioJack2, J25 AudioJack2, J26 AudioJack2, J27 AudioJack2, J28 AudioJack2, J9 Conn_01x09, Q1 2N3904, Q2 2N3904, U7 TL074

Commit message: Libraries, redo gerbers
Parts:
- C18, C19: footprint ao_tht:C_Disc_D3.0mm_W1.6mm_P2.50mm -> ao_tht:C_Disc_D5.0mm_W2.5mm_P5.00mm
- J18, J19, J20, J21, J22, J24, J25, J26, J27, J28: footprint ao_tht:Jack_6.35mm_PJ_629HAN -> ao_tht:Jack_6.35mm_PJ_629HAN_slots
- moved C18 6.01 mm to (149.9, 100.7)
- moved B2 3.91 mm to (158.7, 25.0)
- moved C14 3.91 mm to (162.6, 94.3)
- moved C15 3.91 mm to (168.9, 94.3)
- moved C16 3.91 mm to (157.4, 77.8)
- moved C17 3.91 mm to (177.7, 77.8)
- moved C19 3.91 mm to (154.9, 66.4)
- moved D3 3.91 mm to (170.1, 104.5)
- moved D4 3.91 mm to (170.1, 128.6)
- moved GRAF3 3.91 mm to (149.8, 49.0)
- moved GRAF4 3.91 mm to (160.8, 34.0)
- moved H4 3.91 mm to (192.8, 131.0)
- moved H5 3.91 mm to (141.8, 28.0)
- moved H6 3.91 mm to (123.3, 106.0)
- moved J10 3.91 mm to (163.1, 47.3)
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Routing:
- net Board_0-/Outputs and sin/LINK_OUT_SAW: track 44.2 -> 44.9 mm
