File: Hardware/PCB/herovco/Separate PCBs/herovco_front.kicad_pcb (KiCad board)
At the start: 2 copper layers, 94 x 125 mm, 78 parts, among them J1 Conn_01x09, J2 Conn_01x03, J3 Conn_01x03, J4 3_pin_Molex_header, J5 Wire pads, J6 Conn_01x01, J7 Conn_01x01, J8 Conn_01x01, U1 TL074, U2 TL072, U3 AS3340A, U4 LM4040BIZ-5, U5 LM4040BIZ-5, U6 L79L05_TO92

Commit message: Libraries, redo gerbers
Parts:
- added B1: Board, ao_tht:Board_Marker, F.Cu at (157.1, 36.5)
- R19, R2, R20, R30: moved to F.Cu
- U6: footprint Package_TO_SOT_THT:TO-92_Inline -> ao_tht:TO-92_Inline_Wide
- moved U6 1.70 mm to (180.8, 44.3)
- moved R8 1.56 mm to (166.9, 126.9)
- moved U1 1.56 mm to (150.4, 123.1)
- moved R23 1.56 mm to (152.9, 53.2)
- moved TP6 1.56 mm to (171.9, 38.0)
- moved R1 1.56 mm to (166.9, 69.7)
- moved R12 1.56 mm to (166.9, 105.3)
- moved R25 1.56 mm to (166.9, 65.9)
- moved R26 1.56 mm to (166.9, 78.6)
- moved R31 1.56 mm to (166.9, 101.5)
- moved C10 1.56 mm to (126.3, 87.5)
- moved D1 1.56 mm to (109.8, 79.9)
- moved J4 1.56 mm to (106.0, 101.5)
- moved C2 1.56 mm to (145.3, 90.0)
- moved C3 1.56 mm to (163.1, 100.2)
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Routing:
- net Board_0--12V: track 163.5 -> 164.5 mm
Other:
- board text added: "Match these 2 resistors"
- board text added: "Match these 4 resistors"
- board text added: "Octave switch with 10 matched resistors added"
- board text removed: "Octave switch"

Commit message: 20k trimmers to 10k
Parts:
- RV5, RV6: value 20k -> 10k
